File: emonDCbike/emonDCbike.brd (EAGLE design)
At the start: 95.2 x 71.1 mm, 61 parts, among them Q1 16Mhz XT49M-2016M, U1_TQFP ATMEGA328P

Commit message: folder update
Parts:
- removed C24: 0.1uF 100V, rcl:C0603
- added C17: 470uF 16V, rcl:E3,5-8
- C1: value 10UF -> 0.22uF 6.3V; device Panasonic-EEEFK_EEEFP:CAPAE430X610N -> rcl:C0402K
- C10, C2, C5, C7, C8: device rcl:C0603 -> rcl:C0402K
- C11, C4: device rcl:C0603 -> resistor:C0603
- C12: value 220nF -> 100nF 100V; device rcl:C0603 -> rcl:C0805K
- C13, C14, C21, C22, C48: value 100nF -> 0.1uF; device rcl:C0603 -> rcl:C0805K
- C15: value 220UF -> 10uF 35v; device Panasonic-EEE-EEV-EEF-ECQ:CAPAE1350X1400N -> rcl:E1,8-4
- C18: value 100UF -> 330UF 63V; device Panasonic-EEEFT_EEEH:CAPAE430X610N -> Panasonic-ECA_01:CAPPR500-1000X2000
- C3: value 470UF -> 100uF; device Panasonic-EEEFK_EEEFP:CAPAE830X1050N -> resistor:153CLV-0605
- C51: value 100nF -> 0.1uF; device rcl:C0603 -> resistor:C0805
- C6, C9: value 0.1uF 100V -> 100nF 100V; device rcl:C0603 -> rcl:C0805K
- moved C18 48.9 mm to (35.3, 49.3), turned to 270 degrees
- moved C15 38.1 mm to (70.8, 56.4), turned to 180 degrees
- moved C3 34.4 mm to (80.5, 66.9), turned to 180 degrees
- moved C1 28.2 mm to (47.3, 37.5), turned to 0 degrees
- moved C12 10.9 mm to (46.1, 27.8), turned to 90 degrees
- moved C9 10.5 mm to (43.6, 37.8)
- moved C21 9.78 mm to (62.7, 57.5), turned to 270 degrees
- moved LOGO1 6.36 mm to (24.4, 11.9)
- moved C6 3.22 mm to (43.4, 27.8), turned to 270 degrees
- moved C2 1.47 mm to (38.6, 7.73)
- moved R2 1.27 mm to (47.6, 40.7)
- moved UART 0.79 mm to (64.1, 20.5)
- moved R4 0.51 mm to (80.5, 50.7)
- moved C5 0.49 mm to (80.9, 48.5)
- moved R6 0.23 mm to (38.0, 10.1)
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- renumbered MC32882 to U$1
Connections:
- net 3.3V: now also C3.+; no longer C18.1
- net 5VHIGH: now also C17.+; no longer C3.1
- net 5VLOW: now also C15.+; no longer C1.1
- net D9/PWM1: now also C1.1; no longer C12.1
- net GND: now also C12.1, C15.-, C17.-, C3.-, C9.1; no longer C12.2, C15.2, C24.1, C3.2, C9.2
- net INPUTLINE: now also C9.2; no longer C24.2
- net N$7: now also C12.2; no longer C9.1
- net POWERIN: now also C18.1; no longer C15.1
Routing:
- net GND: track 16.1 -> 31.7 mm, vias 21 -> 23
- net 5VLOW: track 131.4 -> 122.7 mm, vias 4 -> 3
- net 5VHIGH: track 28.8 -> 24.3 mm
- net D9/PWM1: track 8.82 -> 6.49 mm
- net POWERIN: track 33.3 -> 31.5 mm
- net LOAD: track 18.0 -> 16.3 mm
- net N$10: track 3.21 -> 4.95 mm
- net INPUTLINE: track 57.1 -> 55.3 mm
- net RESET-ISO: track 2.95 -> 1.50 mm
- net N$2: track 5.15 -> 4.15 mm
- net D0/RX: track 49.8 -> 49.0 mm
- net N$7: track 8.39 -> 7.57 mm
- net D1/TX: track 59.8 -> 59.0 mm
- net N$3: track 5.18 -> 4.45 mm
- net D5/PWM0: track 59.4 -> 58.9 mm
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Other:
- board text added: "based on emonTx v3.4 by GH"
- board text added: "v0.2 Sept 2016 by DB"
- board text removed: "Designed in North Wales UK by Megni"
- board text removed: "MC32882"
- board text removed: "based on emonTx v3.4 by GH and TL"
- board text removed: "v0.3 Oct 2016 by DB"
