File: emonDCbike/emonDCbike.sch (EAGLE design)
At the start: 76 parts, among them Q1 16Mhz XT49M-2016M, U1_TQFP ATMEGA328P, X1 PSG01540, X2 PSG01540, X3 PSG01540, X4 PSG01540

Commit message: folder update
Parts:
- removed ATMEGA328: ATMEGA168MLF, SparkFun-DigitalIC:ATMEGA168MLF
- removed C23, C24, C25, C27: 100nF 100V, rcl:C-EUC0805K
- removed C26, C29: 100nF, rcl:C-EUC0402K
- removed LMP2: LMP8481SMCLMP8481, lmp8481b:LMP8481SMCLMP8481
- removed PAD1, PAD2, PAD3, PAD4, PAD6: WIREPAD2,54/1,1, wirepad:WIREPAD2,54/1,1
- removed R1: 1K, adafruit:R-US_R0603
- removed R11: 120K, adafruit:R-US_R0603
- removed R12, R9: 9K1, adafruit:R-US_R0603
- removed R8: 3.9K, adafruit:R-US_R0603
- removed V-READING_SEL: M20-9990346, SparkFun-Connectors:M03SMD_RA_FEMALE_NOWRITE
- removed X1, X2, X3, X4: PSG01540, con-lumberg:WBTOR1
- added AMP_POW_SEL: M20-9990346, SparkFun-Connectors:M03SMD_RA_FEMALE_NOWRITE
- added ANALOG, JP-LOAD, JP-SOURCE: 2212S-06SG-85, con-lsta:FE05-1
- added D1: BAT60J, diode:BAT60J
- added I/O: 2212S-02SG-85, SparkFun-Connectors:M02LOCK
- added JP1: 2211S-02G, jumper:JP1Q
- added UART: 2211S-06G, SparkFun:FTDI_BASICPTH
- C22: value 0.22uF 6.3V -> 0.1uF; device rcl:C-EUC0402K -> rcl:C-EUC0805K; MF AVX -> WALSIN; MPN 04026D224KAT2A -> 0805B104K160CT; OC_FARNELL 1327659 -> 2496942
- renumbered ISP1 to ISP
Connections:
- net ADC0A renamed ADCYES
- net NETDG renamed D9/PWM1
- removed net 5V: 3.3V_REG.VIN, 5V_REG.FEEDBACK, C12.2, C15.+, C17.+, C21.1, C25.2, C48.1, I1.P$2, LMP2.VCC, LMP8481.VCC, OK1.VCC, OK2.A, OK3.VCC, USB.VBUS
- removed net A6: ATMEGA328.ADC6, U1_TQFP.ADC6
- removed net A7: ATMEGA328.ADC7, U1_TQFP.ADC7
- removed net ACD2: ATMEGA328.PC2(ADC2), C29.1, R11.1, R12.2, U1_TQFP.PC2(ADC2)
- removed net ADC1A: R1.2, R9.2
- removed net ADC1AYEA: ATMEGA328.PC1(ADC1), C26.2, R9.1, U1_TQFP.PC1(ADC1)
- removed net D4/PWM0: ATMEGA328.PD4(XCK/T0), R2.2, U1_TQFP.PD4(XCK/T0)
- removed net D5/PWM1: ATMEGA328.PD5(T1), R8.2, U1_TQFP.PD5(T1)
- removed net INPUTLINE1: 5V_REG.VIN, C18.1, C51.1, C9.2, LMP8481.RSN, PAD1.P, V-READING_SEL.1, X1.T
- removed net INPUTLINE2: C24.2, LMP2.RSN, PAD3.P, V-READING_SEL.3, X4.T
- removed net N$5: ATMEGA328.PC4(ADC4/SDA), U1_TQFP.PC4(ADC4/SDA)
- removed net NETDF: C22.1, LMP2.REFA, LMP2.REFB, R8.1
- removed net TOLOAD1: C6.1, LMP8481.RSP, PAD2.P, X2.T
- removed net TOLOAD2: C23.1, LMP2.RSP, PAD4.P, X3.T
- removed net VSEL: C27.1, R11.2, V-READING_SEL.2
- new net 5VHIGH: 5V_REG.FEEDBACK, C17.+, C48.1, D1.A, I1.P$2
- new net 5VLOW: 3.3V_REG.VIN, AMP_POW_SEL.3, C15.+, C21.1, D1.C, OK1.VCC, OK2.A, OK3.VCC, UART.4, USB.VBUS
- new net ADC1: ANALOG.5, U1_TQFP.PC1(ADC1)
- new net ADC2: ANALOG.4, U1_TQFP.PC2(ADC2)
- new net ADC3: ANALOG.3, U1_TQFP.PC3(ADC3)
- new net D4: I/O.2, U1_TQFP.PD4(XCK/T0)
- new net D5/PWM0: R2.2, U1_TQFP.PD5(T1)
- new net INPUTLINE: AMP_POW_SEL.1, C9.2, JP-SOURCE.1, JP-SOURCE.2, JP-SOURCE.3, JP-SOURCE.4, JP-SOURCE.5, JP1.1, LMP8481.RSN
- new net LOAD: C6.1, JP-LOAD.1, JP-LOAD.2, JP-LOAD.3, JP-LOAD.4, JP-LOAD.5, LMP8481.RSP
- new net N$7: AMP_POW_SEL.2, C12.2, LMP8481.VCC
- new net POWERIN: 5V_REG.VIN, C18.1, C51.1, JP1.2
- net 3.3V: no longer ATMEGA328.AVCC, ATMEGA328.VCC@1, ATMEGA328.VCC@2
- net ADC4: now also ANALOG.2, U1_TQFP.PC4(ADC4/SDA); no longer ATMEGA328.PC3(ADC3), U1_TQFP.PC3(ADC3)
- net ADC5: now also ANALOG.1; no longer ATMEGA328.PC5(ADC5/SCL)
- net AGND: no longer ATMEGA328.AGND
- net D0/RX: now also UART.3; no longer ATMEGA328.PD0(RXD)
- net D1/TX: now also UART.2; no longer ATMEGA328.PD1(TXD)
- net D10: no longer ATMEGA328.PB2(SS/OC1B)
- net D11/MOSI: no longer ATMEGA328.PB3(MOSI/OC2)
- net D12/MISO: no longer ATMEGA328.PB4(MISO)
- net D13/SCK: no longer ATMEGA328.PB5(SCK)
- net D2: no longer ATMEGA328.PD2(INT0)
- net D3: now also I/O.1; no longer ATMEGA328.PD3(INT1), PAD6.P
- net D6: no longer ATMEGA328.PD6(AIN0)
- net D7: no longer ATMEGA328.PD7(AIN1)
- net D8: no longer ATMEGA328.PB0(ICP)
- net D9: no longer ATMEGA328.PB1(OC1A)
- net GND: now also UART.6; no longer ATMEGA328.GND@1, ATMEGA328.GND@2, C22.2, C23.2, C24.1, C25.1, C26.1, C27.2, C29.2, LMP2.GND, R12.1, X1.S, X2.S, X3.S, X4.S
- net N$1: no longer ATMEGA328.PB6(XTAL1/TOSC1)
- net N$2: no longer ATMEGA328.PC0(ADC0)
- net N$20: no longer ATMEGA328.AREF
- net N$3: now also C22.1, UART.1; no longer LMP2.VOUT, R1.1
- net N$9: no longer ATMEGA328.PB7(XTAL2/TOSC2)
- net RESET: now also C22.2; no longer ATMEGA328.PC6(/RESET)
Other:
- note added: "Shunt Amplifier"
- note removed: "Shunt Amplifiers"
- moved on the sheet: 3.3V_REG, C1, C12, C15, C22, C6, C9, R2, R5, S3
