File: emonDCbike/emonBike v0.2.sch (EAGLE design)
At the start: 24 parts

Commit message: updating v1.0
Parts:
- removed 3.3V_REG: REG1117, burr-brown:REG1117
- removed C13: 100nF, rcl:C-EUC0603
- removed C18: 10uF TANT, rcl:C-EUC0603
- removed SHUNTMON-A: LMP8481, lmp8481b:LMP8481LMP8481-H
- added C2: 10uF TANT, rcl:C-EUC0603
- added CURRENT_SENSE_AMP: ZXCT1086E5TA, Diodes_Inc-ZXCT1086E5TA:ZXCT1086E5TA
- added DUAL_ADC: MCP3002-I/SN, Microchip-MCP3002-I_SN:MCP3002-I/SN
- added U1YEAH: MAX5023TASA-T, MAX2053:MAX5023TASA-T
Connections:
- removed net 4.7V: SHUNTMON-A.VCC
- removed net 5.0V: 3.3V_REG.VIN, C1.1
- removed net INPUT-POS-A: PAD2.P, R1.R2, R2.2, SHUNTMON-A.RSP
- removed net LOAD-NEG-A: PAD1.P, R1.R1, SHUNTMON-A.RSN
- new net INPUT-POS: C2.1, U1YEAH.IN
- new net N$2: CURRENT_SENSE_AMP.S-, PAD1.P, R1.R1
- new net N$3: CURRENT_SENSE_AMP.S+, CURRENT_SENSE_AMP.VCC, PAD2.P, R1.R2, R2.2
- net 3.3V: now also C1.1, U1YEAH.OUT; no longer 3.3V_REG.VOUT, C13.1, C18.1
- net ADC: no longer SHUNTMON-A.VOUT
- net GND: now also C2.2, CURRENT_SENSE_AMP.GND, U1YEAH.GND; no longer 3.3V_REG.GND, C13.2, C18.2, SHUNTMON-A.GND, SHUNTMON-A.REFA, SHUNTMON-A.REFB
Other:
- note added: "Current Sense Amplifier"
- note added: "Daniel Bates Jan 2017"
- note added: "emonDCbike v0.1 : OpenEnergyMonitor.org"
- note removed: "4.7V AFTER DIODE TO 3.3V"
- note removed: "Daniel Bates Dec 2016"
- note removed: "Shunt Amplifier A"
- note removed: "emonDC v0.4 : based on emonTx v3.4 by Glyn Hudson and Trystan Lea OpenEnergyMonitor.org"
- moved on the sheet: C1, C21, C22, FTDI1, PAD1, PAD2, PAD3, PAD4, R1, R17, R18, R19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

Commit message: emonBIKE v0.2 camexport
Parts:
- removed DUAL_ADC: MCP3002-I/SN, Microchip-MCP3002-I_SN:MCP3002-I/SN
- removed R1: 0.022 OHM, Panasonic-ERJ3_ERJ8_ERJA_ERJB:ERJ-8CWFR022V
- removed R30: 10k, rcl:R-EU_R0603
- removed U$1: 47219-2001_MICROSD, 47219-2001_SD_MICRO:47219-2001_MICROSD
- removed U1YEAH: MAX5023TASA-T, MAX2053:MAX5023TASA-T
- added MAX2053: MAX5023TASA-T, MAX2053:MAX5023TASA-T
- added MCP3002: MCP3002-I/SN, Microchip-MCP3002-I_SN:MCP3002-I/SN
- added R_SENSE: 0.022 OHM, Panasonic-ERJ3_ERJ8_ERJA_ERJB:ERJ-8CWFR022V
- added U$2: MOLEX_MICRO_SD_1040310811, MOLEX MICRO SD [exposed pins]:MOLEX_MICRO_SD_1040310811
- C1: value 10uF TANT -> 10uF 16V TANT
- C2: value 10uF TANT -> 10uF 60V TANT
- renumbered CURRENT_SENSE_AMP to ZXCT1086
Connections:
- removed net 3.3V: C1.1, C22.2, ESP-12.VCC, R19.2, R6.2, R7.2, U$1.VDD, U1YEAH.OUT
- removed net ADCVSENSE-A: R2.1, R3.2
- removed net GPIO15: C22.1, ESP-12.GND, ESP-12.GPIO15, R30.2
- removed net INPUT-POS: C2.1, U1YEAH.IN
- removed net N$2: PAD1.P, R1.R1, ZXCT1086.S-
- removed net N$3: PAD2.P, R1.R2, R2.2, ZXCT1086.S+, ZXCT1086.VCC
- removed net N$32: U$1.DAT1
- removed net N$7: U$1.DAT2
- new net +3V3: C1.1, C22.2, ESP-12.VCC, MAX2053.OUT, MCP3002.VDD/VREF, R19.2, R6.2, R7.2, U$2.VDD
- new net ADC_CSENSE: MCP3002.CH1, ZXCT1086.OUT
- new net ADC_VSENSE: MCP3002.CH0, R2.1, R3.2
- new net LOAD-: PAD1.P, R_SENSE.R1, ZXCT1086.S-
- new net SOURCE+: C2.1, MAX2053.IN, PAD2.P, R2.2, R_SENSE.R2, ZXCT1086.S+, ZXCT1086.VCC
- net GND: now also C22.1, ESP-12.GND, ESP-12.GPIO15, MAX2053.GND, MCP3002.VSS, U$2.GND, U$2.VSS; no longer R30.1, U$1.GND, U$1.VSS, U1YEAH.GND
- net GPIO12: now also MCP3002.DOUT, U$2.DAT0; no longer U$1.DAT0
- net GPIO13: now also U$2.CMD; no longer U$1.CMD
- net GPIO14: now also MCP3002.CLK, U$2.CLK; no longer U$1.CLK
- net GPIO2: now also U$2.CD/DAT3; no longer U$1.CD/DAT3
- net GPIO4: now also MCP3002.~CS/SHDN
- net GPIO5: now also MCP3002.DIN
Other:
- note added: "DUAL ADC"
- note added: "Daniel Bates March 2017"
- note added: "PINS FREE 4 5 16"
- note added: "POWER"
- note added: "emonDCbike v0.2 : OpenEnergyMonitor.org"
- note removed: "Daniel Bates Jan 2017"
- note removed: "emonDCbike v0.1 : OpenEnergyMonitor.org"
- moved on the sheet: C1, C2, C21, C22, FTDI1, PAD1, PAD2, PAD4, R17, R18, R19, R2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

Commit message: tidy
Other:
- note added: "SHUNT MONITOR"
- note removed: "Current Sense Amplifier"
- moved on the sheet: C1, C2, C21, C22, FTDI1, MCP3002, R17, R18, R19, R6, R7
