File: emonDCuno/gotoDUO emonDC v0.3a.brd (EAGLE design)
At the start: 95.2 x 71.1 mm, 61 parts, among them Q1 16Mhz XT49M-2016M, U1_TQFP ATMEGA328P

Commit message: updating
Parts:
- removed AMP_POW_SEL: M20-9990346, SparkFun-Connectors:1X03_SMD_RA_FEMALE_NOWRITE
- removed ANALOG: 2212S-06SG-85, con-lsta:FE05-1
- removed C22: 0.1uF, rcl:C0805K
- removed JP1: 2211S-02G, jumper:JP1
- removed UART: 2211S-06G, SparkFun:FTDI_BASIC
- added ANA: 2212S-02SG-85, SparkFun-Connectors:1X02_LOCK
- added C25, C26, C6, C9: 0.1uF 100V, rcl:C0603
- added C27: 100nF, rcl:C0603
- added FTDI/UART: 2211S-06G, SparkFun:FTDI_BASIC
- added JP-LOAD1, JP-SOURCE1: 2212S-06SG-85, con-lsta:FE05-1
- added JP3: 2211S-02G, jumper:JP1
- added LMP1: LMP8481LMP8481-H, libsexportlmp8481b:S-PDSO-G08
- added R1, R14: 100K 60V, rcl:R0603
- added R11, R12, R13, R9: 1K, rcl:R0603
- added R15: 5.9K, rcl:R0603
- added R16: 9K1, rcl:R0603
- added R8: 3.9K, rcl:R0603
- added REFSEL: 2212S-02SG-85, SparkFun-Connectors:1X03
- added SC1, SC2: SOLDERJUMPERNO, SparkFun:SJ_2S-NO
- added T1, T2: (no value), con-weidmueller-sl35:180-2
- C1: value 0.22uF 6.3V -> 10UF; device rcl:C0402K -> Panasonic-EEEFK_EEEFP:CAPAE430X610N
- C10, C2, C5, C7, C8: device rcl:C0402K -> rcl:C0603
- C11, C4: device resistor:C0603 -> rcl:C0603
- C12: value 100nF 100V -> 220nF; device rcl:C0805K -> rcl:C0603
- C13, C14, C21, C48: value 0.1uF -> 100nF; device rcl:C0805K -> rcl:C0603
- C15: value 10uF 35v -> 220UF; device rcl:E1,8-4 -> Panasonic-EEE-EEV-EEF-ECQ:CAPAE1350X1400N
- C17: value 470uF 16V -> 100nF; device rcl:E3,5-8 -> rcl:C0603
- C18: value 330UF 63V -> 100UF; device Panasonic-ECA_01:CAPPR500-1000X2000 -> Panasonic-EEEFT_EEEH:CAPAE430X610N
- C23, C24: value 100nF 100V -> 0.1uF 100V; device Multicomp_By_element14_Batch_1:CAPC1608X85N -> rcl:C0603
- C3: value 100uF -> 470UF; device resistor:153CLV-0605 -> Panasonic-EEEFK_EEEFP:CAPAE830X1050N
- C51: value 0.1uF -> 100nF; device resistor:C0805 -> rcl:C0603
- LMP8481: value LMP8481SMCLMP8481 -> LMP8481-H; device lmp8481b:S-PDSO-G08 -> libsexportlmp8481b:S-PDSO-G08
- R2: value 3.9K -> 5.9K; device adafruit:R0603 -> rcl:R0603
- R3, R32, R4, R5, R6, R7: device adafruit:R0603 -> rcl:R0603
- moved C23 99.3 mm to (18.8, -113.0)
- moved C24 75.9 mm to (42.8, 34.6)
- moved C18 48.9 mm to (80.7, 67.6), turned to 0 degrees
- moved C15 38.1 mm to (33.1, 50.5), turned to 270 degrees
- moved C3 34.4 mm to (51.7, 48.1), turned to 270 degrees
- moved C17 31.9 mm to (42.9, 23.4), turned to 90 degrees
- moved C1 28.2 mm to (69.1, 55.4), turned to 180 degrees
- moved R2 24.5 mm to (23.3, 43.3), turned to 270 degrees
- moved C12 10.9 mm to (44.7, 38.6), turned to 180 degrees
- moved C21 9.78 mm to (71.8, 61.1), turned to 90 degrees
- moved LOGO1 6.36 mm to (21.0, 6.53)
- moved C2 1.47 mm to (40.1, 7.73)
- moved R5 1.30 mm to (51.0, 37.3)
- moved R4 0.51 mm to (80.5, 51.3)
- moved C5 0.49 mm to (80.5, 48.7)
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- renumbered U$1 to MC32882
Connections:
- net ADCYES renamed ADCSHUNT2
- removed net ADC1: ANALOG.5, U1_TQFP.24
- removed net ADC2: ANALOG.4, U1_TQFP.25
- removed net ADC3: ANALOG.3, U1_TQFP.26
- removed net ADC4: ANALOG.2, U1_TQFP.27
- removed net ADC5: ANALOG.1, U1_TQFP.28
- removed net D9/PWM1: C1.1, LMP8481.6, LMP8481.7, R2.1
- removed net INPUTLINE: AMP_POW_SEL.1, C23.1, JP-SOURCE.1, JP-SOURCE.2, JP-SOURCE.3, JP-SOURCE.4, JP-SOURCE.5, JP1.1, LMP8481.8
- removed net LOAD: C24.2, JP-LOAD.1, JP-LOAD.2, JP-LOAD.3, JP-LOAD.4, JP-LOAD.5, LMP8481.1
- removed net N$7: AMP_POW_SEL.2, C12.2, LMP8481.2
- new net ADCSHUNT1: R13.2, R16.2
- new net ADCVSENSE1: R14.1, R15.2, U1_TQFP.28
- new net ADCVSENSE2: R1.1, R2.2, U1_TQFP.27
- new net INPUTHIGH1: C25.1, JP-LOAD1.1, JP-LOAD1.2, JP-LOAD1.3, JP-LOAD1.4, JP-LOAD1.5, LMP1.1, R14.2, T1.2
- new net INPUTHIGH2: C6.1, JP-LOAD.1, JP-LOAD.2, JP-LOAD.3, JP-LOAD.4, JP-LOAD.5, JP3.2, LMP8481.1, R1.2, T2.2
- new net LOADLOW1: C23.2, JP-SOURCE1.1, JP-SOURCE1.2, JP-SOURCE1.3, JP-SOURCE1.4, JP-SOURCE1.5, LMP1.8, T1.1
- new net LOADLOW2: C24.2, JP-SOURCE.1, JP-SOURCE.2, JP-SOURCE.3, JP-SOURCE.4, JP-SOURCE.5, LMP8481.8, T2.1
- new net N$22: ANA.2, U1_TQFP.26
- new net N$23: ANA.1, U1_TQFP.25
- new net N$27: R16.1, U1_TQFP.24
- new net N$28: LMP1.6, LMP1.7, REFSEL.2
- new net N$4: LMP1.5, R13.1
- new net N$5: R9.1, SC1.2
- new net REFINPUT: C12.1, LMP8481.6, LMP8481.7, R8.1, REFSEL.1
- new net RES: C17.1, FTDI/UART.DTR, OK3.4, SC2.1
- net +5V-ISO: now also R12.1
- net 3.3V: now also C18.1; no longer C3.+
- net 5VHIGH: now also C3.1; no longer C17.+
- net 5VLOW: now also C1.1, C26.1, C9.1, FTDI/UART.VCC, LMP1.2, LMP8481.2, R11.2, R9.2; no longer AMP_POW_SEL.3, C15.+, UART.VCC
- net D0/RX: now also FTDI/UART.TXO, SC1.1; no longer UART.TXO
- net D1/TX: now also FTDI/UART.RXI; no longer UART.RXI
- net D5/PWM0: now also R8.2; no longer R2.2
- net GND: now also C12.2, C15.2, C23.1, C25.2, C26.2, C27.1, C3.2, C6.2, C9.2, FTDI/UART.GND, LMP1.4, R15.1, R2.1, REFSEL.3; no longer C12.1, C15.-, C17.-, C23.2, C3.-, UART.GND
- net N$2: now also C27.2
- net N$3: now also R11.1, SC2.2; no longer C22.1, UART.DTR
- net POWERIN: now also C15.1, JP3.1; no longer C18.1, JP1.2
- net RESET: now also C17.2; no longer C22.2, OK3.4
- net RX-ISO: now also R12.2
Routing:
- net ADCVSENSE1: track 0.00 -> 55.4 mm, vias 0 -> 2
- net INPUTLINE: track 49.1 -> 0.00 mm, vias 2 -> 0
- net INPUTHIGH2: track 0.00 -> 26.5 mm
- net LOADLOW2: track 0.00 -> 26.2 mm, vias 0 -> 2
- net 5VLOW: track 124.5 -> 103.5 mm, vias 3 -> 4
- net GND: track 31.6 -> 16.1 mm, vias 23 -> 22
- net +5V-ISO: track 63.0 -> 74.2 mm
- net ADCVSENSE2: track 0.00 -> 10.6 mm
- net LOAD: track 10.2 -> 0.00 mm
- net ADC5: track 9.78 -> 0.00 mm
- net REFINPUT: track 0.00 -> 8.82 mm
- net ADC4: track 7.85 -> 0.00 mm
- net N$7: track 7.57 -> 0.00 mm
- net N$22: track 0.00 -> 6.55 mm
- net D9/PWM1: track 6.49 -> 0.00 mm
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Other:
- board text added: "Designed in North Wales UK by Megni"
- board text added: "MC32882"
- board text added: "POWER SELECT"
- board text added: "UART / FTDI"
- board text added: "VSENSE"
- board text added: "based on emonTx v3.4 by GH and TL"
- board text added: "v0.3 Dec 2016 by DB"
- board text removed: "POWER"
- board text removed: "based on emonTx v3.4 by GH"
- board text removed: "v0.2 Sept 2016 by DB"
