File: emonDCuno/emonDC v0.2.sch (EAGLE design)
At the start: 61 parts, among them Q1 16Mhz XT49M-2016M, U1_TQFP ATMEGA328P

Commit message: RFM69 onto board
Other:
- note added: "RFM12B RFM69CW"
- note removed: "RFM12B RFM1269CW"
Changed lines of the file:
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@@
 <setting verticaltext="up"/>
 </settings>
-<grid distance="0.05" unitdist="inch" unit="inch" style="lines" multiple="1" display="no" altdistance="0.01" altunitdist="inch" altunit="inch"/>
+<grid distance="0.1" unitdist="inch" unit="inch" style="lines" multiple="1" display="no" altdistance="0.01" altunitdist="inch" altunit="inch"/>
 <layers>
 <layer number="1" name="Top" color="4" fill="1" visible="no" active="no"/>
@@
 <text x="94.615" y="370.84" size="3.81" layer="91">ATmega328</text>
 <text x="173.99" y="381.635" size="3.81" layer="91">RFM12B
-RFM1269CW</text>
+RFM69CW</text>
 <text x="263.144" y="377.063" size="2.54" layer="91">DIP
 Switch</text>
