File: emonDCduo/emonDC v0.3a.brd (EAGLE design)
At the start: 95.2 x 71.1 mm, 63 parts, among them Q1 16Mhz XT49M-2016M, U1_TQFP ATMEGA328P

Commit message: updating
Parts:
- removed AMP_POW_SEL: M20-9990346, SparkFun-Connectors:1X03_SMD_RA_FEMALE_NOWRITE
- removed C22: 100nF, rcl:C0603
- removed JP1: 2211S-02G, jumper:JP1
- removed SV1: (no value), con-lstb:MA04-1
- added ANA: 2212S-02SG-85, SparkFun-Connectors:1X02_LOCK
- added C17, C27: 100nF, rcl:C0603
- added C23, C25, C26: 0.1uF 100V, rcl:C0603
- added JP-LOAD1, JP-SOURCE1: 2212S-06SG-85, con-lsta:FE05-1
- added JP3: 2211S-02G, jumper:JP1
- added LMP1: LMP8481LMP8481-H, libsexportlmp8481b:S-PDSO-G08
- added R11, R12, R13, R9: 1K, rcl:R0603
- added R14: 100K 60V, rcl:R0603
- added R15: 5.9K, rcl:R0603
- added R16: 9K1, rcl:R0603
- added REFSEL: 2212S-02SG-85, SparkFun-Connectors:1X03
- added SC1, SC2: SOLDERJUMPERNO, SparkFun:SJ_2S-NO
- added T1, T2: (no value), con-weidmueller-sl35:180-2
- LMP8481: value LMP8481SMCLMP8481 -> LMP8481-H; device lmp8481b:S-PDSO-G08 -> libsexportlmp8481b:S-PDSO-G08
- moved R5 1.30 mm to (51.0, 37.3)
- renumbered UART to FTDI/UART
Connections:
- net ADCSHUNT renamed ADCSHUNT2
- removed net ADC2: SV1.1, U1_TQFP.25
- removed net ADC3: SV1.2, U1_TQFP.26
- removed net ADC4: SV1.3, U1_TQFP.27
- removed net ADC5: SV1.4, U1_TQFP.28
- removed net ADCVSENSE: R1.1, R2.2, U1_TQFP.24
- removed net D9/PWM1: C12.1, LMP8481.6, LMP8481.7, R8.1
- removed net INPUTLINE: AMP_POW_SEL.1, C24.2, JP-SOURCE.1, JP-SOURCE.2, JP-SOURCE.3, JP-SOURCE.4, JP-SOURCE.5, JP1.1, LMP8481.8, R1.2
- removed net LOAD: C6.1, JP-LOAD.1, JP-LOAD.2, JP-LOAD.3, JP-LOAD.4, JP-LOAD.5, LMP8481.1
- removed net N$7: AMP_POW_SEL.2, C9.1, LMP8481.2
- new net ADCSHUNT1: R13.2, R16.2
- new net ADCVSENSE1: R14.1, R15.2, U1_TQFP.28
- new net ADCVSENSE2: R1.1, R2.2, U1_TQFP.27
- new net INPUTHIGH1: C25.1, JP-LOAD1.1, JP-LOAD1.2, JP-LOAD1.3, JP-LOAD1.4, JP-LOAD1.5, LMP1.1, R14.2, T1.2
- new net INPUTHIGH2: C6.1, JP-LOAD.1, JP-LOAD.2, JP-LOAD.3, JP-LOAD.4, JP-LOAD.5, JP3.2, LMP8481.1, R1.2, T2.2
- new net LOADLOW1: C23.2, JP-SOURCE1.1, JP-SOURCE1.2, JP-SOURCE1.3, JP-SOURCE1.4, JP-SOURCE1.5, LMP1.8, T1.1
- new net LOADLOW2: C24.2, JP-SOURCE.1, JP-SOURCE.2, JP-SOURCE.3, JP-SOURCE.4, JP-SOURCE.5, LMP8481.8, T2.1
- new net N$22: ANA.2, U1_TQFP.26
- new net N$23: ANA.1, U1_TQFP.25
- new net N$27: R16.1, U1_TQFP.24
- new net N$28: LMP1.6, LMP1.7, REFSEL.2
- new net N$4: LMP1.5, R13.1
- new net N$5: R9.1, SC1.2
- new net REFINPUT: C12.1, LMP8481.6, LMP8481.7, R8.1, REFSEL.1
- new net RES: C17.1, FTDI/UART.DTR, OK3.4, SC2.1
- net +5V-ISO: now also R12.1
- net 5VLOW: now also C26.1, C9.1, LMP1.2, LMP8481.2, R11.2, R9.2; no longer AMP_POW_SEL.3
- net D0/RX: now also SC1.1
- net GND: now also C23.1, C25.2, C26.2, C27.1, LMP1.4, R15.1, REFSEL.3
- net N$2: now also C27.2
- net N$3: now also R11.1, SC2.2; no longer C22.1, FTDI/UART.DTR
- net POWERIN: now also JP3.1; no longer JP1.2
- net RESET: now also C17.2; no longer C22.2, OK3.4
- net RX-ISO: now also R12.2
Routing:
- net ADCVSENSE: track 62.2 -> 0.00 mm, vias 4 -> 0
- net INPUTLINE: track 59.0 -> 0.00 mm, vias 2 -> 0
- net ADCVSENSE1: track 0.00 -> 55.4 mm, vias 0 -> 2
- net 5VLOW: track 131.4 -> 103.5 mm
- net INPUTHIGH2: track 0.00 -> 26.5 mm
- net LOADLOW2: track 0.00 -> 26.2 mm, vias 0 -> 2
- net LOAD: track 18.0 -> 0.00 mm
- net +5V-ISO: track 63.0 -> 74.2 mm
- net ADCVSENSE2: track 0.00 -> 10.6 mm
- net ADC5: track 9.08 -> 0.00 mm
- net REFINPUT: track 0.00 -> 8.82 mm
- net D9/PWM1: track 8.82 -> 0.00 mm
- net N$7: track 8.39 -> 0.00 mm
- net ADC4: track 6.94 -> 0.00 mm
- net N$22: track 0.00 -> 6.55 mm
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Other:
- board text added: "POWER SELECT"
- board text added: "UART / FTDI"
- board text added: "v0.3 Dec 2016 by DB"
- board text removed: "POWER"
- board text removed: "v0.3 Oct 2016 by DB"

Commit message: commit
Parts:
- SC1, SC2: value SOLDERJUMPERNO -> (none)
- moved JP-LOAD 22.1 mm to (12.8, 28.6)
- moved JP-SOURCE 22.1 mm to (12.8, 37.1)
- moved C15 18.1 mm to (19.5, 62.4), turned to 180 degrees
- moved C3 4.60 mm to (51.2, 52.7)
- moved R8 3.31 mm to (48.6, 37.4)
- moved R5 2.40 mm to (49.8, 35.2)
- moved D1 2.29 mm to (56.8, 58.5)
- moved C9 1.81 mm to (44.8, 29.0), turned to 180 degrees
- moved 5V_REG 1.78 mm to (35.2, 64.4)
- moved I1 1.78 mm to (50.5, 62.6)
- moved C12 1.27 mm to (44.7, 37.3)
- moved D2 0.80 mm to (44.9, 55.3)
- moved C51 0.76 mm to (41.7, 56.5)
Routing:
- net LOADLOW2: track 26.2 -> 11.9 mm, vias 2 -> 0
- net INPUTHIGH2: track 26.5 -> 13.8 mm
- net N$31: track 11.5 -> 0.00 mm
- net 5VHIGH: track 28.8 -> 34.6 mm
- net N$6: track 5.18 -> 1.88 mm
- net IND: track 9.54 -> 12.7 mm
- net REFINPUT: track 8.82 -> 11.5 mm
- net POWERIN: track 31.8 -> 34.4 mm
- net 5VLOW: track 103.5 -> 106.0 mm
- net D5/PWM0: track 59.4 -> 61.2 mm
