File: emonDCduo/emonDC v0.3a.sch (EAGLE design)
At the start: 63 parts, among them Q1 16Mhz XT49M-2016M, U1_TQFP ATMEGA328P

Commit message: updating
Parts:
- removed AMP_POW_SEL: M20-9990346, SparkFun-Connectors:M03SMD_RA_FEMALE_NOWRITE
- removed C22: 100nF, rcl:C-EUC0603
- removed JP1: 2211S-02G, jumper:JP1Q
- removed SV1: (no value), con-lstb:MA04-1
- removed UART: 2211S-06G, SparkFun:FTDI_BASICPTH
- added ANA: 2212S-02SG-85, SparkFun-Connectors:M02LOCK
- added C17, C27: 100nF, rcl:C-EUC0603
- added C23, C25, C26: 0.1uF 100V, rcl:C-EUC0603
- added FTDI/UART: 2211S-06G, SparkFun:FTDI_BASICPTH
- added JP-LOAD1, JP-SOURCE1: 2212S-06SG-85, con-lsta:FE05-1
- added JP3: 2211S-02G, jumper:JP1Q
- added LMP1: LMP8481LMP8481-H, libsexportlmp8481b:LMP8481LMP8481-H
- added R11, R12, R13, R9: 1K, rcl:R-EU_R0603
- added R14: 100K 60V, rcl:R-EU_R0603
- added R15: 5.9K, rcl:R-EU_R0603
- added R16: 9K1, rcl:R-EU_R0603
- added REFSEL: 2212S-02SG-85, SparkFun-Connectors:CONN_03
- added SC1, SC2: SOLDERJUMPERNO, SparkFun:SOLDERJUMPERNO
- added T1, T2: (no value), con-weidmueller-sl35:180-2
- LMP8481: value LMP8481SMCLMP8481 -> LMP8481-H; device lmp8481b:LMP8481SMCLMP8481 -> libsexportlmp8481b:LMP8481LMP8481-H; MPN LMP8481MME-S/NOPB -> LMP8481MME-H/NOPB
Connections:
- net ADCSHUNT renamed ADCSHUNT2
- removed net ADC2: SV1.1, U1_TQFP.PC2(ADC2)
- removed net ADC3: SV1.2, U1_TQFP.PC3(ADC3)
- removed net ADC4: SV1.3, U1_TQFP.PC4(ADC4/SDA)
- removed net ADC5: SV1.4, U1_TQFP.PC5(ADC5/SCL)
- removed net ADCVSENSE: R1.1, R2.2, U1_TQFP.PC1(ADC1)
- removed net D9/PWM1: C12.1, LMP8481.REFA, LMP8481.REFB, R8.1
- removed net INPUTLINE: AMP_POW_SEL.1, C24.2, JP-SOURCE.1, JP-SOURCE.2, JP-SOURCE.3, JP-SOURCE.4, JP-SOURCE.5, JP1.1, LMP8481.RSN, R1.2
- removed net LOAD: C6.1, JP-LOAD.1, JP-LOAD.2, JP-LOAD.3, JP-LOAD.4, JP-LOAD.5, LMP8481.RSP
- removed net N$7: AMP_POW_SEL.2, C9.1, LMP8481.VCC
- new net ADCSHUNT1: R13.2, R16.2
- new net ADCVSENSE1: R14.1, R15.2, U1_TQFP.PC5(ADC5/SCL)
- new net ADCVSENSE2: R1.1, R2.2, U1_TQFP.PC4(ADC4/SDA)
- new net INPUTHIGH1: C25.1, JP-LOAD1.1, JP-LOAD1.2, JP-LOAD1.3, JP-LOAD1.4, JP-LOAD1.5, LMP1.RSP, R14.2, T1.2
- new net INPUTHIGH2: C6.1, JP-LOAD.1, JP-LOAD.2, JP-LOAD.3, JP-LOAD.4, JP-LOAD.5, JP3.2, LMP8481.RSP, R1.2, T2.2
- new net LOADLOW1: C23.2, JP-SOURCE1.1, JP-SOURCE1.2, JP-SOURCE1.3, JP-SOURCE1.4, JP-SOURCE1.5, LMP1.RSN, T1.1
- new net LOADLOW2: C24.2, JP-SOURCE.1, JP-SOURCE.2, JP-SOURCE.3, JP-SOURCE.4, JP-SOURCE.5, LMP8481.RSN, T2.1
- new net N$22: ANA.2, U1_TQFP.PC3(ADC3)
- new net N$23: ANA.1, U1_TQFP.PC2(ADC2)
- new net N$27: R16.1, U1_TQFP.PC1(ADC1)
- new net N$28: LMP1.REFA, LMP1.REFB, REFSEL.2
- new net N$4: LMP1.VOUT, R13.1
- new net N$5: R9.1, SC1.2
- new net REFINPUT: C12.1, LMP8481.REFA, LMP8481.REFB, R8.1, REFSEL.1
- new net RES: C17.1, FTDI/UART.1, OK3.OUT, SC2.1
- net +5V-ISO: now also R12.1
- net 5VLOW: now also C26.1, C9.1, FTDI/UART.4, LMP1.VCC, LMP8481.VCC, R11.2, R9.2; no longer AMP_POW_SEL.3, UART.4
- net D0/RX: now also FTDI/UART.3, SC1.1; no longer UART.3
- net D1/TX: now also FTDI/UART.2; no longer UART.2
- net GND: now also C23.1, C25.2, C26.2, C27.1, FTDI/UART.6, LMP1.GND, R15.1, REFSEL.3; no longer UART.6
- net N$2: now also C27.2
- net N$3: now also R11.1, SC2.2; no longer C22.1, UART.1
- net POWERIN: now also JP3.1; no longer JP1.2
- net RESET: now also C17.2; no longer C22.2, OK3.OUT
- net RX-ISO: now also R12.2
Other:
- note added: "Daniel Bates Dec 2016"
- note added: "Shunt Amplifier 1"
- note added: "Shunt Amplifier 2"
- note added: "emonDC v0.3 OpenEnergyMonitor.org"
- note removed: "Daniel Bates Dec 2015"
- note removed: "Shunt Amplifier"
- note removed: "emonDC v0.1 OpenEnergyMonitor.org"
- moved on the sheet: C5, OK3

Commit message: commit
Other:
- moved on the sheet: C48
Changed lines of the file:
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@@
 <setting verticaltext="up"/>
 </settings>
-<grid distance="0.01" unitdist="inch" unit="inch" style="lines" multiple="1" display="yes" altdistance="0.01" altunitdist="inch" altunit="inch"/>
+<grid distance="0.1" unitdist="inch" unit="inch" style="lines" multiple="1" display="no" altdistance="0.01" altunitdist="inch" altunit="inch"/>
 <layers>
 <layer number="1" name="Top" color="4" fill="1" visible="no" active="no"/>
@@
 <attribute name="OC_FARNELL" value="1593411"/>
 </part>
-<part name="SC1" library="SparkFun" deviceset="SOLDERJUMPER" device="NO"/>
+<part name="SC1" library="SparkFun" deviceset="SOLDERJUMPER" device="NO" value=""/>
 <part name="SUPPLY9" library="SparkFun-Aesthetics" deviceset="5V" device=""/>
 <part name="R11" library="rcl" deviceset="R-EU_" device="R0603" value="1K"/>
-<part name="SC2" library="SparkFun" deviceset="SOLDERJUMPER" device="NO"/>
+<part name="SC2" library="SparkFun" deviceset="SOLDERJUMPER" device="NO" value=""/>
 </parts>
 <sheets>
@@
 <wire x1="38.1" y1="495.3" x2="-12.7" y2="495.3" width="0.1524" layer="94"/>
 <wire x1="38.1" y1="495.3" x2="38.1" y2="393.7" width="0.1524" layer="94"/>
+<wire x1="236.22" y1="276.86" x2="236.22" y2="213.36" width="1.778" layer="95" style="shortdash"/>
 </plain>
 <instances>
@@
 <attribute name="MPN" x="-17.78" y="241.935" size="1.778" layer="96" display="off"/>
 </instance>
-<instance part="C48" gate="G$1" x="22.86" y="246.38"/>
+<instance part="C48" gate="G$1" x="17.78" y="246.38"/>
 <instance part="C51" gate="G$1" x="-78.74" y="248.92"/>
 <instance part="GND23" gate="1" x="107.95" y="228.6"/>
@@
 <junction x="-17.78" y="233.68"/>
 <pinref part="C48" gate="G$1" pin="2"/>
-<wire x1="22.86" y1="241.3" x2="22.86" y2="233.68" width="0.1524" layer="91"/>
+<wire x1="17.78" y1="241.3" x2="22.86" y2="233.68" width="0.1524" layer="91"/>
 <junction x="22.86" y="233.68"/>
 <wire x1="-7.62" y1="238.76" x2="-7.62" y2="233.68" width="0.1524" layer="91"/>
@@
 <pinref part="C48" gate="G$1" pin="1"/>
 <wire x1="25.4" y1="259.08" x2="22.86" y2="259.08" width="0.1524" layer="91"/>
-<wire x1="22.86" y1="259.08" x2="22.86" y2="248.92" width="0.1524" layer="91"/>
+<wire x1="22.86" y1="259.08" x2="17.78" y2="248.92" width="0.1524" layer="91"/>
 <wire x1="13.97" y1="259.08" x2="22.86" y2="259.08" width="0.1524" layer="91"/>
 <junction x="13.97" y="259.08"/>
