File: emonDCduo/emonDCduo-ESP v1.0.sch (EAGLE design)
At the start: 86 parts, among them Q1 16Mhz XT49M-2016M, U1_TQFP ATMEGA328P

Commit message: update
chip select set to GPIO4 for both mini and duo.
mini updated, various minor changes for v0.5.
molex micro sd card library improved
Parts:
- removed IO2: (no value), SparkFun:M02PTH
- removed REF_SELECT_A: 2212S-02SG-85, SparkFun-Connectors:CONN_03
- added GPIO2: LSP11, solpad:LSP11
- added REF_SEL: 2212S-02SG-85, SparkFun-Connectors:CONN_03
- renumbered C51 to C17
Connections:
- net GND: now also REF_SEL.3; no longer IO2.1, REF_SELECT_A.3
- net GPIO2: now also GPIO2.MP; no longer CD1.2
- net GPIO5: now also CD1.2; no longer IO2.2
- net N$11: now also REF_SEL.2; no longer REF_SELECT_A.2
- net REFINPUT: now also REF_SEL.1; no longer REF_SELECT_A.1
Other:
- moved on the sheet: C12, C15, C23, C24, C25, C26, C6, C9, J1, J2, J3, J4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

Commit message: commit
Parts:
- REG1117: device burr-brown:REG1117 -> burr-brown:REG1117-VOUT4
Connections:
- net GPIO15: now also U$2.CD/DAT3
- net GPIO4: now also CD1.2; no longer U$2.CD/DAT3
- net GPIO5: no longer CD1.2
Other:
- moved on the sheet: REG1117

Commit message: commit
Parts:
- SHUNTMON-A, SHUNTMON-B: device lmp8481b:LMP8481LMP8481-H -> lmp8481b:LMP8481-H
Changed lines of the file:
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@@
 <part name="SUPPLY3" library="supply2" deviceset="GND" device=""/>
 <part name="AGND11" library="supply1" deviceset="AGND" device=""/>
-<part name="SHUNTMON-B" library="lmp8481b" deviceset="LMP8481" device="LMP8481-H" value="LMP8481">
+<part name="SHUNTMON-B" library="lmp8481b" deviceset="LMP8481" device="-H" value="LMP8481">
 <attribute name="MF" value="TEXAS INSTRUMENTS"/>
 <attribute name="MPN" value="LMP8481MME-H/NOPB"/>
@@
 <part name="GND11" library="supply1" deviceset="GND" device=""/>
 <part name="T1" library="con-weidmueller-sl35" deviceset="180-2" device=""/>
-<part name="SHUNTMON-A" library="lmp8481b" deviceset="LMP8481" device="LMP8481-H" value="LMP8481">
+<part name="SHUNTMON-A" library="lmp8481b" deviceset="LMP8481" device="-H" value="LMP8481">
 <attribute name="MF" value="TEXAS INSTRUMENTS"/>
 <attribute name="MPN" value="LMP8481MME-S/NOPB"/>

Commit message: v1.0 duo camexport and prototype
Parts:
- removed C12, C15: 100nF, rcl:C-EUC0603
- removed R8: 3.9K, rcl:R-EU_R0603
- removed REF_GND: (no value), jumper:SJ
- added R11: 30K, rcl:R-EU_R0603
- added R9: 10K, rcl:R-EU_R0603
- added REF_SEL_B: 2212S-02SG-85, SparkFun-Connectors:CONN_03
- renumbered REF_SEL to REF_SEL_A
Connections:
- net N$11 renamed REF_A_INPUT
- removed net REFINPUT: C12.1, C15.1, R8.1, REF_GND.1, REF_SEL_A.1, SHUNTMON-A.REFA, SHUNTMON-A.REFB
- new net REF_B_INPUT: REF_SEL_B.2, SHUNTMON-A.REFA, SHUNTMON-A.REFB
- new net REF_INPUT: R11.2, R9.1, REF_SEL_A.1, REF_SEL_B.3
- net 4.7V: now also R9.2
- net D5/PWM0: no longer R8.2
- net GND: now also R11.1, REF_SEL_B.1; no longer C12.2, C15.2, REF_GND.2
