File: emonDCduo/emonDCduo-ESP v1.1c.brd (EAGLE design)
At the start: 99.1 x 76.5 mm, 68 parts, among them Y1 32Khz

Commit message: commit v1.3c
Parts:
- added ADC-PAD: (no value), wirepad:2,15/1,0
- SV1: device con-lstb:MA04-1 -> con-lstb:MA03-1
- moved R16 11.0 mm to (34.8, 16.4), turned to 90 degrees
- moved R12 10.1 mm to (31.7, 18.1), turned to 90 degrees
- moved Y1 1.98 mm to (82.9, 11.7)
- moved SCREW1 1.02 mm to (22.9, 53.6)
- moved SCREW2 1.02 mm to (22.9, 39.6)
- moved REF_SEL_A 0.51 mm to (33.9, 60.7)
Connections:
- removed net N$1: MCP3208.5, SV1.1
- net ADC: now also ADC-PAD.1
- net N$3: now also SV1.1; no longer SV1.2
- net N$5: now also SV1.2; no longer SV1.3
- net N$9: now also SV1.3; no longer SV1.4
- net REF_INPUT: now also MCP3208.5
Routing:
- net REF_INPUT: track 27.4 -> 61.8 mm, vias 1 -> 3
- net N$1: track 19.0 -> 0.00 mm
- net ADC: track 0.00 -> 12.3 mm
- net GPIO2: track 29.0 -> 17.8 mm, vias 2 -> 0
- net GPIO13: track 114.9 -> 122.5 mm
- net SDA: track 44.6 -> 51.2 mm
- net SCL: track 42.1 -> 48.3 mm
- net +5V: track 103.1 -> 108.3 mm
- net N$44: track 10.1 -> 8.03 mm
- net N$45: track 5.89 -> 4.00 mm
- net GPIO14: track 103.5 -> 102.3 mm
- net N$30: track 27.8 -> 26.6 mm
- net 3.3V-ESP: track 113.8 -> 114.6 mm
- net N$3: track 16.3 -> 16.9 mm
- net N$5: track 13.7 -> 14.2 mm
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Other:
- board text added: "+"
- board text added: "-"
- board text added: "CRYSTAL 8x3.8mm 32KHz"
- board text added: "LOAD"
- board text added: "RF MODULE"
- board text added: "SOURCE"
- board text added: "adc channels 6, 7, 8"
- board text removed: "RFM MODULE"
- board text removed: "adc channels 5-8"

Commit message: commit v1.3c update
Parts:
- removed SV1: (no value), con-lstb:MA03-1
- added B1: (no value), SparkFun:1X02
- added C2: 100nF, rcl:C0603
- added FTDI2: FTDI, JeeLabs:MA06-1
- added J5: 455-1750-1-ND, SparkFun-Connectors:1X03
- added P1: B6B-PH-K, jst-ph:B6B-PH-K
- added R20: 10K, rcl:R0603
- added S1: SWS002, smd-special:SMS-002
- D2: value BAT60J -> BAT60AE6327HTSA1
- J1, J2, J3, J4, PWR: value (none) -> 455-1750-1-ND
- REF_SEL_A, REF_SEL_B: value 2212S-02SG-85 -> 455-1750-1-ND
- moved R16 4.65 mm to (38.4, 19.3), turned to 180 degrees
- moved CR1220 3.81 mm to (88.1, 21.3)
- moved Y1 2.38 mm to (84.0, 9.51), turned to 0 degrees
- moved D1 2.09 mm to (49.3, 61.9)
- moved C1 1.80 mm to (74.5, 72.2)
- moved C18 1.80 mm to (85.4, 69.7)
- moved C13 1.80 mm to (85.4, 66.2)
- moved REG1117 1.80 mm to (79.8, 70.1)
- moved D2 1.78 mm to (74.6, 65.6)
- moved R12 1.71 mm to (32.5, 19.6), turned to 180 degrees
- moved PCF8523 1.55 mm to (76.2, 16.3)
- moved REF_SEL_A 1.27 mm to (35.2, 60.7)
- moved C17 1.05 mm to (45.2, 62.1)
- moved C16 0.80 mm to (42.9, 62.1)
- moved C7 0.76 mm to (73.3, 10.8)
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Connections:
- new net ESPRX: ESP-12.7, R17.2, R18.1, S1.4
- new net ESPTX: ESP-12.8, FTDI1.2, S1.3
- new net N$20: FTDI2.5
- new net N$301: C2.2, FTDI2.1
- net +5V: now also B1.1
- net 4.7V: now also B1.2, FTDI2.4, P1.6
- net D0/RX: now also FTDI2.2, S1.2; no longer ESP-12.8, FTDI1.2
- net D1/TX: now also FTDI2.3, S1.1; no longer ESP-12.7, R17.2, R18.1
- net GND: now also FTDI2.6, P1.1, R20.1
- net GPIO12: now also P1.3
- net GPIO13: now also P1.4
- net GPIO14: now also P1.5
- net GPIO16: now also P1.2, R20.2
- net N$3: now also J5.3; no longer SV1.1
- net N$5: now also J5.2; no longer SV1.2
- net N$9: now also J5.1; no longer SV1.3
- net _RESET: now also C2.1
Routing:
- net 4.7V: track 142.9 -> 190.0 mm
- net ESPTX: track 0.00 -> 33.3 mm, vias 0 -> 1
- net D1/TX: track 76.5 -> 102.5 mm, vias 2 -> 3
- net D0/RX: track 77.6 -> 100.4 mm
- net _RESET: track 0.00 -> 15.3 mm, vias 0 -> 1
- net ESPRX: track 0.00 -> 12.2 mm
- net GPIO13: track 122.5 -> 133.9 mm, vias 4 -> 5
- net GPIO16: track 4.86 -> 16.0 mm
- net N$301: track 0.00 -> 9.85 mm
- net N$2: track 6.33 -> 0.00 mm
- net N$45: track 4.00 -> 8.86 mm
- net GPIO12: track 72.1 -> 76.9 mm
- net 3.3V: track 64.4 -> 69.1 mm
- net +5V: track 108.3 -> 112.6 mm
- net GPIO14: track 102.3 -> 106.6 mm
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Other:
- board text added: "12"
- board text added: "13"
- board text added: "14"
- board text added: "16"
- board text added: "J1"
- board text added: "LCD"
- board text added: "PWR"
- board text added: "RF to ESP (dis)connect"
- board text added: "RFM69Pi RF MODULE"
- board text added: "TX / RX"
- board text added: "disconnect module before FTDI flash"
- board text removed: "FACTORY RESET"
- board text removed: "RF MODULE"
- board text removed: "disconnect RF module before flash"
