File: emonDCduo/emonDCduo-ESP v1.1c.sch (EAGLE design)
At the start: 68 parts, among them Y1 32Khz

Commit message: commit v1.3c
Parts:
- added ADC-PAD: (no value), wirepad:2,15/1,0
- SV1: device con-lstb:MA04-1 -> con-lstb:MA03-1
Connections:
- removed net N$1: MCP3208.CH4, SV1.1
- net ADC: now also ADC-PAD.P
- net N$3: now also SV1.1; no longer SV1.2
- net N$5: now also SV1.2; no longer SV1.3
- net N$9: now also SV1.3; no longer SV1.4
- net REF_INPUT: now also MCP3208.CH4
Changed lines of the file:
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@@
 <part name="SUPPLY3" library="supply1" deviceset="GND" device=""/>
 <part name="SUPPLY6" library="supply1" deviceset="GND" device=""/>
-<part name="SV1" library="con-lstb" library_urn="urn:adsk.eagle:library:162" deviceset="MA04-1" device="" package3d_urn="urn:adsk.eagle:package:8337/1"/>
+<part name="SV1" library="con-lstb" library_urn="urn:adsk.eagle:library:162" deviceset="MA03-1" device="" package3d_urn="urn:adsk.eagle:package:8339/1"/>
 <part name="R4" library="rcl" deviceset="R-EU_" device="R0603" value="1K">
 <attribute name="MPN" value=" MCWR06X5901FTL"/>
@@
 <part name="R12" library="rcl" library_urn="urn:adsk.eagle:library:334" deviceset="R-EU_" device="R0603" package3d_urn="urn:adsk.eagle:package:23555/2" value="5.6K"/>
 <part name="R16" library="rcl" library_urn="urn:adsk.eagle:library:334" deviceset="R-EU_" device="R0603" package3d_urn="urn:adsk.eagle:package:23555/2" value="10K"/>
+<part name="ADC-PAD" library="wirepad" library_urn="urn:adsk.eagle:library:412" deviceset="2,15/1,0" device="" package3d_urn="urn:adsk.eagle:package:30831/1"/>
 </parts>
 <sheets>
@@
 <instance part="SUPPLY3" gate="1" x="106.68" y="378.46" rot="R180"/>
 <instance part="SUPPLY6" gate="1" x="111.76" y="373.38" rot="R180"/>
-<instance part="SV1" gate="1" x="71.12" y="337.82" rot="R180"/>
+<instance part="SV1" gate="G$1" x="71.12" y="337.82" rot="R180"/>
 <instance part="R4" gate="G$1" x="152.4" y="355.6" rot="R90">
 <attribute name="MPN" x="152.4" y="355.6" size="1.778" layer="96" rot="R90" display="off"/>
@@
 <instance part="R12" gate="G$1" x="55.88" y="472.44" rot="R90"/>
 <instance part="R16" gate="G$1" x="50.8" y="464.82"/>
+<instance part="ADC-PAD" gate="1" x="134.62" y="426.72" rot="R180"/>
 </instances>
 <busses>
@@
 <label x="-24.638" y="371.856" size="1.778" layer="95"/>
 </segment>
+<segment>
+<pinref part="MCP3208" gate="G$1" pin="CH4"/>
+<wire x1="91.44" y1="347.98" x2="60.96" y2="347.98" width="0.1524" layer="91"/>
+</segment>
 </net>
 <net name="IND" class="0">
@@
 <segment>
 <pinref part="ESP-12" gate="G$1" pin="ADC"/>
-<wire x1="109.22" y1="441.96" x2="114.3" y2="441.96" width="0.1524" layer="91"/>
 <label x="111.76" y="441.96" size="1.778" layer="95"/>
+<wire x1="109.22" y1="441.96" x2="124.46" y2="441.96" width="0.1524" layer="91"/>
+<wire x1="124.46" y1="441.96" x2="124.46" y2="426.72" width="0.1524" layer="91"/>
+<pinref part="ADC-PAD" gate="1" pin="P"/>
+<wire x1="124.46" y1="426.72" x2="132.08" y2="426.72" width="0.1524" layer="91"/>
 </segment>
 </net>
@@
 </segment>
 </net>
-<net name="N$1" class="0">
-<segment>
-<pinref part="MCP3208" gate="G$1" pin="CH4"/>
-<pinref part="SV1" gate="1" pin="1"/>
-<wire x1="91.44" y1="347.98" x2="68.58" y2="347.98" width="0.1524" layer="91"/>
-<wire x1="68.58" y1="347.98" x2="63.5" y2="342.9" width="0.1524" layer="91"/>
-</segment>
-</net>
 <net name="N$3" class="0">
 <segment>
 <pinref part="MCP3208" gate="G$1" pin="CH5"/>
-<pinref part="SV1" gate="1" pin="2"/>
+<pinref part="SV1" gate="G$1" pin="1"/>
 <wire x1="91.44" y1="345.44" x2="68.58" y2="345.44" width="0.1524" layer="91"/>
 <wire x1="68.58" y1="345.44" x2="63.5" y2="340.36" width="0.1524" layer="91"/>
@@
 <segment>
 <pinref part="MCP3208" gate="G$1" pin="CH6"/>
-<pinref part="SV1" gate="1" pin="3"/>
+<pinref part="SV1" gate="G$1" pin="2"/>
 <wire x1="91.44" y1="342.9" x2="68.58" y2="342.9" width="0.1524" layer="91"/>
 <wire x1="68.58" y1="342.9" x2="63.5" y2="337.82" width="0.1524" layer="91"/>
@@
 <segment>
 <pinref part="MCP3208" gate="G$1" pin="CH7"/>
-<pinref part="SV1" gate="1" pin="4"/>
+<pinref part="SV1" gate="G$1" pin="3"/>
 <wire x1="91.44" y1="340.36" x2="68.58" y2="340.36" width="0.1524" layer="91"/>
 <wire x1="68.58" y1="340.36" x2="63.5" y2="335.28" width="0.1524" layer="91"/>

Commit message: commit v1.3c update
Parts:
- removed SV1: (no value), con-lstb:MA03-1
- added B1: (no value), SparkFun:M02PTH
- added C2: 100nF, rcl:C-EUC0603
- added FTDI2: FTDI, JeeLabs:MA06-1
- added J5: 455-1750-1-ND, SparkFun-Connectors:CONN_03
- added P1: B6B-PH-K, jst-ph:B6B-PH-K
- added R20: 10K, rcl:R-EU_R0603
- added S1: SWS002, smd-special:SWS002
- D2: value BAT60J -> BAT60AE6327HTSA1
- J1, J2, J3, J4, PWR: value (none) -> 455-1750-1-ND
- REF_SEL_A, REF_SEL_B: value 2212S-02SG-85 -> 455-1750-1-ND
Connections:
- new net ESPRX: ESP-12.RXD, R17.2, R18.1, S1.4
- new net ESPTX: ESP-12.TXD, FTDI1.2, S1.3
- new net N$20: FTDI2.5
- new net N$301: C2.2, FTDI2.1
- net +5V: now also B1.1
- net 4.7V: now also B1.2, FTDI2.4, P1.6
- net D0/RX: now also FTDI2.2, S1.2; no longer ESP-12.TXD, FTDI1.2
- net D1/TX: now also FTDI2.3, S1.1; no longer ESP-12.RXD, R17.2, R18.1
- net GND: now also FTDI2.6, P1.1, R20.1
- net GPIO12: now also P1.3
- net GPIO13: now also P1.4
- net GPIO14: now also P1.5
- net GPIO16: now also P1.2, R20.2
- net N$3: now also J5.3; no longer SV1.1
- net N$5: now also J5.2; no longer SV1.2
- net N$9: now also J5.1; no longer SV1.3
- net _RESET: now also C2.1
Other:
- note added: "RFM69Pi Module Interface RFM69CW"
- note added: "SPI LCD DISPLAY"
- note removed: "RFM12B RFM69CW"
