File: emonDCduo/emonDCduo-ESP v1.3.brd (EAGLE design)
At the start: 99.1 x 76.5 mm, 75 parts, among them J1 455-1750-1-ND, J2 455-1750-1-ND, J3 455-1750-1-ND, J4 455-1750-1-ND, J5 455-1750-1-ND, P1 B6B-PH-K, Y1 32Khz

Commit message: commit
Parts:
- removed C17: 0.1uF 100V, rcl:C0603
- removed J1, J2, J3, J4: 455-1750-1-ND, SparkFun-Connectors:1X03
- removed R16, R20: 10K, rcl:R0603
- removed TL2575HV: TL2575HV-5V, TL2575HV:TO-263
- removed U$2: MOLEX_MICRO_SD_1040310811, MOLEX MICRO SD [exposed pins]:MOLEX_MICROSD_EXPOSED
- added C4, C5: 0.1uF MLCC, rcl:C0603
- added U$4: 47219-2001_MICROSD, MOLEX 47219-2001:47219-2001_MICROSD
- added U1: MAX5035, MAX5035:21-0111D_SBE-14
- C10: value 100uF 80V -> 100uF 80V (LOW-ESR)
- J5: device SparkFun-Connectors:1X03 -> SparkFun-Connectors:1X02
- P1: value B6B-PH-K -> B4B-PH-K; device jst-ph:B6B-PH-K -> jst-ph:B4B-PH-K
- R12: value 5.6K -> 10K
- U$1, U$3: value EBW_SERIES_10.5MM -> EBW_SERIES_15.2MM; device EBW series shunt:EBW_SERIES_10.5MM -> EBW series shunt:EBW_SERIES_15.2MM
- moved CR1220 67.0 mm to (21.6, 13.7), turned to 90 degrees
- moved Y1 50.9 mm to (33.7, 17.1)
- moved PCF8523 44.5 mm to (32.0, 21.1)
- moved P1 38.3 mm to (34.3, 26.2)
- moved R9 38.2 mm to (38.8, 16.1)
- moved C7 35.3 mm to (38.2, 14.6)
- moved C22 25.7 mm to (88.6, 24.6)
- moved C21 25.0 mm to (88.9, 19.6)
- moved ESP-12 22.6 mm to (84.8, 26.2)
- moved MC2 20.6 mm to (60.3, 30.5)
- moved IO1 19.4 mm to (86.1, 22.7)
- moved R7 19.1 mm to (83.1, 22.1)
- moved FTDI1 16.8 mm to (77.2, 28.7)
- moved R19 16.1 mm to (85.3, 17.0)
- moved R12 15.7 mm to (43.0, 31.4), turned to 0 degrees
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Connections:
- net N$5 renamed CH6
- net N$9 renamed CH7
- new net N$1: C5.1, U1.2
- new net N$5: C4.2, U1.8
- net +5V: no longer R12.2, TL2575HV.4
- net 3.3V: now also MCP3208.6, P1.3
- net 3.3V-ESP: now also R12.2, U$4.PIN4; no longer U$2.P$4
- net 4.7V: no longer P1.6
- net ADCSHUNT-A: now also MCP3208.1, R13.2; no longer MCP3208.3, R5.2
- net ADCSHUNT-B: now also MCP3208.3, R5.2; no longer MCP3208.1, R13.2
- net GND: now also C5.2, P1.4, U$4.P$1, U$4.P$2, U$4.P$3, U$4.P$4, U$4.PIN6, U1.3, U1.6; no longer C17.2, P1.1, R16.1, R20.1, TL2575HV.3, TL2575HV.5, TL2575HV.6, U$2.GND1, U$2.GND2, U$2.GND3, U$2.GND4, U$2.P$6
- net GPIO0: now also R12.1
- net GPIO12: now also U$4.PIN7; no longer P1.3, U$2.P$7
- net GPIO13: now also U$4.PIN3; no longer P1.4, U$2.P$3
- net GPIO14: now also U$4.PIN5; no longer P1.5, U$2.P$5
- net GPIO15: now also U$4.PIN2; no longer U$2.P$2
- net GPIO16: no longer P1.2, R20.2
- net GPIO2: no longer R12.1, R16.2
- net IND: no longer TL2575HV.2
- net LOAD-NEG-A: no longer J1.1, J1.2, J1.3
- net LOAD-NEG-B: no longer J4.1, J4.2, J4.3
- net N$3: now also C4.1, U1.1; no longer J5.3, MCP3208.6
- net N$32: now also U$4.PIN8; no longer U$2.P$8
- net N$7: now also U$4.PIN1; no longer U$2.P$1
- net PWR_IN: now also U1.5, U1.7; no longer C17.1, TL2575HV.1
- net SCL: now also P1.2
- net SDA: now also P1.1
- net SOURCE-POS-A: no longer J2.1, J2.2, J2.3
- net SOURCE-POS-B: no longer J3.1, J3.2, J3.3
- net VSENSEA: now also MCP3208.2, R14.1, R15.2; no longer MCP3208.4, R1.1, R2.2
- net VSENSEB: now also MCP3208.4, R1.1, R2.2; no longer MCP3208.2, R14.1, R15.2
Routing:
- net GPIO13: track 133.9 -> 0.00 mm, vias 5 -> 0
- net 3.3V-ESP: track 114.4 -> 0.00 mm, vias 1 -> 0
- net GPIO14: track 106.6 -> 0.00 mm, vias 2 -> 0
- net D0/RX: track 100.4 -> 0.00 mm, vias 2 -> 0
- net 4.7V: track 190.0 -> 98.6 mm, vias 5 -> 3
- net D1/TX: track 102.5 -> 21.6 mm, vias 3 -> 1
- net GPIO12: track 76.9 -> 0.00 mm, vias 2 -> 0
- net 3.3V: track 69.1 -> 3.62 mm, vias 2 -> 0
- net SDA: track 52.2 -> 0.00 mm, vias 2 -> 0
- net GPIO15: track 49.7 -> 0.00 mm, vias 2 -> 0
- net SCL: track 48.4 -> 0.00 mm, vias 2 -> 0
- net ESPTX: track 33.3 -> 0.00 mm, vias 1 -> 0
- net GPIO0: track 28.1 -> 0.00 mm
- net N$30: track 26.4 -> 0.00 mm, vias 1 -> 0
- net GPIO12A: track 26.0 -> 0.02 mm, vias 2 -> 0
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Other:
- board text added: "CH6 CH7 ADC"
- board text added: "I2C"
- board text added: "LMP8481"
- board text added: "v1.2 Dec 2017 by DB"
- board text removed: "12"
- board text removed: "13"
- board text removed: "14"
- board text removed: "16"
- board text removed: "LMP"
- board text removed: "PWR"
- board text removed: "adc channels 6, 7, 8"
- board text removed: "v1.1 Dec 2017 by DB"

Commit message: commit
Parts:
- removed I1: 330uH, SRR0603-331KL:SRR0603-331KL
- added L1: SRR1208, inductor-bourns:SSR1208
- C48: value 100nF -> 0.1uF MLCC
- D1: value MBRA130LT3G -> MBRS1100T3G; device CASE 403D Diode:DO-214 -> diodes:SMB_1
- moved D1 119.8 mm to (-2.11, -46.2), turned to 0 degrees
Connections:
- removed net IND: D1.P$1, I1.P$1
- net +5V: now also L1.2, U1.4; no longer I1.P$2
- net GND: now also D1.A; no longer D1.P$2
- net N$5: now also D1.C, L1.1
Routing:
- net +5V: track 109.0 -> 99.0 mm
- net IND: track 7.58 -> 0.00 mm
Changed lines of the file:
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@@
 <attribute name="NAME" x="38.039325" y="40.55670625" size="1.016" layer="25" font="vector"/>
 </element>
-<element name="D1" library="CASE 403D Diode" package="DO-214" value="MBRA130LT3G" x="49.348221875" y="61.9364" rot="R270">
-<attribute name="MF" value="ON SEMICONDUCTOR" x="49.348221875" y="61.9364" size="1.778" layer="27" rot="R270" display="off"/>
-<attribute name="MPN" value="MBRA130LT3G" x="49.348221875" y="61.9364" size="1.778" layer="27" rot="R270" display="off"/>
-<attribute name="OC_FARNELL" value="9555978" x="49.348221875" y="61.9364" size="1.778" layer="27" rot="R270" display="off"/>
-</element>
-<element name="C48" library="rcl" package="C0603" value="100nF" x="50.241" y="75.3888" smashed="yes">
+<element name="C48" library="rcl" package="C0603" value="0.1uF MLCC" x="50.241" y="75.3888" smashed="yes">
 <attribute name="NAME" x="48.84839375" y="76.267609375" size="1.016" layer="25" font="vector"/>
 </element>
@@
 <attribute name="OC_FARNELL" value="1097566" x="150.335" y="147.604" size="1.778" layer="27" rot="R180" display="off"/>
 <attribute name="OC_NEWARK" value="14P6981" x="150.335" y="147.604" size="1.778" layer="27" rot="R180" display="off"/>
-</element>
-<element name="I1" library="SRR0603-331KL" package="SRR0603-331KL" value="330uH" x="54.5336" y="69.9396" smashed="yes" rot="SR0">
-<attribute name="INDUCTANCE" value="330uH" x="54.5336" y="69.9396" size="1.778" layer="27" rot="SR0" display="off"/>
-<attribute name="MF" value="BOURNS" x="54.5336" y="69.9396" size="1.778" layer="27" rot="SR0" display="off"/>
-<attribute name="MPN" value="SRR0603-331KL" x="54.5336" y="69.9396" size="1.778" layer="27" rot="SR0" display="off"/>
-<attribute name="OC_FARNELL" value="2333890" x="54.5336" y="69.9396" size="1.778" layer="27" rot="SR0" display="off"/>
 </element>
 <element name="D2" library="diode" library_urn="urn:adsk.eagle:library:210" package="SOD323_ST" package3d_urn="urn:adsk.eagle:package:43461/1" value="BAT60AE6327HTSA1" x="74.566" y="65.6258" smashed="yes" rot="R180">
@@
 <element name="C4" library="rcl" package="C0603" value="0.1uF MLCC" x="-5.842" y="-22.86"/>
 <element name="C5" library="rcl" package="C0603" value="0.1uF MLCC" x="-5.842" y="-27.94"/>
+<element name="D1" library="diodes" package="SMB_1" value="MBRS1100T3G" x="-2.11" y="-46.228"/>
+<element name="L1" library="inductor-bourns" package="SSR1208" value="SRR1208" x="3.048" y="-57.658">
+<attribute name="MPN" value="SRR1208-151YL" x="3.048" y="-57.658" size="1.778" layer="27" display="off"/>
+</element>
 </elements>
 <signals>
@@
 <contactref element="C13" pad="2"/>
 <contactref element="REG1117" pad="1"/>
-<contactref element="D1" pad="P$2"/>
 <contactref element="C48" pad="2"/>
 <contactref element="C3" pad="2"/>
@@
 <contactref element="C16" pad="2"/>
 <contactref element="C10" pad="2"/>
+<contactref element="D1" pad="A"/>
 <wire x1="86.200121875" y1="69.671171875" x2="92.326296875" y2="69.00523125" width="0" layer="19" extent="1-1"/>
 <wire x1="86.25708125" y1="66.159571875" x2="86.200121875" y2="69.671171875" width="0" layer="19" extent="1-1"/>
@@
 <wire x1="54.262" y1="60.96" x2="59.512" y2="59.66" width="0" layer="19" extent="1-1"/>
 <wire x1="49.34828125" y1="61.7980375" x2="54.262" y2="60.96" width="0" layer="19" extent="1-1"/>
-<wire x1="49.348221875" y1="59.9364" x2="49.34828125" y2="61.7980375" width="0" layer="19" extent="1-1"/>
-<wire x1="47.0885125" y1="60.01310625" x2="49.348221875" y2="59.9364" width="0" layer="19" extent="1-1"/>
+<wire x1="47.0885125" y1="60.01310625" x2="49.34828125" y2="61.7980375" width="0" layer="19" extent="1-1"/>
 <wire x1="44.0915" y1="59.981271875" x2="47.0885125" y2="60.01310625" width="0" layer="19" extent="1-1"/>
 <wire x1="42.91565" y1="61.228715625" x2="44.0915" y2="59.981271875" width="0" layer="19" extent="1-1"/>
@@
 <wire x1="-5.9563" y1="-18.415" x2="-0.6477" y2="-18.415" width="0" layer="19" extent="1-1"/>
 <wire x1="-4.992" y1="-27.94" x2="-5.9563" y2="-18.415" width="0" layer="19" extent="1-1"/>
+<wire x1="0" y1="-46.228" x2="-4.992" y2="-27.94" width="0" layer="19" extent="1-1"/>
 </signal>
 <signal name="3.3V">
@@
 <wire x1="50.21" y1="46.736" x2="50.546" y2="44.958" width="0.254" layer="1"/>
 <wire x1="49.022" y1="48.178" x2="50.21" y2="46.736" width="0.254" layer="1"/>
-</signal>
-<signal name="IND">
-<contactref element="D1" pad="P$1"/>
-<contactref element="I1" pad="P$1"/>
-<wire x1="49.8812" y1="69.814" x2="51.5336" y2="69.9396" width="1.016" layer="1"/>
-<wire x1="49.8812" y1="69.814" x2="49.8812" y2="66.8822" width="1.016" layer="1"/>
-<wire x1="49.8812" y1="66.8822" x2="49.348221875" y2="63.9364" width="1.016" layer="1"/>
 </signal>
 <signal name="4.7V" class="1">
@@
 </signal>
 <signal name="+5V">
-<contactref element="I1" pad="P$2"/>
 <contactref element="D2" pad="A"/>
 <contactref element="C48" pad="1"/>
-<contactref element="C3" pad="1"/>
 <wire x1="71.882" y1="65.6258" x2="56.0096" y2="65.6258" width="0.6096" layer="1"/>
 <wire x1="71.882" y1="65.6258" x2="73.316" y2="65.6258" width="0.6096" layer="1"/>
 <wire x1="49.391" y1="73.2176" x2="49.391" y2="75.3888" width="1.016" layer="1"/>
-<wire x1="57.5336" y1="69.9396" x2="56.0096" y2="73.2176" width="1.016" layer="1"/>
 <wire x1="56.0096" y1="73.2176" x2="49.391" y2="73.2176" width="1.016" layer="1"/>
 <via x="58.674" y="76.2" extent="1-16" drill="1.1" shape="square"/>
 <wire x1="58.674" y1="76.2" x2="58.674" y2="73.2176" width="1.016" layer="1"/>
 <wire x1="58.674" y1="73.2176" x2="56.0096" y2="73.2176" width="1.016" layer="1"/>
-<wire x1="56.0096" y1="65.6258" x2="57.5336" y2="69.9396" width="0.6096" layer="1"/>
-<wire x1="61.5188" y1="69.9516" x2="55.7556" y2="69.9516" width="1.016" layer="1"/>
-<wire x1="55.7556" y1="69.9516" x2="57.5336" y2="69.9396" width="1.016" layer="1"/>
 <wire x1="44.704" y1="46.482" x2="34.036" y2="35.814" width="0.254" layer="16"/>
 <wire x1="44.704" y1="46.482" x2="49.784" y2="46.482" width="0.254" layer="16"/>
@@
 <wire x1="34.036" y1="22.804246875" x2="32.337765625" y2="21.1060125" width="0.254" layer="16"/>
 <wire x1="34.036" y1="35.814" x2="34.036" y2="22.804246875" width="0.254" layer="16"/>
+<contactref element="C3" pad="1"/>
+<contactref element="L1" pad="2"/>
+<contactref element="U1" pad="4"/>
+<wire x1="61.5188" y1="69.9516" x2="55.7556" y2="69.9516" width="1.016" layer="1"/>
+<wire x1="56.0096" y1="73.2176" x2="55.7556" y2="69.9516" width="0" layer="19" extent="1-1"/>
+<wire x1="55.9764" y1="65.659" x2="55.7556" y2="69.9516" width="0" layer="19" extent="1-1"/>
+<wire x1="-5.9563" y1="-19.685" x2="32.32710625" y2="20.94058125" width="0" layer="19" extent="1-1"/>
+<wire x1="3.048" y1="-62.658" x2="-5.9563" y2="-19.685" width="0" layer="19" extent="1-1"/>
 </signal>
 <signal name="N$20">
@@
 <contactref element="C4" pad="2"/>
 <contactref element="U1" pad="8"/>
+<contactref element="L1" pad="1"/>
+<contactref element="D1" pad="C"/>
+<wire x1="-4.22" y1="-46.228" x2="3.048" y2="-52.658" width="0" layer="19" extent="1-1"/>
+<wire x1="-4.992" y1="-22.86" x2="-4.22" y2="-46.228" width="0" layer="19" extent="1-1"/>
 <wire x1="-0.6477" y1="-15.875" x2="-4.992" y2="-22.86" width="0" layer="19" extent="1-1"/>
 </signal>

Commit message: commit
Parts:
- added C8: 68UF, Panasonic-EEE-EEV-EEF-ECQ:CAPAE1350X1400N
- added U$2: (no value), DRAGON_LOGO:DRAGON_LOGO_NOTEXT
- moved L1 133.2 mm to (51.1, 66.5), turned to 180 degrees
- moved D1 121.7 mm to (42.2, 67.1), turned to 270 degrees
- moved C5 112.7 mm to (43.4, 73.4), turned to 90 degrees
- moved C4 102.3 mm to (37.8, 69.6), turned to 180 degrees
- moved U1 100.1 mm to (38.1, 73.4), turned to 180 degrees
- moved C16 9.11 mm to (34.6, 65.7), turned to 90 degrees
- moved MINI_USB-B 6.12 mm to (64.0, 60.5)
Routing:
- net 4.7V: track 98.6 -> 103.6 mm

Commit message: commit
Parts:
- removed B1: (no value), SparkFun:1X02
- removed C1, C18: 10uF TANT, rcl:C0603
- removed C8: 68UF, Panasonic-EEE-EEV-EEF-ECQ:CAPAE1350X1400N
- removed D2: BAT60AE6327HTSA1, diode:SOD323_ST
- removed ESP-PWR: (no value), jumper:SJ
- removed MC2: MC32882, multicomp tact switch:SWITCH_TACT_MULTICOMP
- removed MINI_USB-B: 5000751517_SD, 5000751517_sd:5000751517_SD
- removed REG1117: REG1117-3.3V, burr-brown:SOT223
- removed U$2: (no value), DRAGON_LOGO:DRAGON_LOGO_NOTEXT
- removed U1: MAX5035, MAX5035:21-0111D_SBE-14
- added BOOTL, ESP_PWR: (no value), SparkFun:1X02
- added C11T, C18T, C1T: 10uF TANT, rcl:C0603
- added C14: 0.1uF, rcl:C0603
- added R20: 57.6k, rcl:R0603
- added R21: 13.3k, rcl:R0603
- added REG0: MAX5035, MAX5035:21-0111D_SBE-14
- added REG1: REG1117-5.0V, burr-brown:SOT223
- added REG2: REG1117-3.3V, burr-brown:SOT223
- added USB_PWR: 5000751517_SD, 5000751517_sd:5000751517_SD
- C13: value 100nF -> 0.1uF
- C4, C5: value 0.1uF MLCC -> 0.1uF 16V MLCC
- moved S1 39.6 mm to (61.7, 36.3)
- moved U$4 31.3 mm to (31.8, 5.84), turned to 90 degrees
- moved PCF8523 27.9 mm to (58.4, 12.2)
- moved R12 27.0 mm to (69.6, 36.0), turned to 90 degrees
- moved Y1 24.6 mm to (58.1, 20.7)
- moved PWR 22.6 mm to (37.6, 61.1), turned to 180 degrees
- moved C48 20.6 mm to (69.4, 67.7), turned to 270 degrees
- moved P1 18.8 mm to (53.1, 27.5)
- moved REF_SEL_B 14.1 mm to (42.1, 34.3), turned to 90 degrees
- moved C9 12.6 mm to (30.7, 27.8), turned to 270 degrees
- moved ADC-PAD 10.4 mm to (86.9, 4.32)
- moved R19 10.4 mm to (95.3, 20.1), turned to 0 degrees
- moved REF_SEL_A 10.2 mm to (42.0, 53.2), turned to 90 degrees
- moved C26 9.59 mm to (30.8, 46.4), turned to 270 degrees
- moved R5 9.28 mm to (33.6, 34.9)
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- renumbered U$1 to SCREW_TERM_2, U$3 to SCREW_TERM_1
Connections:
- removed net +5V: B1.1, C3.1, C48.1, D2.A, L1.2, U1.4
- removed net 4.7V: B1.2, C1.1, C26.1, C9.1, D2.C, FTDI1.4, FTDI2.4, MCP3208.16, MINI_USB-B.VBUS, R10.2, REG1117.3, SHUNTMON-A.2, SHUNTMON-B.2
- removed net N$1: C5.1, U1.2
- removed net N$3: C4.1, U1.1
- removed net N$5: C4.2, D1.C, L1.1, U1.8
- removed net PWR_IN: C10.1, C16.1, PWR.2, U1.5, U1.7
- new net 5.0V: C14.1, C1T.1, C26.1, C9.1, FTDI1.4, FTDI2.4, MCP3208.16, R10.2, REG1.2, REG1.4, REG2.3, SHUNTMON-A.2, SHUNTMON-B.2, USB_PWR.VBUS
- new net 6.5V: C11T.1, C3.1, C48.1, L1.2, R20.2, REG1.3
- new net BST: C4.1, REG0.1
- new net FB: R20.1, R21.2, REG0.4
- new net LX: C4.2, D1.C, L1.1, REG0.8
- new net VD: C5.1, REG0.2
- new net V_IN: C10.1, C16.1, PWR.2, REG0.5, REG0.7
- net 3.3V: now also C18T.1, ESP_PWR.2, REG2.2, REG2.4; no longer C18.1, ESP-PWR.2, P1.3, REG1117.2, REG1117.4
- net 3.3V-ESP: now also ESP_PWR.1, P1.3; no longer ESP-PWR.1
- net GND: now also BOOTL.1, C11T.2, C14.2, C18T.2, C1T.2, R21.1, REG0.3, REG0.6, REG1.1, REG2.1, USB_PWR.GND1, USB_PWR.GND2, USB_PWR.GND3; no longer C1.2, C18.2, MC2.P$1, MC2.P$2, MINI_USB-B.GND1, MINI_USB-B.GND2, MINI_USB-B.GND3, REG1117.1, U1.3, U1.6
- net GPIO0: now also BOOTL.2; no longer MC2.P$3, MC2.P$4
Routing:
- net 5.0V: track 0.00 -> 147.1 mm, vias 0 -> 4
- net 4.7V: track 103.6 -> 0.00 mm, vias 3 -> 0
- net +5V: track 99.0 -> 0.00 mm, vias 5 -> 0
- net 3.3V: track 3.62 -> 50.7 mm, vias 0 -> 1
- net PWR_IN: track 46.8 -> 0.00 mm
- net V_IN: track 0.00 -> 40.0 mm
- net FB: track 0.00 -> 26.0 mm
- net 6.5V: track 0.00 -> 26.0 mm
- net LX: track 0.00 -> 17.9 mm
- net ADCSHUNT-B: track 37.0 -> 54.6 mm
- net SOURCE-POS-B: track 87.4 -> 76.4 mm
- net ADCSHUNT-A: track 32.6 -> 42.2 mm, vias 0 -> 2
- net REF_B_INPUT: track 8.74 -> 16.8 mm
- net REF_A_INPUT: track 9.34 -> 17.1 mm
- net LOAD-NEG-B: track 41.6 -> 35.0 mm
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Other:
- board text added: "150uH"
- board text added: "v1.3 Dec 2017 by DB"
- board text removed: "330uH"
- board text removed: "4.7V"
- board text removed: "5.0V"
- board text removed: "BOOT- LOADER MODE"
- board text removed: "D1"
- board text removed: "I1"
- board text removed: "RF to ESP (dis)connect"
- board text removed: "v1.2 Dec 2017 by DB"

Commit message: commit
Parts:
- removed ESP_PWR: (no value), SparkFun:1X02
- removed S1: SWS002, smd-special:SMS-002
- added RX, TX: (no value), SparkFun:1X02
- moved R6 23.3 mm to (65.7, 20.7)
- moved R3 22.7 mm to (65.7, 22.7), turned to 180 degrees
- moved R17 19.9 mm to (65.7, 14.8)
- moved PCF8523 18.9 mm to (41.9, 21.3), turned to 90 degrees
- moved R12 17.9 mm to (65.7, 18.6), turned to 180 degrees
- moved R18 17.1 mm to (65.7, 12.6)
- moved CR1220 16.6 mm to (33.8, 22.4), turned to 180 degrees
- moved Y1 15.7 mm to (62.6, 5.70)
- moved BOOTL 11.2 mm to (62.2, 34.5), turned to 180 degrees
- moved R9 10.9 mm to (41.6, 29.6), turned to 0 degrees
- moved C7 9.90 mm to (40.5, 26.2), turned to 0 degrees
- moved LOGO1 6.18 mm to (22.5, 10.0)
- moved U$4 2.61 mm to (30.0, 3.87)
- moved R4 1.43 mm to (82.4, 43.8), turned to 90 degrees
- moved P1 1.27 mm to (53.9, 28.5)
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Connections:
- removed net 3.3V-ESP: C22.2, ESP-12.16, ESP_PWR.1, IO1.2, P1.3, R12.2, R19.2, R6.2, R7.2, R9.2, U$4.PIN4
- removed net GPIO4: MCP3208.10
- net 3.3V: now also C22.2, ESP-12.16, IO1.2, P1.3, R12.2, R19.2, R6.2, R7.2, R9.2, U$4.PIN4; no longer ESP_PWR.2
- net D0/RX: now also TX.2; no longer S1.2
- net D1/TX: now also RX.1; no longer S1.1
- net ESPRX: now also RX.2; no longer S1.4
- net ESPTX: now also TX.1; no longer S1.3
- net GPIO2: now also MCP3208.10
Routing:
- net 3.3V: track 50.7 -> 198.0 mm, vias 1 -> 7
- net GPIO14: track 0.00 -> 111.1 mm, vias 0 -> 4
- net GPIO13: track 0.00 -> 106.9 mm, vias 0 -> 2
- net GPIO12: track 0.00 -> 105.4 mm, vias 0 -> 6
- net D0/RX: track 0.00 -> 84.0 mm
- net GPIO15: track 0.00 -> 83.0 mm, vias 0 -> 4
- net D1/TX: track 21.6 -> 72.0 mm
- net ESPTX: track 0.00 -> 48.0 mm
- net N$30: track 0.00 -> 47.1 mm, vias 0 -> 2
- net SCL: track 0.00 -> 41.6 mm, vias 0 -> 1
- net GPIO2: track 0.12 -> 39.3 mm, vias 0 -> 2
- net SDA: track 0.00 -> 38.3 mm, vias 0 -> 1
- net GPIO0: track 0.00 -> 26.4 mm, vias 0 -> 1
- net N$45: track 0.00 -> 26.3 mm
- net ESPRX: track 0.00 -> 25.1 mm
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Other:
- board text removed: "J1"
