File: emonDCduo/emonDCduo-ESP v1.3.sch (EAGLE design)
At the start: 75 parts, among them J1 455-1750-1-ND, J2 455-1750-1-ND, J3 455-1750-1-ND, J4 455-1750-1-ND, J5 455-1750-1-ND, P1 B6B-PH-K, Y1 32Khz

Commit message: commit
Parts:
- removed C17: 0.1uF 100V, rcl:C-EUC0603
- removed J1, J2, J3, J4: 455-1750-1-ND, SparkFun-Connectors:CONN_03
- removed R16, R20: 10K, rcl:R-EU_R0603
- removed TL2575HV: TL2575HV-5V, TL2575HV:TL2575HV-05IKTTR
- removed U$2: MOLEX_MICRO_SD_1040310811, MOLEX MICRO SD [exposed pins]:MOLEX_MICRO_SD_1040310811
- added C4, C5: 0.1uF MLCC, rcl:C-EUC0603
- added U$4: 47219-2001_MICROSD, MOLEX 47219-2001:47219-2001_MICROSD
- added U1: MAX5035, MAX5035:MAX5035
- C10: value 100uF 80V -> 100uF 80V (LOW-ESR)
- J5: device SparkFun-Connectors:CONN_03 -> SparkFun-Connectors:CONN_02
- P1: value B6B-PH-K -> B4B-PH-K; device jst-ph:B6B-PH-K -> jst-ph:B4B-PH-K
- R12: value 5.6K -> 10K
- U$1, U$3: value EBW_SERIES_10.5MM -> EBW_SERIES_15.2MM; device EBW series shunt:EBW_SERIES_10.5MM -> EBW series shunt:EBW_SERIES_15.2MM
Connections:
- net N$5 renamed CH6
- net N$9 renamed CH7
- new net N$1: C5.1, U1.VD
- new net N$5: C4.2, U1.LX/OUT
- net +5V: no longer R12.2, TL2575HV.FEEDBACK
- net 3.3V: now also MCP3208.CH5, P1.3
- net 3.3V-ESP: now also R12.2, U$4.VDD; no longer U$2.VDD
- net 4.7V: no longer P1.6
- net ADCSHUNT-A: now also MCP3208.CH0, R13.2; no longer MCP3208.CH2, R5.2
- net ADCSHUNT-B: now also MCP3208.CH2, R5.2; no longer MCP3208.CH0, R13.2
- net GND: now also C5.2, P1.4, U$4.GND, U$4.VSS, U1.GND, U1.SGND; no longer C17.2, P1.1, R16.1, R20.1, TL2575HV.GND, TL2575HV.GND-TAB, TL2575HV.ON/OFF, U$2.GND, U$2.VSS
- net GPIO0: now also R12.1
- net GPIO12: now also U$4.DAT0; no longer P1.3, U$2.DAT0
- net GPIO13: now also U$4.CMD; no longer P1.4, U$2.CMD
- net GPIO14: now also U$4.CLK; no longer P1.5, U$2.CLK
- net GPIO15: now also U$4.CD/DAT3; no longer U$2.CD/DAT3
- net GPIO16: no longer P1.2, R20.2
- net GPIO2: no longer R12.1, R16.2
- net IND: no longer TL2575HV.VOUT
- net LOAD-NEG-A: no longer J1.1, J1.2, J1.3
- net LOAD-NEG-B: no longer J4.1, J4.2, J4.3
- net N$3: now also C4.1, U1.BST; no longer J5.3, MCP3208.CH5
- net N$32: now also U$4.DAT1; no longer U$2.DAT1
- net N$7: now also U$4.DAT2; no longer U$2.DAT2
- net PWR_IN: now also U1.ON/OFF, U1.V_IN; no longer C17.1, TL2575HV.VIN
- net SCL: now also P1.2
- net SDA: now also P1.1
- net SOURCE-POS-A: no longer J2.1, J2.2, J2.3
- net SOURCE-POS-B: no longer J3.1, J3.2, J3.3
- net VSENSEA: now also MCP3208.CH1, R14.1, R15.2; no longer MCP3208.CH3, R1.1, R2.2
- net VSENSEB: now also MCP3208.CH3, R1.1, R2.2; no longer MCP3208.CH1, R14.1, R15.2
Other:
- note added: "Daniel Bates Dec 2017"
- note added: "emonDC v1.3 : based on emonTx v3.4 by Glyn Hudson and Trystan Lea OpenEnergyMonitor.org"
- note removed: "Daniel Bates Nov 2017"
- note removed: "emonDC v1.1 : based on emonTx v3.4 by Glyn Hudson and Trystan Lea OpenEnergyMonitor.org"
- moved on the sheet: C10, C16, R12

Commit message: commit
Parts:
- removed I1: 330uH, SRR0603-331KL:SRR0603-331KL
- added L1: SRR1208, inductor-bourns:SRR1208
- C48: value 100nF -> 0.1uF MLCC
- D1: value MBRA130LT3G -> MBRS1100T3G; device CASE 403D Diode:MBRA130LT3G -> diodes:MBRS1100T3G; MF ON SEMICONDUCTOR -> (none); MPN MBRA130LT3G -> (none); OC_FARNELL 9555978 -> (none)
Connections:
- removed net IND: D1.C, I1.P$1
- net +5V: now also L1.2, U1.FB; no longer I1.P$2
- net N$5: now also D1.C, L1.1
Other:
- note added: "DC INPUT & REGULATORS"
- note removed: "DC INPUT, ELS POWER & VOLTAGE REGULATORS"
- moved on the sheet: C3
Changed lines of the file:
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@@
 <part name="GND7" library="supply1" deviceset="GND" device=""/>
 <part name="R5" library="rcl" deviceset="R-EU_" device="R0603" value="1K"/>
-<part name="D1" library="CASE 403D Diode" deviceset="MBRA130LT3G" device="">
-<attribute name="MF" value="ON SEMICONDUCTOR"/>
-<attribute name="MPN" value="MBRA130LT3G"/>
-<attribute name="OC_FARNELL" value="9555978"/>
-</part>
-<part name="C48" library="rcl" deviceset="C-EU" device="C0603" value="100nF"/>
+<part name="C48" library="rcl" deviceset="C-EU" device="C0603" value="0.1uF MLCC"/>
 <part name="GND23" library="supply1" deviceset="0V" device="" value="GND"/>
 <part name="C13" library="rcl" deviceset="C-EU" device="C0603" value="100nF"/>
@@
 </part>
 <part name="SUPPLY4" library="SparkFun-Aesthetics" deviceset="3.3V" device=""/>
-<part name="I1" library="SRR0603-331KL" deviceset="SRR0603-331KL" device="" value="330uH">
-<attribute name="MF" value="BOURNS"/>
-<attribute name="MPN" value="SRR0603-331KL"/>
-<attribute name="OC_FARNELL" value="2333890"/>
-</part>
 <part name="SUPPLY5" library="SparkFun-Aesthetics" deviceset="5V" device=""/>
 <part name="D2" library="diode" library_urn="urn:adsk.eagle:library:210" deviceset="BAT60J" device="" package3d_urn="urn:adsk.eagle:package:43461/1" value="BAT60AE6327HTSA1"/>
@@
 <part name="C4" library="rcl" deviceset="C-EU" device="C0603" value="0.1uF MLCC"/>
 <part name="C5" library="rcl" deviceset="C-EU" device="C0603" value="0.1uF MLCC"/>
+<part name="D1" library="diodes" deviceset="MBRS1100T3G" device=""/>
+<part name="L1" library="inductor-bourns" deviceset="SRR1208" device="">
+<attribute name="MPN" value="SRR1208-151YL"/>
+</part>
 </parts>
 <sheets>
@@
 <text x="-83.82" y="190.5" size="1.778" layer="91">Design is provided "AS IS" and "WITH ALL FAULTS. OpenEnergyMonitor DISCLAIMS ALL OTHER WARRANTIES, EXPRESS OR IMPLIED,</text>
 <text x="-83.82" y="194.31" size="1.778" layer="91">Hardware design files are licensed under the Creative Commons Attribution-ShareAlike 3.0 Unported License</text>
-<text x="-35.306" y="279.908" size="2.286" layer="91">DC INPUT, ELS POWER &amp; VOLTAGE REGULATORS</text>
+<text x="-35.306" y="279.908" size="2.286" layer="91">DC INPUT &amp; REGULATORS</text>
 <wire x1="147.32" y1="292.1" x2="182.88" y2="292.1" width="0.1524" layer="94"/>
 <wire x1="182.88" y1="292.1" x2="284.48" y2="292.1" width="0.1524" layer="94"/>
@@
 <instance part="GND7" gate="1" x="-60.96" y="307.34"/>
 <instance part="R5" gate="G$1" x="-27.94" y="347.98"/>
-<instance part="D1" gate="G$1" x="-17.78" y="241.3" smashed="yes" rot="R90">
-<attribute name="OC_FARNELL" x="-17.78" y="241.3" size="1.778" layer="96" display="off"/>
-<attribute name="MF" x="-17.78" y="241.3" size="1.778" layer="96" display="off"/>
-<attribute name="MPN" x="-17.78" y="241.3" size="1.778" layer="96" display="off"/>
-</instance>
 <instance part="C48" gate="G$1" x="17.78" y="246.38"/>
 <instance part="GND23" gate="1" x="93.98" y="231.14"/>
@@
 <instance part="REG1117" gate="G$1" x="63.5" y="254"/>
 <instance part="SUPPLY4" gate="G$1" x="93.98" y="256.54"/>
-<instance part="I1" gate="G$1" x="-15.24" y="259.08">
-<attribute name="OC_FARNELL" x="-15.24" y="259.08" size="1.778" layer="96" display="off"/>
-<attribute name="MF" x="-15.24" y="259.08" size="1.778" layer="96" display="off"/>
-<attribute name="MPN" x="-15.24" y="259.08" size="1.778" layer="96" display="off"/>
-</instance>
 <instance part="SUPPLY5" gate="G$1" x="-22.86" y="325.12"/>
 <instance part="D2" gate="G$1" x="27.94" y="259.08"/>
@@
 <attribute name="MPN" x="-45.72" y="320.04" size="1.778" layer="96" display="off"/>
 </instance>
-<instance part="C3" gate="A" x="-7.62" y="246.38" rot="R270"/>
+<instance part="C3" gate="A" x="0" y="246.38" rot="R270"/>
 <instance part="C1" gate="G$1" x="45.72" y="246.38"/>
 <instance part="C18" gate="G$1" x="78.74" y="246.38"/>
@@
 <instance part="C4" gate="G$1" x="-30.48" y="259.08"/>
 <instance part="C5" gate="G$1" x="-30.48" y="241.3"/>
+<instance part="D1" gate="G$1" x="-20.32" y="243.84" smashed="yes" rot="R90">
+<attribute name="NAME" x="-22.098" y="241.3" size="1.778" layer="95" rot="R90"/>
+</instance>
+<instance part="L1" gate="G$1" x="-5.08" y="254" smashed="yes">
+<attribute name="NAME" x="-11.43" y="255.778" size="1.778" layer="95"/>
+</instance>
 </instances>
 <busses>
@@
 <pinref part="REG1117" gate="G$1" pin="GND"/>
 <wire x1="63.5" y1="241.3" x2="63.5" y2="233.68" width="0.1524" layer="91"/>
-<pinref part="D1" gate="G$1" pin="A"/>
-<wire x1="-17.78" y1="238.76" x2="-17.78" y2="233.68" width="0.1524" layer="91"/>
-<wire x1="-17.78" y1="233.68" x2="-30.48" y2="233.68" width="0.1524" layer="91"/>
+<wire x1="-20.32" y1="241.3" x2="-20.32" y2="233.68" width="0.1524" layer="91"/>
+<wire x1="-20.32" y1="233.68" x2="-30.48" y2="233.68" width="0.1524" layer="91"/>
 <wire x1="-30.48" y1="233.68" x2="-45.72" y2="233.68" width="0.1524" layer="91"/>
 <wire x1="-45.72" y1="233.68" x2="-55.88" y2="233.68" width="0.1524" layer="91"/>
@@
 <wire x1="-71.12" y1="233.68" x2="-91.44" y2="233.68" width="0.1524" layer="91"/>
 <wire x1="-91.44" y1="233.68" x2="-121.92" y2="233.68" width="0.1524" layer="91"/>
-<wire x1="-17.78" y1="233.68" x2="-7.62" y2="233.68" width="0.1524" layer="91"/>
-<wire x1="-7.62" y1="233.68" x2="17.78" y2="233.68" width="0.1524" layer="91"/>
-<junction x="-17.78" y="233.68"/>
+<wire x1="-20.32" y1="233.68" x2="0" y2="233.68" width="0.1524" layer="91"/>
+<wire x1="0" y1="233.68" x2="17.78" y2="233.68" width="0.1524" layer="91"/>
+<junction x="-20.32" y="233.68"/>
 <pinref part="C48" gate="G$1" pin="2"/>
 <wire x1="17.78" y1="241.3" x2="17.78" y2="233.68" width="0.1524" layer="91"/>
 <junction x="17.78" y="233.68"/>
-<wire x1="-7.62" y1="238.76" x2="-7.62" y2="233.68" width="0.1524" layer="91"/>
-<junction x="-7.62" y="233.68"/>
+<wire x1="0" y1="238.76" x2="0" y2="233.68" width="0.1524" layer="91"/>
+<junction x="0" y="233.68"/>
 <wire x1="17.78" y1="233.68" x2="45.72" y2="233.68" width="0.1524" layer="91"/>
 <wire x1="45.72" y1="241.3" x2="45.72" y2="233.68" width="0.1524" layer="91"/>
@@
 <wire x1="-71.12" y1="254" x2="-71.12" y2="233.68" width="0.1524" layer="91"/>
 <junction x="-71.12" y="233.68"/>
+<pinref part="D1" gate="G$1" pin="A"/>
 </segment>
 <segment>
@@
 <wire x1="91.44" y1="347.98" x2="66.04" y2="347.98" width="0.1524" layer="91"/>
 <label x="53.34" y="347.98" size="1.778" layer="95"/>
-</segment>
-</net>
-<net name="IND" class="0">
-<segment>
-<wire x1="-15.24" y1="259.08" x2="-17.78" y2="259.08" width="0.1524" layer="91"/>
-<pinref part="D1" gate="G$1" pin="C"/>
-<wire x1="-17.78" y1="243.84" x2="-17.78" y2="259.08" width="0.1524" layer="91"/>
-<junction x="-17.78" y="259.08"/>
-<wire x1="-17.78" y1="259.08" x2="-22.86" y2="259.08" width="0.1524" layer="91"/>
-<wire x1="-22.86" y1="259.08" x2="-25.4" y2="254" width="0.1524" layer="91"/>
-<pinref part="I1" gate="G$1" pin="P$1"/>
 </segment>
 </net>
@@
 <net name="+5V" class="0">
 <segment>
-<pinref part="I1" gate="G$1" pin="P$2"/>
-<wire x1="15.24" y1="259.08" x2="12.7" y2="259.08" width="0.1524" layer="91"/>
-<wire x1="-7.62" y1="251.46" x2="-7.62" y2="246.38" width="0.1524" layer="91"/>
-<wire x1="-7.62" y1="251.46" x2="15.24" y2="251.46" width="0.1524" layer="91"/>
-<wire x1="15.24" y1="251.46" x2="15.24" y2="259.08" width="0.1524" layer="91"/>
+<pinref part="C48" gate="G$1" pin="1"/>
+<pinref part="B1" gate="G$1" pin="1"/>
+<wire x1="25.4" y1="264.16" x2="26.67" y2="264.16" width="0.1524" layer="91"/>
 <pinref part="D2" gate="G$1" pin="A"/>
-<pinref part="C48" gate="G$1" pin="1"/>
+<wire x1="25.4" y1="259.08" x2="25.4" y2="264.16" width="0.1524" layer="91"/>
+<junction x="25.4" y="259.08"/>
 <wire x1="25.4" y1="259.08" x2="17.78" y2="259.08" width="0.1524" layer="91"/>
-<wire x1="17.78" y1="259.08" x2="17.78" y2="248.92" width="0.1524" layer="91"/>
-<wire x1="15.24" y1="259.08" x2="17.78" y2="259.08" width="0.1524" layer="91"/>
-<junction x="15.24" y="259.08"/>
 <junction x="17.78" y="259.08"/>
-<pinref part="C3" gate="A" pin="1"/>
 <pinref part="P+1" gate="1" pin="+5V"/>
 <wire x1="17.78" y1="266.7" x2="17.78" y2="259.08" width="0.1524" layer="91"/>
-<pinref part="B1" gate="G$1" pin="1"/>
-<wire x1="25.4" y1="259.08" x2="25.4" y2="264.16" width="0.1524" layer="91"/>
-<wire x1="25.4" y1="264.16" x2="26.67" y2="264.16" width="0.1524" layer="91"/>
-<junction x="25.4" y="259.08"/>
+<wire x1="17.78" y1="259.08" x2="17.78" y2="248.92" width="0.1524" layer="91"/>
+<wire x1="0" y1="248.92" x2="0" y2="246.38" width="0.1524" layer="91"/>
+<pinref part="C3" gate="A" pin="1"/>
+<pinref part="L1" gate="G$1" pin="2"/>
+<wire x1="0" y1="254" x2="0" y2="248.92" width="0.1524" layer="91"/>
+<junction x="0" y="248.92"/>
+<pinref part="U1" gate="G$1" pin="FB"/>
+<wire x1="0" y1="248.92" x2="-33.02" y2="248.92" width="0.1524" layer="91"/>
+<wire x1="0" y1="254" x2="7.62" y2="254" width="0.1524" layer="91"/>
+<junction x="0" y="254"/>
+<wire x1="7.62" y1="254" x2="7.62" y2="259.08" width="0.1524" layer="91"/>
+<wire x1="7.62" y1="259.08" x2="17.78" y2="259.08" width="0.1524" layer="91"/>
 </segment>
 </net>
@@
 <pinref part="U1" gate="G$1" pin="LX/OUT"/>
 <wire x1="-30.48" y1="254" x2="-33.02" y2="254" width="0.1524" layer="91"/>
-</segment>
-</net>
+<pinref part="L1" gate="G$1" pin="1"/>
+<wire x1="-10.16" y1="254" x2="-20.32" y2="254" width="0.1524" layer="91"/>
+<junction x="-30.48" y="254"/>
+<pinref part="D1" gate="G$1" pin="C"/>
+<wire x1="-20.32" y1="254" x2="-30.48" y2="254" width="0.1524" layer="91"/>
+<wire x1="-20.32" y1="246.38" x2="-20.32" y2="254" width="0.1524" layer="91"/>
+<junction x="-20.32" y="254"/>
+</segment>
+</net>

Commit message: commit
Parts:
- added C8: 68UF, Panasonic-EEE-EEV-EEF-ECQ:EEV-FK2A680Q-CASE-H13
Changed lines of the file:
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@@
 <attribute name="MPN" value="SRR1208-151YL"/>
 </part>
+<part name="C8" library="Panasonic-EEE-EEV-EEF-ECQ" deviceset="EEV-" device="-CASE-H13" technology="FK2A680Q" value="68UF"/>
 </parts>
 <sheets>
@@
 <attribute name="NAME" x="-11.43" y="255.778" size="1.778" layer="95"/>
 </instance>
+<instance part="C8" gate="A" x="22.86" y="368.3"/>
 </instances>
 <busses>

Commit message: commit
Parts:
- removed B1: (no value), SparkFun:M02PTH
- removed C1, C18: 10uF TANT, rcl:C-EUC0603
- removed C8: 68UF, Panasonic-EEE-EEV-EEF-ECQ:EEV-FK2A680Q-CASE-H13
- removed D2: BAT60AE6327HTSA1, diode:BAT60J
- removed ESP-PWR: (no value), jumper:SJ
- removed MC2: MC32882, multicomp tact switch:MC32882
- removed MINI_USB-B: 5000751517_SD, 5000751517_sd:5000751517_SD
- removed REG1117: REG1117-3.3V, burr-brown:REG1117-VOUT4
- removed U1: MAX5035, MAX5035:MAX5035
- added BOOTL, ESP_PWR: (no value), SparkFun:M02PTH
- added C11T, C18T, C1T: 10uF TANT, rcl:C-EUC0603
- added C14: 0.1uF, rcl:C-EUC0603
- added R20: 57.6k, rcl:R-EU_R0603
- added R21: 13.3k, rcl:R-EU_R0603
- added REG0: MAX5035, MAX5035:MAX5035
- added REG1: REG1117-5.0V, burr-brown:REG1117-VOUT4
- added REG2: REG1117-3.3V, burr-brown:REG1117-VOUT4
- added USB_PWR: 5000751517_SD, 5000751517_sd:5000751517_SD
- C13: value 100nF -> 0.1uF
- C4, C5: value 0.1uF MLCC -> 0.1uF 16V MLCC
- D1: MPN (none) -> MBRS1100T3G
- renumbered U$1 to SCREW_TERM_2, U$3 to SCREW_TERM_1
Connections:
- removed net +5V: B1.1, C3.1, C48.1, D2.A, L1.2, U1.FB
- removed net 4.7V: B1.2, C1.1, C26.1, C9.1, D2.C, FTDI1.4, FTDI2.4, MCP3208.VDD, MINI_USB-B.1, R10.2, REG1117.VIN, SHUNTMON-A.VCC, SHUNTMON-B.VCC
- removed net N$1: C5.1, U1.VD
- removed net N$3: C4.1, U1.BST
- removed net N$5: C4.2, D1.C, L1.1, U1.LX/OUT
- removed net PWR_IN: C10.1, C16.1, PWR.2, U1.ON/OFF, U1.V_IN
- new net 5.0V: C14.1, C1T.1, C26.1, C9.1, FTDI1.4, FTDI2.4, MCP3208.VDD, R10.2, REG1.VOUT, REG2.VIN, SHUNTMON-A.VCC, SHUNTMON-B.VCC, USB_PWR.1
- new net 6.5V: C11T.1, C3.1, C48.1, L1.2, R20.2, REG1.VIN
- new net BST: C4.1, REG0.BST
- new net FB: R20.1, R21.2, REG0.FB
- new net LX: C4.2, D1.C, L1.1, REG0.LX/OUT
- new net VD: C5.1, REG0.VD
- new net V_IN: C10.1, C16.1, PWR.2, REG0.ON/OFF, REG0.V_IN
- net 3.3V: now also C18T.1, ESP_PWR.2, REG2.VOUT; no longer C18.1, ESP-PWR.2, P1.3, REG1117.VOUT
- net 3.3V-ESP: now also ESP_PWR.1, P1.3; no longer ESP-PWR.1
- net GND: now also BOOTL.1, C11T.2, C14.2, C18T.2, C1T.2, R21.1, REG0.GND, REG0.SGND, REG1.GND, REG2.GND, USB_PWR.5; no longer C1.2, C18.2, MC2.P$1, MINI_USB-B.5, REG1117.GND, U1.GND, U1.SGND
- net GPIO0: now also BOOTL.2; no longer MC2.P$2
Other:
- note added: "Power Supply"
- note removed: "4.7V AFTER DIODE TO 3.3V"
- note removed: "Power"
- moved on the sheet: C10, C13, C16, C2, C3, C4, C48, C5, D1, FTDI2, GPIO_1, L1

Commit message: commit
Parts:
- removed ESP_PWR: (no value), SparkFun:M02PTH
- removed S1: SWS002, smd-special:SWS002
- added RX, TX: (no value), SparkFun:M02PTH
- CR1220: MPN (none) -> Harwin S8411-45R
Connections:
- removed net 3.3V-ESP: C22.2, ESP-12.VCC, ESP_PWR.1, IO1.2, P1.3, R12.2, R19.2, R6.2, R7.2, R9.2, U$4.VDD
- removed net GPIO4: MCP3208.!CS
- net 3.3V: now also C22.2, ESP-12.VCC, IO1.2, P1.3, R12.2, R19.2, R6.2, R7.2, R9.2, U$4.VDD; no longer ESP_PWR.2
- net D0/RX: now also TX.2; no longer S1.2
- net D1/TX: now also RX.1; no longer S1.1
- net ESPRX: now also RX.2; no longer S1.4
- net ESPTX: now also TX.1; no longer S1.3
- net GPIO2: now also MCP3208.!CS

Commit message: commit
Parts:
- REG0: MANUFACTURER_PART_NUMBER MAX5035EASA+ -> (none)
Changed lines of the file:
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@@
 <part name="GND10" library="supply1" deviceset="0V" device="" value="GND"/>
 <part name="CR1220" library="IotaWatt_parts" deviceset="CR1220SMD" device="">
-<attribute name="MPN" value="Harwin
-S8411-45R"/>
+<attribute name="MPN" value="Harwin S8411-45R"/>
 </part>
 <part name="ADC-PAD" library="wirepad" library_urn="urn:adsk.eagle:library:412" deviceset="2,15/1,0" device="" package3d_urn="urn:adsk.eagle:package:30831/1"/>
@@
 <part name="U$4" library="MOLEX 47219-2001" deviceset="47219-2001_MICROSD" device=""/>
 <part name="REG0" library="MAX5035" deviceset="MAX5035" device="">
-<attribute name="MANUFACTURER_PART_NUMBER" value="MAX5035EASA+"/>
 <attribute name="MPN" value="MAX5035EASA+"/>
 </part>
