File: emonDCduo-ESP/emonDCduo-ESP v0.3.brd (EAGLE design)
At the start: 99.1 x 76.5 mm, 89 parts, among them Q1 16Mhz XT49M-2016M, U1_TQFP ATMEGA328P

Commit message: SD CARD TO DUO
Parts:
- added X1: SDBMF, farnell:SDBMF-009XXBXX2
Connections:
- removed net RESET1: ESP-12.15, MC1.P$1, MC1.P$2
- new net GPIO12: ESP-12.14, X1.7
- new net GPIO13: ESP-12.15, X1.2
- new net GPIO14: ESP-12.13, X1.5
- new net GPIO16: ESP-12.12, MC1.P$1, MC1.P$2
- new net GPIO2: ESP-12.3, X1.1
- new net GPIO4: ESP-12.6
- new net GPIO5: ESP-12.5
- new net N$33: X1.8
- new net N$34: X1.9
- new net N$44: ESP-12.10
- net 3.3V: now also X1.4
- net GND: now also X1.3, X1.6
Routing:
- net RESET1: track 21.6 -> 0.00 mm, vias 2 -> 0

Commit message: short write protect pins
Connections:
- new net N$11: X1.SW2, X1.SW3
Changed lines of the file:
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@@
 <wire x1="-17.898" y1="10.151" x2="86.868" y2="26.48" width="0" layer="19" extent="1-1"/>
+</signal>
+<signal name="N$11">
+<contactref element="X1" pad="SW2"/>
+<contactref element="X1" pad="SW3"/>
+<wire x1="-35.798" y1="27.526" x2="-35.498" y2="0.076" width="0" layer="19" extent="1-1"/>
 </signal>
 </signals>

Commit message: micro sd card library
pinout in schematic TBD
Parts:
- added U$1: 47219-2001_MICROSD, 47219-2001_SD_MICRO:47219-2001_MICROSD
Changed lines of the file:
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@@
 </element>
 <element name="X1" library="farnell" package="SDBMF-009XXBXX2" value="SDBMF" x="-22.098" y="4.826"/>
+<element name="U$1" library="47219-2001_SD_MICRO" package="47219-2001_MICROSD" value="47219-2001_MICROSD" x="15.24" y="12.7"/>
 </elements>
 <signals>
