File: emonDCduo-ESP/emonDCduo-ESP+RF v0.3.brd (EAGLE design)
At the start: 99.1 x 76.5 mm, 78 parts, among them Q1 16Mhz XT49M-2016M, U1_TQFP ATMEGA328P

Commit message: board layout changes
Parts:
- removed R7: 10k, rcl:R0603
- added ANT1: (no value), discrete:PAD-01
- added C16, C19: 22pF, rcl:C0603
- added C2: 100nF, rcl:C0603
- added C20: tune, rcl:C0603
- added CH_PD: SOLDERJUMPERNO, SparkFun:SJ_2S-NO
- added J$1: SMA_EDGE, SparkFun-Connectors:SMA-EDGE
- added R24: 120K, rcl:R0603
- added RF: RFM12B, JeeParts:RFM12B
- moved R6 117.1 mm to (-5.33, -63.8), turned to 0 degrees
- moved R3 113.9 mm to (-5.33, -58.9), turned to 0 degrees
- moved MC32882 13.3 mm to (25.7, 21.9), turned to 0 degrees
- moved U$1 4.88 mm to (52.1, 15.5), turned to 0 degrees
- moved R19 3.81 mm to (92.5, 18.0)
- moved GPIO0 2.55 mm to (65.3, 30.2)
Connections:
- new net DIG1: C16.1, C19.1, C20.1, RF.ANT
- new net N$11: ANT1.1, C16.2
- new net N$24: C19.2, J$1.SIG
- net 3.3V: now also C2.1, CH_PD.1, R24.2, RF.VDD; no longer R7.2
- net CH_PD: now also CH_PD.2; no longer R7.1
- net D10: now also R24.1, RF.SEL
- net D11/MOSI: now also RF.SDI
- net D12/MISO: now also RF.SDO
- net D13/SCK: now also RF.SCK
- net D2: now also RF.IRQ
- net GND: now also C2.2, C20.2, J$1.GND@0, J$1.GND@1, J$1.GND@2, J$1.GND@3, RF.GND, RF.P$12; no longer U$1.P$1, U$1.P$2, U$1.P$3, U$1.P$4
Routing:
- net 3.3V: track 235.1 -> 158.5 mm, vias 5 -> 3
- net GPIO13: track 53.3 -> 0.00 mm, vias 2 -> 0
- net GPIO12: track 52.7 -> 0.00 mm
- net GPIO14: track 50.0 -> 0.00 mm
- net GPIO2: track 49.5 -> 0.00 mm, vias 2 -> 0
- net GPIO15: track 27.1 -> 1.64 mm, vias 2 -> 0
- net GPIO16: track 16.0 -> 0.00 mm, vias 2 -> 0
- net 4.7V: track 148.1 -> 158.5 mm
- net ESPTX: track 48.5 -> 42.2 mm
- net RESTESP: track 11.1 -> 7.20 mm
- net GPIO0: track 19.6 -> 17.1 mm
- net N$30: track 38.4 -> 35.9 mm
- net RES: track 52.0 -> 50.7 mm
- net D0/RX: track 76.7 -> 77.3 mm
- net CH_PD: track 2.51 -> 1.90 mm
- added copper zone on layer 1, net GNDI
- added copper zone on layer 16, net GNDI
Other:
- outline, holes or cut-outs redrawn
- board text added: "ISOLATED UART / FTDI"
