File: emonDCduo-ESP/emonDCduo-ESP+RF v0.3.sch (EAGLE design)
At the start: 78 parts, among them Q1 16Mhz XT49M-2016M, U1_TQFP ATMEGA328P

Commit message: board layout changes
Parts:
- removed R7: 10k, rcl:R-EU_R0603
- added ANT1: (no value), discrete:ANTENNA
- added C16, C19: 22pF, rcl:C-EUC0603
- added C2: 100nF, rcl:C-EUC0603
- added C20: tune, rcl:C-EUC0603
- added CH_PD: SOLDERJUMPERNO, SparkFun:SOLDERJUMPERNO
- added J$1: SMA_EDGE, SparkFun-Connectors:SMA_EDGE
- added R24: 120K, rcl:R-EU_R0603
- added RF: RFM12B, JeeParts:RFM12B
Connections:
- new net DIG1: C16.1, C19.1, C20.1, RF.ANT
- new net N$11: ANT1.1, C16.2
- new net N$24: C19.2, J$1.SIGNAL
- net 3.3V: now also C2.1, CH_PD.1, R24.2, RF.VCC; no longer R7.2
- net CH_PD: now also CH_PD.2; no longer R7.1
- net D10: now also R24.1, RF.SEL
- net D11/MOSI: now also RF.SDI
- net D12/MISO: now also RF.SDO
- net D13/SCK: now also RF.SCK
- net D2: now also RF.IRQ
- net GND: now also C2.2, C20.2, J$1.GND@0, J$1.GND@1, J$1.GND@2, J$1.GND@3, RF.GND; no longer U$1.GND
Other:
- note added: "RFM12B RFM69CW"
- moved on the sheet: C21, C22, FTDI1, GPIO0, R17, R18, R19, R3, R6, RX, TX
