File: emonDCduo-ESP/emonDCduo-ESP v0.4.brd (EAGLE design)
At the start: 99.1 x 76.5 mm, 82 parts, among them Q1 16Mhz XT49M-2016M, U1_TQFP ATMEGA328P

Commit message: gerber
Parts:
- removed C20-TUNE: tune, rcl:C0603
- added C19: 22pF, rcl:C0603
- added C20/TUNE: tune, rcl:C0603
- added GPIO-4/5: (no value), SparkFun:1X02
- added PAD1: (no value), wirepad:SMD1,27-2,54
- moved MC32882 17.5 mm to (83.2, 74.7), turned to 270 degrees
- moved C13 5.56 mm to (81.1, 76.1), turned to 90 degrees
- moved C1 3.87 mm to (72.8, 72.0), turned to 270 degrees
- moved ANT1 3.30 mm to (85.2, 9.91)
- moved 3.3V_REG 2.54 mm to (78.1, 69.8)
- moved C18 2.45 mm to (77.2, 75.7)
- moved REFERENCE_SELECT 2.12 mm to (42.2, 53.7)
- moved TX 1.52 mm to (37.1, 18.5)
- moved RX 1.27 mm to (37.1, 15.5)
- moved R32 1.02 mm to (86.8, 65.3)
- moved R13 0.51 mm to (38.9, 56.6)
- moved R5 0.51 mm to (38.9, 42.6)
- moved C26 0.20 mm to (38.6, 50.8)
Connections:
- new net N$3: ANT1.1, C19.2
- new net N$5: PAD1.1
- net DIG1: now also C19.1, C20/TUNE.1; no longer ANT1.1, C20-TUNE.1
- net GND: now also C20/TUNE.2; no longer C20-TUNE.2
- net GPIO4: now also GPIO-4/5.1
- net GPIO5: now also GPIO-4/5.2
Routing:
- net GPIO5: track 0.00 -> 32.0 mm
- net GPIO4: track 0.00 -> 30.5 mm
- net RES: track 64.3 -> 77.6 mm
- net DIG1: track 11.9 -> 5.14 mm, vias 1 -> 0
- net RESET: track 49.1 -> 46.3 mm
- net N$3: track 0.00 -> 2.32 mm
- net 3.3V: track 269.7 -> 267.4 mm
- net REFINPUT: track 17.1 -> 19.4 mm
- net 4.7V: track 161.7 -> 163.5 mm
- net D1/TX: track 86.1 -> 84.6 mm
- net ESPTX: track 42.7 -> 43.9 mm
- net GPIO12: track 52.5 -> 53.6 mm
- net D0/RX: track 93.7 -> 93.0 mm
- net N$31: track 168.2 -> 168.7 mm, vias 1 -> 0
- net ADCSHUNT-A: track 39.8 -> 39.3 mm
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Other:
- board text added: "GPIO4"
- board text added: "GPIO5"

Commit message: refinement
Parts:
- I1: value (none) -> 330uH
Other:
- board text added: "ADC2"
- board text added: "ADC3"
- board text added: "I1"
- board text removed: "Ind1"
