File: emonDCduo-ESP/emonDCduo-ESP v1.0.sch (EAGLE design)
At the start: 86 parts, among them Q1 16Mhz XT49M-2016M, U1_TQFP ATMEGA328P

Commit message: update
Parts:
- added GPIO1: (no value), SparkFun:M02PTH
- added MINI_USB-B: 5000751517_SD, 5000751517_sd:5000751517_SD
- D1: value BAT60J -> MBRA130LT3G; device diode:BAT60J -> CASE 403D Diode:MBRA130LT3G; MF (none) -> ON SEMICONDUCTOR; MPN (none) -> MBRA130LT3G; OC_FARNELL (none) -> 9555978
- D2: value MBRA130LT3G -> BAT60J; device CASE 403D Diode:MBRA130LT3G -> diode:BAT60J; MF ON SEMICONDUCTOR -> (none); MPN MBRA130LT3G -> (none); OC_FARNELL 9555978 -> (none)
Connections:
- net 4.7V: now also D2.C, FTDI1.4, MINI_USB-B.1; no longer D1.C
- net 5.0V: now also D2.A; no longer D1.A
- net GND: now also D1.A, GPIO1.1, MINI_USB-B.5; no longer D2.A
- net GPIO15: now also GPIO1.2
- net IND: now also D1.C; no longer D2.C
Other:
- moved on the sheet: R3
Changed lines of the file:
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@@
 <?xml version="1.0" encoding="utf-8"?>
 <!DOCTYPE eagle SYSTEM "eagle.dtd">
-<eagle version="8.0.1">
+<eagle version="7.7.0">
 <drawing>
 <settings>
@@
 <setting verticaltext="up"/>
 </settings>
-<grid distance="0.1" unitdist="inch" unit="inch" style="lines" multiple="1" display="no" altdistance="0.01" altunitdist="inch" altunit="inch"/>
+<grid distance="0.1" unitdist="inch" unit="inch" style="lines" multiple="1" display="no" altdistance="0.05" altunitdist="inch" altunit="inch"/>
 <layers>
 <layer number="1" name="Top" color="4" fill="1" visible="no" active="no"/>
@@
 <part name="R5" library="rcl" deviceset="R-EU_" device="R0603" value="1K"/>
 <part name="GND8" library="supply1" deviceset="GND" device=""/>
-<part name="D2" library="CASE 403D Diode" deviceset="MBRA130LT3G" device="">
+<part name="D1" library="CASE 403D Diode" deviceset="MBRA130LT3G" device="">
 <attribute name="MF" value="ON SEMICONDUCTOR"/>
 <attribute name="MPN" value="MBRA130LT3G"/>
@@
 <part name="SUPPLY14" library="supply2" deviceset="GND" device=""/>
 <part name="MC32882" library="multicomp tact switch" deviceset="MC32882" device=""/>
-<part name="D1" library="diode" deviceset="BAT60J" device=""/>
+<part name="D2" library="diode" deviceset="BAT60J" device=""/>
 <part name="FTDI/UART" library="SparkFun" deviceset="FTDI_BASIC" device="PTH" value="2211S-06G">
 <attribute name="MF" value="MULTICOMP"/>
@@
 <part name="R9" library="rcl" deviceset="R-EU_" device="R0603" value="10k"/>
 <part name="GPIO5" library="wirepad" deviceset="2,15/1,0" device=""/>
+<part name="MINI_USB-B" library="5000751517_sd" deviceset="5000751517_SD" device=""/>
+<part name="GPIO1" library="SparkFun" deviceset="M02" device="PTH"/>
 </parts>
 <sheets>
@@
 <instance part="R5" gate="G$1" x="-53.34" y="347.98"/>
 <instance part="GND8" gate="1" x="-45.72" y="358.14"/>
-<instance part="D2" gate="G$1" x="-17.78" y="241.3" smashed="yes" rot="R90">
+<instance part="D1" gate="G$1" x="-17.78" y="241.3" smashed="yes" rot="R90">
 <attribute name="OC_FARNELL" x="-17.78" y="241.3" size="1.778" layer="96" display="off"/>
 <attribute name="MF" x="-17.78" y="241.3" size="1.778" layer="96" display="off"/>
@@
 <instance part="SUPPLY14" gate="GND" x="205.74" y="297.18"/>
 <instance part="MC32882" gate="G$1" x="205.74" y="309.88"/>
-<instance part="D1" gate="G$1" x="27.94" y="259.08"/>
+<instance part="D2" gate="G$1" x="27.94" y="259.08"/>
 <instance part="FTDI/UART" gate="G$1" x="203.2" y="246.38">
 <attribute name="OC_FARNELL" x="203.2" y="246.38" size="1.778" layer="96" display="off"/>
@@
 <instance part="J3" gate="J$1" x="-96.52" y="335.28" rot="R270"/>
 <instance part="J4" gate="J$1" x="-96.52" y="337.82" rot="R90"/>
-<instance part="R3" gate="G$1" x="190.5" y="457.2"/>
+<instance part="R3" gate="G$1" x="189.23" y="457.2"/>
 <instance part="R6" gate="G$1" x="200.66" y="462.28" rot="R90"/>
 <instance part="P+5" gate="G$1" x="200.66" y="469.9"/>
@@
 <instance part="R9" gate="G$1" x="200.66" y="441.96" rot="R180"/>
 <instance part="GPIO5" gate="1" x="208.28" y="401.32"/>
+<instance part="MINI_USB-B" gate="G$1" x="129.54" y="269.24"/>
+<instance part="GPIO1" gate="G$1" x="187.96" y="469.9" rot="R270"/>
 </instances>
 <busses>
@@
 </segment>
 <segment>
-<wire x1="185.42" y1="457.2" x2="177.8" y2="457.2" width="0.1524" layer="91"/>
+<wire x1="184.15" y1="457.2" x2="177.8" y2="457.2" width="0.1524" layer="91"/>
 <wire x1="177.8" y1="457.2" x2="177.8" y2="414.02" width="0.1524" layer="91"/>
 <pinref part="FTDI1" gate="1" pin="6"/>
@@
 <junction x="190.5" y="414.02"/>
 <pinref part="R3" gate="G$1" pin="1"/>
+<pinref part="GPIO1" gate="G$1" pin="1"/>
+<wire x1="187.96" y1="462.28" x2="184.15" y2="462.28" width="0.1524" layer="91"/>
+<wire x1="184.15" y1="462.28" x2="184.15" y2="457.2" width="0.1524" layer="91"/>
+<junction x="184.15" y="457.2"/>
 </segment>
 <segment>
@@
 <wire x1="-78.74" y1="233.68" x2="-68.58" y2="233.68" width="0.1524" layer="91"/>
 <wire x1="-68.58" y1="233.68" x2="-68.58" y2="246.38" width="0.1524" layer="91"/>
-<pinref part="D2" gate="G$1" pin="A"/>
+<pinref part="D1" gate="G$1" pin="A"/>
 <wire x1="-17.78" y1="238.76" x2="-17.78" y2="233.68" width="0.1524" layer="91"/>
 <wire x1="-17.78" y1="233.68" x2="-68.58" y2="233.68" width="0.1524" layer="91"/>
@@
 <pinref part="C10" gate="A" pin="2"/>
 <pinref part="GND18" gate="1" pin="0V"/>
+<pinref part="MINI_USB-B" gate="G$1" pin="5"/>
+<wire x1="121.92" y1="264.16" x2="121.92" y2="233.68" width="0.1524" layer="91"/>
+<wire x1="121.92" y1="233.68" x2="93.98" y2="233.68" width="0.1524" layer="91"/>
 </segment>
 <segment>
@@
 <segment>
 <wire x1="-15.24" y1="259.08" x2="-17.78" y2="259.08" width="0.1524" layer="91"/>
-<pinref part="D2" gate="G$1" pin="C"/>
+<pinref part="D1" gate="G$1" pin="C"/>
 <wire x1="-17.78" y1="243.84" x2="-17.78" y2="259.08" width="0.1524" layer="91"/>
 <junction x="-17.78" y="259.08"/>
@@
 <net name="4.7V" class="1">
 <segment>
-<pinref part="D1" gate="G$1" pin="C"/>
+<pinref part="D2" gate="G$1" pin="C"/>
 <label x="38.608" y="259.588" size="1.778" layer="95"/>
-<wire x1="30.48" y1="259.08" x2="45.72" y2="259.08" width="0.1524" layer="91"/>
+<wire x1="30.48" y1="259.08" x2="33.02" y2="259.08" width="0.1524" layer="91"/>
+<wire x1="33.02" y1="259.08" x2="45.72" y2="259.08" width="0.1524" layer="91"/>
 <wire x1="45.72" y1="259.08" x2="45.72" y2="254" width="0.1524" layer="91"/>
 <wire x1="45.72" y1="248.92" x2="45.72" y2="254" width="0.1524" layer="91"/>
@@
 <junction x="45.72" y="254"/>
 <pinref part="C1" gate="G$1" pin="1"/>
+<pinref part="MINI_USB-B" gate="G$1" pin="1"/>
+<wire x1="121.92" y1="274.32" x2="33.02" y2="274.32" width="0.1524" layer="91"/>
+<wire x1="33.02" y1="274.32" x2="33.02" y2="259.08" width="0.1524" layer="91"/>
+<junction x="33.02" y="259.08"/>
 </segment>
 <segment>
@@
 <wire x1="-48.26" y1="322.58" x2="-48.26" y2="325.12" width="0.1524" layer="91"/>
 <junction x="-71.12" y="322.58"/>
+</segment>
+<segment>
+<pinref part="FTDI1" gate="1" pin="4"/>
+<wire x1="213.36" y1="419.1" x2="210.82" y2="419.1" width="0.1524" layer="91"/>
 </segment>
 </net>
@@
 <wire x1="-7.62" y1="251.46" x2="15.24" y2="251.46" width="0.1524" layer="91"/>
 <wire x1="15.24" y1="251.46" x2="15.24" y2="259.08" width="0.1524" layer="91"/>
-<pinref part="D1" gate="G$1" pin="A"/>
+<pinref part="D2" gate="G$1" pin="A"/>
 <pinref part="C48" gate="G$1" pin="1"/>
 <wire x1="25.4" y1="259.08" x2="17.78" y2="259.08" width="0.1524" layer="91"/>
@@
 <wire x1="195.58" y1="452.12" x2="195.58" y2="454.66" width="0.1524" layer="91"/>
 <junction x="195.58" y="454.66"/>
-<wire x1="195.58" y1="454.66" x2="195.58" y2="457.2" width="0.1524" layer="91"/>
+<wire x1="195.58" y1="454.66" x2="194.31" y2="457.2" width="0.1524" layer="91"/>
 <pinref part="R3" gate="G$1" pin="2"/>
 <wire x1="195.58" y1="452.12" x2="210.82" y2="452.12" width="0.1524" layer="91"/>
-</segment>
-</net>
+<pinref part="GPIO1" gate="G$1" pin="2"/>
+<wire x1="190.5" y1="462.28" x2="194.31" y2="462.28" width="0.1524" layer="91"/>
+<wire x1="194.31" y1="462.28" x2="194.31" y2="457.2" width="0.1524" layer="91"/>
+<junction x="194.31" y="457.2"/>
+</segment>
+</net>

Commit message: added DIP switch to ESP RX/TX
Parts:
- removed C28, C29, C30, C31: 0.1uF 100V, rcl:C-EUC0603
- removed GPIO0, GPIO1, RX, TX: (no value), SparkFun:M02PTH
- removed GPIO5: (no value), wirepad:2,15/1,0
- removed MC32882: MC32882, multicomp tact switch:MC32882
- removed R3, R9: 10k, rcl:R-EU_R0603
- added CD1, ESP-PWR, RF-PWR: (no value), jumper:SJ
- added IO2: (no value), SparkFun:M02PTH
- added MC2: MC32882, multicomp tact switch:MC32882
- added S1: A6S-2104-PH, OpenEnergyMonitor:2_SMT_DIP_SWITCH
- added T3: (no value), con-weidmueller-sl35:180-2
Connections:
- net ADCVSENSE-A renamed ADC5-VSENSEB
- net ADCVSENSE-B renamed ADC4-VSENSEA
- net N$2 renamed ADC0
- net N$27 renamed ADC1
- removed net GPIO15: C22.1, ESP-12.GND, ESP-12.GPIO15, GPIO1.2, R3.2
- new net 3.3V-ESP: C22.2, ESP-12.VCC, ESP-PWR.1, MC1.P$2, R19.2, R6.2, R7.2, U$2.VDD
- new net N$17: C2.1, R24.2, RF-PWR.2, RF.VCC
- net 3.3V: now also ESP-PWR.2, RF-PWR.1; no longer C2.1, C22.2, ESP-12.VCC, MC1.P$2, R19.2, R24.2, R6.2, R7.2, RF.VCC, U$2.VDD
- net ADCSHUNT-A: now also R4.2, R5.2; no longer R13.2, R16.2
- net ADCSHUNT-B: now also R13.2, R16.2; no longer R4.2, R5.2
- net D0/RX: now also S1.1; no longer RX.2
- net D1/TX: now also S1.2; no longer TX.2
- net ESPRX: now also S1.3; no longer TX.1
- net ESPTX: now also S1.4; no longer RX.1
- net GND: now also C22.1, ESP-12.GND, ESP-12.GPIO15, MC2.P$1, T3.1, T3.2; no longer C28.2, C29.2, C30.2, C31.2, GPIO0.1, GPIO1.1, MC32882.P$2, R3.1
- net GPIO0: now also MC2.P$2; no longer GPIO0.2
- net GPIO4: now also CD1.2, IO2.1; no longer R9.1
- net GPIO5: now also IO2.2; no longer GPIO5.P
- net INPUT-POS-A: no longer C30.1
- net INPUT-POS-B: no longer C29.1
- net LOAD-NEG-A: no longer C31.1
- net LOAD-NEG-B: no longer C28.1
- net N$10: now also CD1.1; no longer R9.2
- net RES: no longer MC32882.P$1
Other:
- moved on the sheet: ANA, ANT1, C19, C2, C20, C21, C22, C27, C5, FTDI1, PAD1, R16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

Commit message: emonBIKE v0.2 camexport
Parts:
- removed C-TANT: 10uF 63V, 2917 footprint capacitor:293D
- removed C17: 100nF, rcl:C-EUC0603
- removed JP_PWR: 2211S-02G, jumper:JP1Q
- removed MC1: MC32882, multicomp tact switch:MC32882
- removed REF_SELECT: 2212S-02SG-85, SparkFun-Connectors:CONN_03
- added C14, C15: 100nF, rcl:C-EUC0603
- added C16: 0.1uF 100V, rcl:C-EUC0603
- added IO1: (no value), SparkFun:M02PTH
- added PWR: (no value), SparkFun-Connectors:CONN_03
- added REF_GND: (no value), jumper:SJ
- added REF_SELECT_A: 2212S-02SG-85, SparkFun-Connectors:CONN_03
- C12: value 220nF -> 100nF
- C26, C9: value 0.1uF 100V -> 100nF
- C3: value 470uF -> 470uF 16V
- C51: value 100nF -> 0.1uF 100V
- R1, R14: value 100K 60V -> 100K 75V
- R15, R2: value 5.9K -> 5.6K
- R17: value 5.6k -> 5.6K
- R18, R19, R6, R7: value 10k -> 10K
- R32: value 10K -> 10k
Connections:
- net N$17 renamed 3.3V-RF
- removed net INPUT-POS-A: C25.1, J2.1, J2.2, J2.3, R14.2, SHUNTMON-A.RSP, T1.2
- removed net INPUT-POS-B: C6.1, J3.1, J3.2, J3.3, R1.2, SHUNTMON-B.RSP, T2.2
- removed net POWERIN: C10.1, C51.1, JP_PWR.1, TL2575HV.VIN
- removed net RES: C17.1, FTDI/UART.1
- removed net RESET: C17.2, ISP.5, R32.1, U1_TQFP.PC6(/RESET)
- new net PWR_IN: C10.1, C16.1, C51.1, PWR.2, TL2575HV.VIN
- new net RESET1: C14.2, FTDI/UART.1, ISP.5
- new net RESET2: C14.1, R32.1, U1_TQFP.PC6(/RESET)
- new net SOURCE-POS-A: C6.1, J3.1, J3.2, J3.3, PWR.1, R1.2, SHUNTMON-B.RSP, T2.2
- new net SOURCE-POS-B: C25.1, J2.1, J2.2, J2.3, PWR.3, R14.2, SHUNTMON-A.RSP, T1.2
- net 3.3V-ESP: now also IO1.2; no longer MC1.P$2
- net GND: now also C15.2, C16.2, REF_GND.2, REF_SELECT_A.3; no longer C-TANT.2, REF_SELECT.3
- net GPIO16: now also IO1.1; no longer MC1.P$1
- net LOAD-NEG-A: now also C24.2, J4.1, J4.2, J4.3, SHUNTMON-B.RSN, T2.1; no longer C23.2, J1.1, J1.2, J1.3, JP_PWR.2, SHUNTMON-A.RSN, T1.1
- net LOAD-NEG-B: now also C23.2, J1.1, J1.2, J1.3, SHUNTMON-A.RSN, T1.1; no longer C-TANT.1, C24.2, J4.1, J4.2, J4.3, SHUNTMON-B.RSN, T2.1
- net N$11: now also REF_SELECT_A.2, SHUNTMON-B.REFA, SHUNTMON-B.REFB; no longer REF_SELECT.2, SHUNTMON-A.REFA, SHUNTMON-A.REFB
- net REFINPUT: now also C15.1, REF_GND.1, REF_SELECT_A.1, SHUNTMON-A.REFA, SHUNTMON-A.REFB; no longer REF_SELECT.1, SHUNTMON-B.REFA, SHUNTMON-B.REFB
Other:
- note added: "ICSP"
- note added: "LED"
- note added: "Shunt Monitor A"
- note added: "Shunt Monitor B"
- note removed: "Shunt Amplifier A"
- note removed: "Shunt Amplifier B"
- moved on the sheet: ANT1, C10, C12, C19, C2, C20, C51, FTDI/UART, PAD1, R1, R2, R24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
