File: emonDCmini/emonDCmini v0.4.brd (EAGLE design)
At the start: 24.1 x 42.9 mm, 27 parts

Commit message: emonDCmini v0.4 sent to ragworm
Parts:
- removed LP3990: LP3990MF-3.3/NOPBMF05AL, LP3990:MF05AL
- removed R1, R4: 5.9K, rcl:R0603
- added RT9080: TPS73633DBVTG4, TSOT-23-5 REGULATOR 3.3v:SOT95P280X145-5N
- C4: value 1uF 16V -> 1uF CERAMIC
Connections:
- removed net +3V3: C22.2, ESP-12.16, MCP3202.8, R19.2, R6.2, R7.2, U$2.P$4
- net +5V: now also RT9080.1; no longer LP3990.1
- net 3.3V: now also C22.2, ESP-12.16, MCP3202.8, R19.2, R6.2, R7.2, RT9080.5, U$2.P$4; no longer LP3990.5
- net GND: now also RT9080.2; no longer LP3990.2
Routing:
- net 3.3V: track 1.93 -> 83.6 mm, vias 0 -> 7
- net +3V3: track 74.8 -> 0.00 mm, vias 7 -> 0
