File: emonDCmini/emonDCmini v0.4.sch (EAGLE design)
At the start: 26 parts

Commit message: emonDCmini v0.4 sent to ragworm
Parts:
- removed LP3990: LP3990MF-3.3/NOPBMF05AL, LP3990:LP3990MF-3.3/NOPBMF05AL
- removed R1, R4: 5.9K, rcl:R-EU_R0603
- added RT9080: TPS73633DBVTG4, TSOT-23-5 REGULATOR 3.3v:TPS73633DBVTG4
- C4: value 1uF 16V -> 1uF CERAMIC
Connections:
- removed net +3V3: C22.2, ESP-12.VCC, MCP3202.VDD/VREF, R19.2, R6.2, R7.2, U$2.VDD
- net +5V: now also RT9080.IN; no longer LP3990.VIN
- net 3.3V: now also C22.2, ESP-12.VCC, MCP3202.VDD/VREF, R19.2, R6.2, R7.2, RT9080.OUT, U$2.VDD; no longer LP3990.VOUT
- net GND: now also RT9080.GND; no longer LP3990.GND
Changed lines of the file:
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@@
 <part name="MCP3202" library="Microchip-MCP3202-BI_SN" deviceset="MCP3202-BI/SN" device=""/>
 <part name="P+1" library="supply1" deviceset="+5V" device=""/>
-<part name="LP3990" library="LP3990" deviceset="LP3990MF-3.3/NOPB" device="MF05AL" value="LP3990MF-3.3/NOPBMF05AL"/>
 <part name="P+2" library="SparkFun" deviceset="3.3V" device=""/>
 <part name="C3" library="rcl" deviceset="C-EU" device="C0603" value="1uF 16V"/>
-<part name="C4" library="rcl" deviceset="C-EU" device="C0603" value="1uF 16V"/>
+<part name="C4" library="rcl" deviceset="C-EU" device="C0603" value="1uF CERAMIC"/>
 <part name="GND4" library="supply1" deviceset="GND" device=""/>
 <part name="C5" library="rcl" deviceset="C-EU" device="C0603" value="10uF 16V"/>
 <part name="LMP8481" library="lmp8481b" deviceset="LMP8481" device="LMP8481-H" value="LMP8481-H"/>
 <part name="GND5" library="supply1" deviceset="GND" device=""/>
-<part name="R1" library="rcl" deviceset="R-EU_" device="R0603" value="5.9K">
-<attribute name="MPN" value=" MCWR06X5901FTL"/>
-</part>
-<part name="R4" library="rcl" deviceset="R-EU_" device="R0603" value="5.9K">
-<attribute name="MPN" value=" MCWR06X5901FTL"/>
-</part>
+<part name="RT9080" library="TSOT-23-5 REGULATOR 3.3v" deviceset="TPS73633DBVTG4" device=""/>
 </parts>
 <sheets>
@@
 <instance part="MCP3202" gate="A" x="104.14" y="342.9"/>
 <instance part="P+1" gate="1" x="-12.7" y="358.14"/>
-<instance part="LP3990" gate="A" x="-45.72" y="251.46"/>
 <instance part="P+2" gate="G$1" x="-22.86" y="256.54"/>
 <instance part="C3" gate="G$1" x="-66.04" y="251.46"/>
@@
 <instance part="LMP8481" gate="G$1" x="-10.16" y="335.28" rot="MR270"/>
 <instance part="GND5" gate="1" x="-2.54" y="353.06"/>
-<instance part="R1" gate="G$1" x="7.62" y="317.5" rot="R90">
-<attribute name="MPN" x="7.62" y="317.5" size="1.778" layer="96" rot="R90" display="off"/>
-</instance>
-<instance part="R4" gate="G$1" x="15.24" y="317.5" rot="R90">
-<attribute name="MPN" x="15.24" y="317.5" size="1.778" layer="96" rot="R90" display="off"/>
-</instance>
+<instance part="RT9080" gate="A" x="-43.18" y="259.08"/>
 </instances>
 <busses>
@@
 <pinref part="C1" gate="G$1" pin="2"/>
 <pinref part="GND2" gate="1" pin="GND"/>
-<pinref part="LP3990" gate="A" pin="GND"/>
 <wire x1="-60.96" y1="248.92" x2="-60.96" y2="243.84" width="0.1524" layer="91"/>
 <wire x1="-60.96" y1="243.84" x2="-66.04" y2="243.84" width="0.1524" layer="91"/>
@@
 <wire x1="-81.28" y1="246.38" x2="-81.28" y2="243.84" width="0.1524" layer="91"/>
 <junction x="-81.28" y="243.84"/>
+<pinref part="RT9080" gate="A" pin="GND"/>
 </segment>
 <segment>
@@
 </segment>
 </net>
-<net name="+3V3" class="0">
+<net name="+5V" class="0">
+<segment>
+<pinref part="P+1" gate="1" pin="+5V"/>
+<wire x1="-12.7" y1="350.52" x2="-12.7" y2="355.6" width="0.1524" layer="91"/>
+</segment>
+<segment>
+<pinref part="MAX5053" gate="A" pin="OUT"/>
+<wire x1="-86.36" y1="254" x2="-83.82" y2="254" width="0.1524" layer="91"/>
+<pinref part="C1" gate="G$1" pin="1"/>
+<pinref part="+3V1" gate="1" pin="+5V"/>
+<wire x1="-83.82" y1="254" x2="-81.28" y2="254" width="0.1524" layer="91"/>
+<wire x1="-81.28" y1="254" x2="-78.74" y2="254" width="0.1524" layer="91"/>
+<wire x1="-78.74" y1="254" x2="-78.74" y2="256.54" width="0.1524" layer="91"/>
+<junction x="-83.82" y="254"/>
+<wire x1="-78.74" y1="254" x2="-66.04" y2="254" width="0.1524" layer="91"/>
+<junction x="-78.74" y="254"/>
+<pinref part="C3" gate="G$1" pin="1"/>
+<wire x1="-66.04" y1="254" x2="-60.96" y2="254" width="0.1524" layer="91"/>
+<junction x="-66.04" y="254"/>
+<pinref part="C5" gate="G$1" pin="1"/>
+<junction x="-81.28" y="254"/>
+<pinref part="RT9080" gate="A" pin="IN"/>
+</segment>
+</net>
+<net name="3.3V" class="0">
+<segment>
+<pinref part="P+2" gate="G$1" pin="3.3V"/>
+<pinref part="C4" gate="G$1" pin="1"/>
+<junction x="-22.86" y="254"/>
+<wire x1="-25.4" y1="254" x2="-22.86" y2="254" width="0.1524" layer="91"/>
+<wire x1="-22.86" y1="254" x2="-22.86" y2="256.54" width="0.1524" layer="91"/>
+<pinref part="RT9080" gate="A" pin="OUT"/>
+<wire x1="-25.4" y1="261.62" x2="-25.4" y2="254" width="0.1524" layer="91"/>
+</segment>
 <segment>
 <wire x1="152.4" y1="238.76" x2="147.32" y2="238.76" width="0.1524" layer="91"/>
@@
 </segment>
 </net>
-<net name="+5V" class="0">
-<segment>
-<pinref part="P+1" gate="1" pin="+5V"/>
-<wire x1="-12.7" y1="350.52" x2="-12.7" y2="355.6" width="0.1524" layer="91"/>
-</segment>
-<segment>
-<pinref part="MAX5053" gate="A" pin="OUT"/>
-<wire x1="-86.36" y1="254" x2="-83.82" y2="254" width="0.1524" layer="91"/>
-<pinref part="C1" gate="G$1" pin="1"/>
-<pinref part="+3V1" gate="1" pin="+5V"/>
-<wire x1="-83.82" y1="254" x2="-81.28" y2="254" width="0.1524" layer="91"/>
-<wire x1="-81.28" y1="254" x2="-78.74" y2="254" width="0.1524" layer="91"/>
-<wire x1="-78.74" y1="254" x2="-78.74" y2="256.54" width="0.1524" layer="91"/>
-<junction x="-83.82" y="254"/>
-<pinref part="LP3990" gate="A" pin="VIN"/>
-<wire x1="-78.74" y1="254" x2="-66.04" y2="254" width="0.1524" layer="91"/>
-<junction x="-78.74" y="254"/>
-<pinref part="C3" gate="G$1" pin="1"/>
-<wire x1="-66.04" y1="254" x2="-60.96" y2="254" width="0.1524" layer="91"/>
-<junction x="-66.04" y="254"/>
-<pinref part="C5" gate="G$1" pin="1"/>
-<junction x="-81.28" y="254"/>
-</segment>
-</net>
-<net name="3.3V" class="0">
-<segment>
-<pinref part="LP3990" gate="A" pin="VOUT"/>
-<wire x1="-30.48" y1="254" x2="-22.86" y2="254" width="0.1524" layer="91"/>
-<pinref part="P+2" gate="G$1" pin="3.3V"/>
-<pinref part="C4" gate="G$1" pin="1"/>
-<junction x="-22.86" y="254"/>
-<wire x1="-22.86" y1="254" x2="-22.86" y2="256.54" width="0.1524" layer="91"/>
-</segment>
-</net>
