File: emonDCmini/emonDCmini v0.6.brd (EAGLE design)
At the start: 24.1 x 42.9 mm, 27 parts

Commit message: commit
Parts:
- removed C3: 1uF 16V, rcl:C0603
- removed C5: 10uF 16V, rcl:C0603
- removed JP1: (no value), jumper:JP1
- added S1: DTSM-3, switch-tact:DTSM-3
- C1: value 10uF 16V -> 10uF >70V CERAMIC
- C2: value 10uF >70V -> 22uF 6.3V K7R MLCC; device rcl:C0603 -> rcl:C1206
- moved C1 4.60 mm to (16.3, 42.8), flipped to the bottom
- moved C2 4.51 mm to (9.41, 41.8), flipped to the top
- moved R2 1.42 mm to (17.0, 40.6)
- moved R3 0.19 mm to (19.6, 41.0)
Connections:
- net +5V: now also C2.1; no longer C1.1, C3.1, C5.1
- net GND: now also S1.1; no longer C3.2, C5.2, JP1.1
- net GPIO0: now also S1.2; no longer JP1.2
- net SOURCE+: now also C1.1, MAX5053.2; no longer C2.1
Routing:
- net GND: track 23.8 -> 11.7 mm, vias 29 -> 28
- net +5V: track 36.4 -> 33.4 mm
- net RST: track 31.6 -> 34.1 mm
- net SOURCE+: track 33.8 -> 36.0 mm
- net ADC_VSENSE: track 15.3 -> 14.2 mm
- net GPIO0: track 13.8 -> 14.5 mm
Other:
- board text added: "SRC"
- board text removed: "SOURCE"

Commit message: commit
Parts:
- removed U$1: MOLEX_104031-0811, MOLEX MICRO SD [exposed pins]:MOLEX_MICROSD_EXPOSED
- added AB0815: AB0815_RTC, qfn16:QFN16
- added C3: 0.1uF CRMIC 100V, rcl:C0603
- added TFWF1-EBXX-1X0X: MICRO-SD3, TFWF1-EBXX-1X0X:TF-MICRO-SD_PP3*
- C1: value 10uF >70V CERAMIC -> (none); device rcl:C0603 -> rcl:C1206
- moved C1 0.43 mm to (15.9, 42.6)
- moved R3 0.40 mm to (19.5, 41.4), turned to 270 degrees
- moved R2 0.11 mm to (16.9, 40.5)
Connections:
- removed net GPIO16: ESP-12.12
- net 3.3V: now also TFWF1-EBXX-1X0X.4; no longer U$1.P$4
- net GND: now also C3.2, TFWF1-EBXX-1X0X.6, TFWF1-EBXX-1X0X.MT1, TFWF1-EBXX-1X0X.MT2, TFWF1-EBXX-1X0X.MT3, TFWF1-EBXX-1X0X.MT4; no longer U$1.CD1, U$1.CD2, U$1.GND1, U$1.GND2, U$1.GND3, U$1.GND4, U$1.P$6
- net GPIO12: now also TFWF1-EBXX-1X0X.7; no longer U$1.P$7
- net GPIO13: now also TFWF1-EBXX-1X0X.3; no longer U$1.P$3
- net GPIO14: now also TFWF1-EBXX-1X0X.5; no longer U$1.P$5
- net GPIO4: now also TFWF1-EBXX-1X0X.2; no longer U$1.P$2
- net GPIO5: no longer ESP-12.5
- net LOAD-: now also C3.1
Routing:
- net GPIO5: track 27.7 -> 0.00 mm, vias 1 -> 0
- net 3.3V: track 91.8 -> 112.8 mm, vias 8 -> 7
- net GPIO12: track 34.4 -> 16.8 mm, vias 4 -> 1
- net ESPTX: track 23.6 -> 30.7 mm
- net GPIO4: track 7.79 -> 14.3 mm
- net GPIO13: track 23.1 -> 17.6 mm
- net RESTESP: track 44.0 -> 49.1 mm
- net LOAD-: track 53.6 -> 56.8 mm
- net N$36: track 31.0 -> 34.1 mm, vias 4 -> 2
- net ADC_VSENSE: track 14.2 -> 13.3 mm
- net GPIO0: track 14.5 -> 15.3 mm
- net GND: vias 28 -> 19
