File: emonDCmini/emonDCmini v0.6.sch (EAGLE design)
At the start: 24 parts

Commit message: commit
Parts:
- removed U$1: MOLEX_104031-0811, MOLEX MICRO SD [exposed pins]:MOLEX_104031-0811
- added AB0815: AB0815_RTC, qfn16:AB0815_RTC
- added C3: 0.1uF CRMIC 100V, rcl:C-EUC0603
- added TFWF1-EBXX-1X0X: MICRO-SD3, TFWF1-EBXX-1X0X:MICRO-SD3
- C1: value 10uF >70V CERAMIC -> (none); device rcl:C-EUC0603 -> rcl:C-EUC1206
Connections:
- removed net GPIO16: ESP-12.GPIO16
- net 3.3V: now also TFWF1-EBXX-1X0X.4; no longer U$1.VDD
- net GND: now also C3.2, TFWF1-EBXX-1X0X.6, TFWF1-EBXX-1X0X.MT@1, TFWF1-EBXX-1X0X.MT@2, TFWF1-EBXX-1X0X.MT@3, TFWF1-EBXX-1X0X.MT@4; no longer U$1.CD1, U$1.CD2, U$1.GND, U$1.VSS
- net GPIO12: now also TFWF1-EBXX-1X0X.7; no longer U$1.DAT0
- net GPIO13: now also TFWF1-EBXX-1X0X.3; no longer U$1.CMD
- net GPIO14: now also TFWF1-EBXX-1X0X.5; no longer U$1.CLK
- net GPIO4: now also TFWF1-EBXX-1X0X.2; no longer U$1.CD/DAT3
- net GPIO5: no longer ESP-12.GPIO5
- net LOAD-: now also C3.1
Other:
- note added: "PINS FREE 15 5 16"
- note removed: "104031-0811"
- note removed: "PINS FREE 4 5 16"
