File: emonDCmini/emonDCmini v0.7 RTC.brd (EAGLE design)
At the start: 24.1 x 42.9 mm, 26 parts

Commit message: new boards and library files
Parts:
- MAX5033: value MAX5023TASA-T21-0111D_SBE-14-L -> MAX5033BUSA+; device MAX5053:21-0111D_SBE-14-L -> MAX5033:21-0111D_SBE-14
Connections:
- net GND: now also MAX5033.9; no longer MAX5033.EPAD
Changed lines of the file:
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@@
 <?xml version="1.0" encoding="utf-8"?>
 <!DOCTYPE eagle SYSTEM "eagle.dtd">
-<eagle version="7.7.0">
+<eagle version="8.3.2">
 <drawing>
 <settings>
 <setting alwaysvectorfont="no"/>
+<setting keepoldvectorfont="yes"/>
 <setting verticaltext="up"/>
 </settings>
@@
 <elements>
 <element name="LOGO1" library="ohw-logo" package="OSHW_6X200_NOTEXT" value="OSHW_LOGO_6MILX0200-NT" x="15.0274" y="4.0894" rot="MR0">
-<attribute name="OC_FARNELL" value="unknown" x="15.0274" y="4.0894" size="1.778" layer="28" rot="MR0" display="off"/>
 <attribute name="MF" value="" x="15.0274" y="4.0894" size="1.778" layer="28" rot="MR0" display="off"/>
 <attribute name="MPN" value="" x="15.0274" y="4.0894" size="1.778" layer="28" rot="MR0" display="off"/>
+<attribute name="OC_FARNELL" value="unknown" x="15.0274" y="4.0894" size="1.778" layer="28" rot="MR0" display="off"/>
 </element>
 <element name="R2" library="rcl" package="R0603" value="100K &gt;70V" x="16.931865625" y="40.451759375" smashed="yes" rot="MR0">
@@
 <attribute name="NAME" x="25.3492" y="13.6652" size="0.8128" layer="25" rot="R90"/>
 </element>
-<element name="MAX5033" library="MAX5053" package="21-0111D_SBE-14-L" value="MAX5023TASA-T21-0111D_SBE-14-L" x="16.9672" y="38.227" smashed="yes" rot="R90">
-<attribute name="VENDOR" value="MAXIM" x="16.9672" y="38.227" size="1.778" layer="27" rot="R90" display="off"/>
-<attribute name="MANUFACTURER_PART_NUMBER" value="max5033" x="16.9672" y="38.227" size="1.778" layer="27" rot="R90" display="off"/>
+<element name="MAX5033" library="MAX5033" package="21-0111D_SBE-14" value="MAX5033BUSA+" x="16.9672" y="38.227" smashed="yes" rot="R90">
+<attribute name="MANUFACTURER_PART_NUMBER" value="MAX5033BUSA+" x="16.9672" y="38.227" size="1.778" layer="27" rot="R90" display="off"/>
 <attribute name="NAME" x="13.7922" y="33.6804" size="1.016" layer="25" ratio="6" rot="SR0"/>
+<attribute name="VENDOR" value="MAXIM" x="16.9672" y="38.227" size="1.778" layer="27" rot="R90" display="off"/>
 </element>
 <element name="U$3" library="DRAGON_LOGO" package="DRAGON_LOGO_NOTEXT" value="" x="18.5928" y="6.5278" rot="MR0"/>
 <element name="EBW_SERIES_10.5" library="EBW series shunt" package="EBW_SERIES_10.5MM" value="EBW_SERIES_10.5MM" x="8.89" y="37.592" rot="MR90"/>
 <element name="MCP3202" library="Microchip-MCP3202-BI_SN" package="SOIC127P600X175-8N" value="MCP3202-BI/SN" x="18.1864" y="33.3502" smashed="yes" rot="MR270">
-<attribute name="PACKAGE" value="SOIC-8" x="18.1864" y="33.3502" size="1.778" layer="28" rot="MR270" display="off"/>
-<attribute name="OC_NEWARK" value="96K3721" x="18.1864" y="33.3502" size="1.778" layer="28" rot="MR270" display="off"/>
-<attribute name="SUPPLIER" value="Microchip" x="18.1864" y="33.3502" size="1.778" layer="28" rot="MR270" display="off"/>
 <attribute name="MPN" value="MCP3202-BI/SN" x="18.1864" y="33.3502" size="1.778" layer="28" rot="MR270" display="off"/>
 <attribute name="OC_FARNELL" value="1196803" x="18.1864" y="33.3502" size="1.778" layer="28" rot="MR270" display="off"/>
+<attribute name="OC_NEWARK" value="96K3721" x="18.1864" y="33.3502" size="1.778" layer="28" rot="MR270" display="off"/>
+<attribute name="PACKAGE" value="SOIC-8" x="18.1864" y="33.3502" size="1.778" layer="28" rot="MR270" display="off"/>
+<attribute name="SUPPLIER" value="Microchip" x="18.1864" y="33.3502" size="1.778" layer="28" rot="MR270" display="off"/>
 </element>
 <element name="C4" library="rcl" package="C0603" value="1uF MLCC" x="9.61025625" y="32.873925" smashed="yes">
@@
 </element>
 <element name="RT9080" library="TSOT-23-5 REGULATOR 3.3v" package="TSOT-23-5" value="RT9080-33GJ5" x="7.670846875" y="36.538678125" smashed="yes" rot="R270">
-<attribute name="PACKAGE" value="SOT-23-5" x="7.670846875" y="36.538678125" size="1.778" layer="27" rot="R270" display="off"/>
-<attribute name="OC_FARNELL" value="2679852" x="7.670846875" y="36.538678125" size="1.778" layer="27" rot="R270" display="off"/>
 <attribute name="NAME" x="4.9366125" y="39.0809625" size="1.016" layer="25" ratio="10" rot="SR270"/>
+<attribute name="OC_FARNELL" value="2679852" x="7.670846875" y="36.538678125" size="1.778" layer="27" rot="R270" display="off"/>
+<attribute name="PACKAGE" value="SOT-23-5" x="7.670846875" y="36.538678125" size="1.778" layer="27" rot="R270" display="off"/>
 <attribute name="VALUE" x="3.225846875" y="39.993078125" size="2.0828" layer="27" ratio="10" rot="SR270"/>
 </element>
@@
 <via x="14.0208" y="38.3032" extent="1-16" drill="0.5"/>
 <contactref element="LMP8481" pad="4"/>
-<wire x1="17.6022" y1="35.6235" x2="17.6022" y2="37.592" width="0.4064" layer="1"/>
+<wire x1="17.6022" y1="35.5727" x2="17.6022" y2="37.592" width="0.4064" layer="1"/>
 <via x="12.970871875" y="32.291315625" extent="1-16" drill="0.5"/>
 <via x="23.114" y="3.556" extent="1-16" drill="3.2"/>
@@
 <via x="4.018853125" y="36.1166625" extent="1-16" drill="0.5"/>
 <via x="9.684878125" y="36.5255375" extent="1-16" drill="0.5"/>
-<contactref element="MAX5033" pad="EPAD"/>
+<contactref element="MAX5033" pad="9"/>
 <contactref element="RT9080" pad="2"/>
 <contactref element="C2" pad="2"/>
@@
 <wire x1="8.89" y1="40.64" x2="8.89" y2="41.892" width="0.4064" layer="16"/>
 <wire x1="8.89" y1="42.6466" x2="8.89" y2="41.892" width="0.4064" layer="16"/>
-<wire x1="15.0622" y1="35.6235" x2="15.0622" y2="35.6108" width="0.4064" layer="1"/>
+<wire x1="15.0622" y1="35.5727" x2="15.0622" y2="35.6108" width="0.4064" layer="1"/>
 <wire x1="12.8778" y1="35.6616" x2="12.8778" y2="40.9956" width="0.4064" layer="1"/>
 <via x="12.8778" y="40.9956" extent="1-16" drill="0.5"/>
@@
 <wire x1="12.192" y1="40.17606875" x2="12.625778125" y2="40.17606875" width="0.6096" layer="16"/>
 <wire x1="12.995" y1="41.0366" x2="13.01446875" y2="41.0366" width="0.254" layer="16"/>
-<wire x1="15.0622" y1="35.6235" x2="15.0622" y2="35.6616" width="0.4064" layer="1"/>
+<wire x1="15.0622" y1="35.5727" x2="15.0622" y2="35.6616" width="0.4064" layer="1"/>
 <wire x1="15.0622" y1="35.6616" x2="12.8778" y2="35.6616" width="0.4064" layer="1"/>
 <contactref element="MAX5033" pad="2"/>
-<wire x1="15.0622" y1="35.6235" x2="16.3322" y2="35.6235" width="0.4064" layer="1"/>
+<wire x1="15.0622" y1="35.5727" x2="16.3322" y2="35.5727" width="0.4064" layer="1"/>
 <wire x1="12.86280625" y1="41.8645375" x2="13.01446875" y2="41.8645375" width="0.254" layer="16"/>
 <wire x1="13.01446875" y1="41.8645375" x2="13.01446875" y2="41.889346875" width="0.254" layer="16"/>
@@
 <wire x1="11.089034375" y1="37.932965625" x2="10.16" y2="38.862" width="0.4064" layer="1"/>
 <wire x1="8.610646875" y1="37.834078125" x2="8.633078125" y2="37.834078125" width="0.4064" layer="1"/>
-<wire x1="15.0622" y1="40.8305" x2="15.0622" y2="41.1187" width="0.4064" layer="1"/>
+<wire x1="15.0622" y1="40.8813" x2="15.0622" y2="41.1187" width="0.4064" layer="1"/>
 <wire x1="15.0622" y1="41.1187" x2="15.0153" y2="41.1187" width="0.4064" layer="1"/>
 <wire x1="15.0153" y1="41.1187" x2="13.97" y2="42.164" width="0.4064" layer="1"/>
@@
 <wire x1="11.089034375" y1="34.82151875" x2="11.620553125" y2="34.29" width="0.254" layer="1"/>
 <wire x1="11.620553125" y1="34.29" x2="18.8722" y2="34.29" width="0.254" layer="1"/>
-<wire x1="18.8722" y1="34.29" x2="18.8722" y2="35.6235" width="0.254" layer="1"/>
+<wire x1="18.8722" y1="34.29" x2="18.8722" y2="35.5727" width="0.254" layer="1"/>
 </signal>
 </signals>
