File: hardware/emonDCduo/emonDCduo-ESP v1.3.1.brd (EAGLE design)
At the start: 99.1 x 76.5 mm, 73 parts, among them J5 455-1750-1-ND, P1 B4B-PH-K, Y1 32Khz

Commit message: unzip firmware
Parts:
- C7: device rcl@1:C0603 -> rcl:C0603
- R1, R14: value 100K 75V -> 20.5k 0.25W
- R10, R11: device rcl@1:0309/12 -> rcl:0309/12
- R15, R2: value 5.6K -> 1.4k
- R20: value 57.6k -> 66.5k; device rcl@1:R0603 -> rcl:R0603
- R21, R9: device rcl@1:R0603 -> rcl:R0603
Routing:
- net SOURCE-POS-B: vias 33 -> 32
- net SOURCE-POS-A: vias 33 -> 32
- net LOAD-NEG-B: vias 32 -> 31
- net LOAD-NEG-A: vias 32 -> 31
- removed copper zone on layer 1, net LOAD-NEG-A
- removed copper zone on layer 16, net LOAD-NEG-A
- removed copper zone on layer 1, net LOAD-NEG-B
- removed copper zone on layer 16, net LOAD-NEG-B
- removed copper zone on layer 1, net SOURCE-POS-A
- removed copper zone on layer 16, net SOURCE-POS-A
- removed copper zone on layer 1, net SOURCE-POS-B
- removed copper zone on layer 16, net SOURCE-POS-B
Other:
- board text added: "v1.3 Dec 2017 by DB"
- board text removed: "v1.4 March 2018 by DB"
