File: hardware/emonDCduo/emonDCduo-ESP v1.3.1.sch (EAGLE design)
At the start: 73 parts, among them J5 455-1750-1-ND, P1 B4B-PH-K, Y1 32Khz

Commit message: unzip firmware
Parts:
- C7: device rcl@1:C-EUC0603 -> rcl:C-EUC0603
- R1, R14: value 100K 75V -> 20.5k 0.25W
- R10, R11: device rcl@1:R-EU_0309/12 -> rcl:R-EU_0309/12
- R15, R2: value 5.6K -> 1.4k
- R20: value 57.6k -> 66.5k; device rcl@1:R-EU_R0603 -> rcl:R-EU_R0603
- R21, R9: device rcl@1:R-EU_R0603 -> rcl:R-EU_R0603
Other:
- note added: "Daniel Bates Dec 2017"
- note added: "emonDC v1.3 : based on emonTx v3.4 by Glyn Hudson and Trystan Lea OpenEnergyMonitor.org"
- note removed: "designed by Daniel Bates March 2018"
- note removed: "emonDC v1.4 : based on emonTx v3.4 OpenEnergyMonitor.org"
Changed lines of the file:
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@@
 <?xml version="1.0" encoding="utf-8"?>
 <!DOCTYPE eagle SYSTEM "eagle.dtd">
-<eagle version="7.7.0">
+<eagle version="8.7.1">
 <drawing>
 <settings>
 <setting alwaysvectorfont="no"/>
+<setting keepoldvectorfont="yes"/>
 <setting verticaltext="up"/>
 </settings>
@@
 <part name="GND23" library="supply1" deviceset="0V" device="" value="GND"/>
 <part name="C13" library="rcl" deviceset="C-EU" device="C0603" value="0.1uF"/>
-<part name="REG2" library="burr-brown" deviceset="REG1117-VOUT4" device="" value="REG1117-3.3V">
+<part name="REG2" library="burr-brown" library_urn="urn:adsk.eagle:library:111" deviceset="REG1117-VOUT4" device="" value="REG1117-3.3V">
 <attribute name="MF" value="TEXAS INSTRUMENTS"/>
 <attribute name="MPN" value="REG1117-3.3"/>
@@
 <part name="C1T" library="rcl" deviceset="C-EU" device="C0603" value="10uF TANT"/>
 <part name="C18T" library="rcl" deviceset="C-EU" device="C0603" value="10uF TANT"/>
-<part name="R1" library="rcl" deviceset="R-EU_" device="R0603" value="100K 75V">
+<part name="R1" library="rcl" deviceset="R-EU_" device="R0603" value="20.5k 0.25W">
 <attribute name="MPN" value="MCWR06X1003FTL"/>
 </part>
-<part name="R2" library="rcl" deviceset="R-EU_" device="R0603" value="5.6K">
+<part name="R2" library="rcl" deviceset="R-EU_" device="R0603" value="1.4k">
 <attribute name="MPN" value=" MCWR06X5901FTL"/>
 </part>
@@
 <attribute name="OC_FARNELL" value="1593458"/>
 </part>
-<part name="R14" library="rcl" deviceset="R-EU_" device="R0603" value="100K 75V">
+<part name="R14" library="rcl" deviceset="R-EU_" device="R0603" value="20.5k 0.25W">
 <attribute name="MPN" value="MCWR06X1003FTL"/>
 </part>
-<part name="R15" library="rcl" deviceset="R-EU_" device="R0603" value="5.6K">
+<part name="R15" library="rcl" deviceset="R-EU_" device="R0603" value="1.4k">
 <attribute name="MPN" value=" MCWR06X5901FTL"/>
 </part>
@@
 </part>
 <part name="GND1" library="supply1" deviceset="GND" device=""/>
-<part name="R10" library="rcl@1" deviceset="R-EU_" device="0309/12" value="10K"/>
-<part name="R11" library="rcl@1" deviceset="R-EU_" device="0309/12" value="3.16K"/>
+<part name="R10" library="rcl" library_urn="urn:adsk.eagle:library:334" deviceset="R-EU_" device="0309/12" package3d_urn="urn:adsk.eagle:package:23571/1" value="10K"/>
+<part name="R11" library="rcl" library_urn="urn:adsk.eagle:library:334" deviceset="R-EU_" device="0309/12" package3d_urn="urn:adsk.eagle:package:23571/1" value="3.16K"/>
 <part name="SUPPLY7" library="supply1" deviceset="GND" device=""/>
-<part name="GPIO_1" library="con-lsta" deviceset="FE05-2" device=""/>
+<part name="GPIO_1" library="con-lsta" library_urn="urn:adsk.eagle:library:161" deviceset="FE05-2" device="" package3d_urn="urn:adsk.eagle:package:8170/1"/>
 <part name="+3V8" library="supply1" deviceset="+3V3" device=""/>
 <part name="GND6" library="supply1" deviceset="GND" device=""/>
@@
 <part name="Y1" library="microbuilder" deviceset="CRYSTAL" device="8X3.8SMT" value="32Khz"/>
 <part name="PCF8523" library="IotaWatt_parts" deviceset="PCF8523_RTC" device=""/>
-<part name="SUPPLY12" library="supply2" deviceset="GND" device=""/>
-<part name="C7" library="rcl@1" deviceset="C-EU" device="C0603" value="10uF"/>
-<part name="R9" library="rcl@1" deviceset="R-EU_" device="R0603" value="1K"/>
-<part name="SCREW1" library="con-weidmueller-sl35" deviceset="180-3" device=""/>
-<part name="SCREW2" library="con-weidmueller-sl35" deviceset="180-3" device=""/>
+<part name="SUPPLY12" library="supply2" library_urn="urn:adsk.eagle:library:372" deviceset="GND" device=""/>
+<part name="C7" library="rcl" library_urn="urn:adsk.eagle:library:334" deviceset="C-EU" device="C0603" package3d_urn="urn:adsk.eagle:package:23616/2" value="10uF"/>
+<part name="R9" library="rcl" library_urn="urn:adsk.eagle:library:334" deviceset="R-EU_" device="R0603" package3d_urn="urn:adsk.eagle:package:23555/2" value="1K"/>
+<part name="SCREW1" library="con-weidmueller-sl35" library_urn="urn:adsk.eagle:library:199" deviceset="180-3" device="" package3d_urn="urn:adsk.eagle:package:11339/1"/>
+<part name="SCREW2" library="con-weidmueller-sl35" library_urn="urn:adsk.eagle:library:199" deviceset="180-3" device="" package3d_urn="urn:adsk.eagle:package:11339/1"/>
 <part name="GND3" library="supply1" deviceset="0V" device="" value="GND"/>
 <part name="GND10" library="supply1" deviceset="0V" device="" value="GND"/>
@@
 <attribute name="MPN" value="Harwin S8411-45R"/>
 </part>
-<part name="ADC-PAD" library="wirepad" deviceset="2,15/1,0" device=""/>
+<part name="ADC-PAD" library="wirepad" library_urn="urn:adsk.eagle:library:412" deviceset="2,15/1,0" device="" package3d_urn="urn:adsk.eagle:package:30831/1"/>
 <part name="FTDI2" library="JeeLabs" deviceset="MA06-1" device="" value="FTDI"/>
 <part name="C2" library="rcl" deviceset="C-EU" device="C0603" value="100nF"/>
@@
 <attribute name="MPN" value="SRR1208-151YL"/>
 </part>
-<part name="R21" library="rcl@1" deviceset="R-EU_" device="R0603" value="13.3k"/>
-<part name="R20" library="rcl@1" deviceset="R-EU_" device="R0603" value="57.6k"/>
-<part name="REG1" library="burr-brown" deviceset="REG1117-VOUT4" device="" value="REG1117-5.0V">
+<part name="R21" library="rcl" library_urn="urn:adsk.eagle:library:334" deviceset="R-EU_" device="R0603" package3d_urn="urn:adsk.eagle:package:23555/2" value="13.3k"/>
+<part name="R20" library="rcl" library_urn="urn:adsk.eagle:library:334" deviceset="R-EU_" device="R0603" package3d_urn="urn:adsk.eagle:package:23555/2" value="66.5k"/>
+<part name="REG1" library="burr-brown" library_urn="urn:adsk.eagle:library:111" deviceset="REG1117-VOUT4" device="" value="REG1117-5.0V">
 <attribute name="MF" value="TEXAS INSTRUMENTS"/>
 <attribute name="MPN" value="REG1117-5.0"/>
@@
 <sheet>
 <plain>
-<text x="-82.55" y="184.15" size="1.778" layer="97">emonDC v1.4 : based on emonTx v3.4
+<text x="-82.55" y="184.15" size="1.778" layer="97">emonDC v1.3 : based on emonTx v3.4 by Glyn Hudson and Trystan Lea
 OpenEnergyMonitor.org</text>
-<text x="-82.55" y="180.34" size="1.778" layer="97">designed by Daniel Bates     March 2018</text>
+<text x="-82.55" y="180.34" size="1.778" layer="97">Daniel Bates     Dec 2017</text>
 <wire x1="38.1" y1="393.7" x2="38.1" y2="292.1" width="0.1524" layer="94"/>
 <wire x1="38.1" y1="393.7" x2="152.4" y2="393.7" width="0.1524" layer="94"/>
@@
 which will not be processed correctly with this version.
 </note>
+<note version="8.2" severity="warning">
+Since Version 8.2, EAGLE supports online libraries. The ids
+of those online libraries will not be understood (or retained)
+with this version.
+</note>
+<note version="8.3" severity="warning">
+Since Version 8.3, EAGLE supports URNs for individual library
+assets (packages, symbols, and devices). The URNs of those assets
+will not be understood (or retained) with this version.
+</note>
+<note version="8.3" severity="warning">
+Since Version 8.3, EAGLE supports the association of 3D packages
+with devices in libraries, schematics, and board files. Those 3D
+packages will not be understood (or retained) with this version.
+</note>
 </compatibility>
