File: hardware/emonDCduo/emonDCduo-ESP v1.4.brd (EAGLE design)
At the start: 99.1 x 76.5 mm, 73 parts, among them J5 455-1750-1-ND, P1 B4B-PH-K, Y1 32Khz

Commit message: unzip firmware
Parts:
- added GND: (no value), con-weidmueller-sl35:180-2
- C7: device rcl:C0603 -> rcl@1:C0603
- R10, R11: device rcl:0309/12 -> rcl@1:0309/12
- R20, R21, R9: device rcl:R0603 -> rcl@1:R0603
- moved R21 12.0 mm to (48.5, 76.2)
- moved R20 11.0 mm to (52.8, 76.2)
- moved SCREW_TERM_2 8.02 mm to (13.8, 32.3)
- moved SCREW_TERM_1 8.00 mm to (13.8, 51.3)
- moved L1 1.78 mm to (48.8, 68.6)
- moved C24 0.51 mm to (28.5, 37.2)
- moved C6 0.51 mm to (28.5, 27.3)
- moved R5 0.51 mm to (33.6, 34.4)
- moved SCREW2 0.51 mm to (23.3, 32.3)
- moved SHUNTMON-B 0.51 mm to (29.8, 32.3)
- moved C9 0.51 mm to (30.7, 27.3)
- moved R1 0.51 mm to (35.8, 29.0)
- moved R2 0.51 mm to (35.8, 25.7)
Connections:
- net GND: now also GND.1, GND.2; no longer SCREW1.2, SCREW2.2
Routing:
- net SOURCE-POS-A: track 68.3 -> 41.8 mm, vias 33 -> 30
- net LOAD-NEG-B: track 35.5 -> 9.89 mm, vias 32 -> 29
- net SOURCE-POS-B: track 81.6 -> 63.7 mm, vias 33 -> 30
- net LOAD-NEG-A: track 26.1 -> 10.4 mm, vias 32 -> 29
- net FB: track 26.0 -> 17.6 mm
- net GND: track 0.00 -> 6.93 mm, vias 45 -> 62
- net 6.5V: track 26.0 -> 30.7 mm
- net GPIO12: track 105.4 -> 106.3 mm
- net REF_B_INPUT: track 16.8 -> 17.7 mm
- net VSENSEB: track 55.7 -> 55.0 mm
- net 5.0V: track 171.2 -> 171.9 mm

Commit message: v1.4 changes. firmware dev.
Parts:
- moved R21 9.18 mm to (57.7, 75.4), turned to 270 degrees
- moved R20 8.77 mm to (61.5, 74.7)
- moved L1 0.76 mm to (48.8, 69.3)
- moved C3 0.25 mm to (62.1, 68.9)
Connections:
- net 5.0V: now also MCP3208.15
- net GND: no longer MCP3208.15
Routing:
- net 5.0V: track 171.9 -> 181.2 mm
- net FB: track 17.6 -> 23.5 mm
- net 6.5V: track 30.7 -> 27.5 mm
- net LX: track 18.2 -> 17.5 mm
- net SOURCE-POS-B: vias 30 -> 38
- net SOURCE-POS-A: vias 30 -> 38
- net LOAD-NEG-B: vias 29 -> 37
- net LOAD-NEG-A: vias 29 -> 37
- net GND: vias 62 -> 61
Other:
- board text added: "by DB"
- board text added: "v1.4 March 2018"
- board text removed: "v1.4 March 2018 by DB"
