File: hardware/emonDCduo/emonDCduo-ESP v1.4.sch (EAGLE design)
At the start: 73 parts, among them J5 455-1750-1-ND, P1 B4B-PH-K, Y1 32Khz

Commit message: commit
Other:
- note added: "note: VSENSE A & B changed to leaded resisted for end-user adaptation?"
Changed lines of the file:
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@@
 <?xml version="1.0" encoding="utf-8"?>
 <!DOCTYPE eagle SYSTEM "eagle.dtd">
-<eagle version="8.3.2">
+<eagle version="8.7.1">
 <drawing>
 <settings>
@@
 <layer number="102" name="Vscore" color="7" fill="1" visible="no" active="yes"/>
 <layer number="103" name="tMap" color="7" fill="1" visible="no" active="yes"/>
-<layer number="104" name="Name" color="7" fill="1" visible="no" active="yes"/>
+<layer number="104" name="Name" color="7" fill="1" visible="yes" active="yes"/>
 <layer number="105" name="tPlate" color="7" fill="1" visible="no" active="yes"/>
 <layer number="106" name="bPlate" color="7" fill="1" visible="no" active="yes"/>
@@
 https://github.com/boblemaire/IoTaWatt/</text>
 <text x="231.394" y="419.1" size="3.81" layer="91">SPI LCD DISPLAY</text>
+<text x="-91.44" y="293.878" size="1.778" layer="104">note: VSENSE A &amp; B changed to leaded resisted for end-user adaptation?</text>
 </plain>
 <instances>

Commit message: unzip firmware
Parts:
- added GND: (no value), con-weidmueller-sl35:180-2
- C7: device rcl:C-EUC0603 -> rcl@1:C-EUC0603
- R10, R11: device rcl:R-EU_0309/12 -> rcl@1:R-EU_0309/12
- R20, R21, R9: device rcl:R-EU_R0603 -> rcl@1:R-EU_R0603
Connections:
- net GND: now also GND.1, GND.2; no longer SCREW1.2, SCREW2.2
Other:
- note removed: "note: VSENSE A & B changed to leaded resisted for end-user adaptation?"
Changed lines of the file:
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@@
 <layer number="102" name="Vscore" color="7" fill="1" visible="no" active="yes"/>
 <layer number="103" name="tMap" color="7" fill="1" visible="no" active="yes"/>
-<layer number="104" name="Name" color="7" fill="1" visible="yes" active="yes"/>
+<layer number="104" name="Name" color="7" fill="1" visible="no" active="yes"/>
 <layer number="105" name="tPlate" color="7" fill="1" visible="no" active="yes"/>
 <layer number="106" name="bPlate" color="7" fill="1" visible="no" active="yes"/>
@@
 <part name="GND23" library="supply1" deviceset="0V" device="" value="GND"/>
 <part name="C13" library="rcl" deviceset="C-EU" device="C0603" value="0.1uF"/>
-<part name="REG2" library="burr-brown" library_urn="urn:adsk.eagle:library:111" deviceset="REG1117-VOUT4" device="" value="REG1117-3.3V">
+<part name="REG2" library="burr-brown" deviceset="REG1117-VOUT4" device="" value="REG1117-3.3V">
 <attribute name="MF" value="TEXAS INSTRUMENTS"/>
 <attribute name="MPN" value="REG1117-3.3"/>
@@
 </part>
 <part name="GND1" library="supply1" deviceset="GND" device=""/>
-<part name="R10" library="rcl" library_urn="urn:adsk.eagle:library:334" deviceset="R-EU_" device="0309/12" package3d_urn="urn:adsk.eagle:package:23571/1" value="10K"/>
-<part name="R11" library="rcl" library_urn="urn:adsk.eagle:library:334" deviceset="R-EU_" device="0309/12" package3d_urn="urn:adsk.eagle:package:23571/1" value="3.16K"/>
+<part name="R10" library="rcl@1" deviceset="R-EU_" device="0309/12" value="10K"/>
+<part name="R11" library="rcl@1" deviceset="R-EU_" device="0309/12" value="3.16K"/>
 <part name="SUPPLY7" library="supply1" deviceset="GND" device=""/>
-<part name="GPIO_1" library="con-lsta" library_urn="urn:adsk.eagle:library:161" deviceset="FE05-2" device="" package3d_urn="urn:adsk.eagle:package:8170/1"/>
+<part name="GPIO_1" library="con-lsta" deviceset="FE05-2" device=""/>
 <part name="+3V8" library="supply1" deviceset="+3V3" device=""/>
 <part name="GND6" library="supply1" deviceset="GND" device=""/>
@@
 <part name="Y1" library="microbuilder" deviceset="CRYSTAL" device="8X3.8SMT" value="32Khz"/>
 <part name="PCF8523" library="IotaWatt_parts" deviceset="PCF8523_RTC" device=""/>
-<part name="SUPPLY12" library="supply2" library_urn="urn:adsk.eagle:library:372" deviceset="GND" device=""/>
-<part name="C7" library="rcl" library_urn="urn:adsk.eagle:library:334" deviceset="C-EU" device="C0603" package3d_urn="urn:adsk.eagle:package:23616/2" value="10uF"/>
-<part name="R9" library="rcl" library_urn="urn:adsk.eagle:library:334" deviceset="R-EU_" device="R0603" package3d_urn="urn:adsk.eagle:package:23555/2" value="1K"/>
-<part name="SCREW1" library="con-weidmueller-sl35" library_urn="urn:adsk.eagle:library:199" deviceset="180-3" device="" package3d_urn="urn:adsk.eagle:package:11339/1"/>
-<part name="SCREW2" library="con-weidmueller-sl35" library_urn="urn:adsk.eagle:library:199" deviceset="180-3" device="" package3d_urn="urn:adsk.eagle:package:11339/1"/>
-<part name="GND3" library="supply1" deviceset="0V" device="" value="GND"/>
-<part name="GND10" library="supply1" deviceset="0V" device="" value="GND"/>
+<part name="SUPPLY12" library="supply2" deviceset="GND" device=""/>
+<part name="C7" library="rcl@1" deviceset="C-EU" device="C0603" value="10uF"/>
+<part name="R9" library="rcl@1" deviceset="R-EU_" device="R0603" value="1K"/>
+<part name="SCREW1" library="con-weidmueller-sl35" deviceset="180-3" device=""/>
+<part name="SCREW2" library="con-weidmueller-sl35" deviceset="180-3" device=""/>
 <part name="CR1220" library="IotaWatt_parts" deviceset="CR1220SMD" device="">
 <attribute name="MPN" value="Harwin S8411-45R"/>
 </part>
-<part name="ADC-PAD" library="wirepad" library_urn="urn:adsk.eagle:library:412" deviceset="2,15/1,0" device="" package3d_urn="urn:adsk.eagle:package:30831/1"/>
+<part name="ADC-PAD" library="wirepad" deviceset="2,15/1,0" device=""/>
 <part name="FTDI2" library="JeeLabs" deviceset="MA06-1" device="" value="FTDI"/>
 <part name="C2" library="rcl" deviceset="C-EU" device="C0603" value="100nF"/>
@@
 <attribute name="MPN" value="SRR1208-151YL"/>
 </part>
-<part name="R21" library="rcl" library_urn="urn:adsk.eagle:library:334" deviceset="R-EU_" device="R0603" package3d_urn="urn:adsk.eagle:package:23555/2" value="13.3k"/>
-<part name="R20" library="rcl" library_urn="urn:adsk.eagle:library:334" deviceset="R-EU_" device="R0603" package3d_urn="urn:adsk.eagle:package:23555/2" value="57.6k"/>
-<part name="REG1" library="burr-brown" library_urn="urn:adsk.eagle:library:111" deviceset="REG1117-VOUT4" device="" value="REG1117-5.0V">
+<part name="R21" library="rcl@1" deviceset="R-EU_" device="R0603" value="13.3k"/>
+<part name="R20" library="rcl@1" deviceset="R-EU_" device="R0603" value="57.6k"/>
+<part name="REG1" library="burr-brown" deviceset="REG1117-VOUT4" device="" value="REG1117-5.0V">
 <attribute name="MF" value="TEXAS INSTRUMENTS"/>
 <attribute name="MPN" value="REG1117-5.0"/>
@@
 <part name="RX" library="SparkFun" deviceset="M02" device="PTH"/>
 <part name="TX" library="SparkFun" deviceset="M02" device="PTH"/>
+<part name="GND" library="con-weidmueller-sl35" library_urn="urn:adsk.eagle:library:199" deviceset="180-2" device="" package3d_urn="urn:adsk.eagle:package:11334/1"/>
 </parts>
 <sheets>
@@
 https://github.com/boblemaire/IoTaWatt/</text>
 <text x="231.394" y="419.1" size="3.81" layer="91">SPI LCD DISPLAY</text>
-<text x="-91.44" y="293.878" size="1.778" layer="104">note: VSENSE A &amp; B changed to leaded resisted for end-user adaptation?</text>
 </plain>
 <instances>
@@
 <attribute name="VALUE" x="-101.6" y="330.454" size="1.778" layer="96"/>
 </instance>
-<instance part="GND3" gate="1" x="-93.98" y="332.74"/>
-<instance part="GND10" gate="1" x="-91.44" y="429.26"/>
 <instance part="CR1220" gate="G$1" x="210.82" y="342.9" rot="R270">
 <attribute name="MPN" x="210.82" y="342.9" size="1.778" layer="96" rot="R270" display="off"/>
@@
 <instance part="RX" gate="G$1" x="115.57" y="403.86" rot="R90"/>
 <instance part="TX" gate="G$1" x="113.03" y="421.64" rot="R270"/>
+<instance part="GND" gate="G$1" x="-116.84" y="223.52" rot="R270"/>
 </instances>
 <busses>
@@
 <wire x1="91.44" y1="231.14" x2="91.44" y2="226.06" width="0.1524" layer="91"/>
 <junction x="91.44" y="226.06"/>
+<wire x1="-101.6" y1="226.06" x2="-116.84" y2="226.06" width="0.1524" layer="91"/>
+<pinref part="GND" gate="G$1" pin="1"/>
+<wire x1="-116.84" y1="226.06" x2="-119.38" y2="226.06" width="0.1524" layer="91"/>
+<junction x="-116.84" y="226.06"/>
+<pinref part="GND" gate="G$1" pin="2"/>
 </segment>
 <segment>
@@
 </segment>
 <segment>
-<pinref part="SCREW1" gate="G$1" pin="2"/>
-<wire x1="-104.14" y1="432.816" x2="-91.44" y2="432.816" width="0.1524" layer="91"/>
-<wire x1="-91.44" y1="432.816" x2="-91.44" y2="431.8" width="0.1524" layer="91"/>
-<pinref part="GND10" gate="1" pin="0V"/>
-</segment>
-<segment>
-<pinref part="SCREW2" gate="G$1" pin="2"/>
-<wire x1="-104.14" y1="336.296" x2="-93.98" y2="336.296" width="0.1524" layer="91"/>
-<wire x1="-93.98" y1="336.296" x2="-93.98" y2="335.28" width="0.1524" layer="91"/>
-<pinref part="GND3" gate="1" pin="0V"/>
-</segment>
-<segment>

Commit message: v1.4 changes. firmware dev.
Connections:
- net 5.0V: now also MCP3208.VREF
- net GND: no longer MCP3208.VREF
Changed lines of the file:
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@@
 <part name="SUPPLY2" library="supply1" deviceset="GND" device=""/>
 <part name="SUPPLY3" library="supply1" deviceset="GND" device=""/>
-<part name="SUPPLY6" library="supply1" deviceset="GND" device=""/>
 <part name="R4" library="rcl" deviceset="R-EU_" device="R0603" value="1K">
 <attribute name="MPN" value=" MCWR06X5901FTL"/>
@@
 <instance part="SUPPLY2" gate="1" x="121.92" y="378.46" rot="R180"/>
 <instance part="SUPPLY3" gate="1" x="106.68" y="378.46" rot="R180"/>
-<instance part="SUPPLY6" gate="1" x="111.76" y="373.38" rot="R180"/>
 <instance part="R4" gate="G$1" x="152.4" y="355.6" rot="R90">
 <attribute name="MPN" x="152.4" y="355.6" size="1.778" layer="96" rot="R90" display="off"/>
@@
 </segment>
 <segment>
-<pinref part="MCP3208" gate="G$1" pin="VREF"/>
-<wire x1="111.76" y1="363.22" x2="111.76" y2="370.84" width="0.1524" layer="91"/>
-<pinref part="SUPPLY6" gate="1" pin="GND"/>
-</segment>
-<segment>
 <pinref part="R8" gate="G$1" pin="1"/>
 <wire x1="152.4" y1="335.28" x2="152.4" y2="330.2" width="0.1524" layer="91"/>
@@
 <wire x1="116.84" y1="363.22" x2="116.84" y2="375.92" width="0.1524" layer="91"/>
 <label x="116.84" y="375.92" size="1.778" layer="95" rot="R90"/>
-</segment>
-<segment>
+<pinref part="MCP3208" gate="G$1" pin="VREF"/>
+<wire x1="111.76" y1="363.22" x2="116.84" y2="363.22" width="0.1524" layer="91"/>
+<junction x="116.84" y="363.22"/>
+</segment>
+<segment>
