File: hardware/emonDCduo/emonDCduo-ESP v1.3.sch (EAGLE design)
At the start: 100 parts, among them P1 B4B-PH-K, X3 GMSTBV2, X4 GMSTBV2, Y1 32Khz

Commit message: commit v3.0 WIP
Parts:
- removed 3.3V_BAT, SJ4: (no value), jumper-con:SJ-CONCON
- removed C1, C8: 0.1uF 100V, rcl:C-EUC0603
- removed C19: 0.1uF, rcl:C-EUC0603
- removed C7T: 10uF, rcl@1:C-EUC0603
- removed CH_PD: (no value), SparkFun:M02PTH
- removed D2, D3, D4, D5, D6: P6SMB75A, diode:DIODE-DO214AA
- removed F1: 445/030_SERIES, LITTELFUSE 455:030 SERIES:445/030_SERIES
- removed GND: (no value), con-weidmueller-sl35_db:180-2
- removed IO16: FACTORY_RESET, SparkFun:M02PTH
- removed LED1: (no value), led:LEDCHIP-LED0805
- removed MH1, MH2, MH3, MH4: 5.3mm, holes-db:MOUNT-PAD-ROUND5.3
- removed R16, R22, R23, R24: 3R 0.5W 0.1%, rcl:R-EU_R0805
- removed R26: 1K, rcl:R-EU_R0603
- removed R27, R28: 10K, rcl:R-EU_R0603
- removed SJ1, SJ2, SJ3, SJ5, SJ6: (no value), jumper-con_db:SJ-CONCON
- removed TP1, TP2, TP3: TPPAD1-13, testpad:TPPAD1-13
- removed U1: (no value), microbuilder:LM358
- removed X3, X4: GMSTBV2, con-phoenix-762:GMSTBV2
- added C13, C14: 0.1uF, rcl:C-EUC0603
- added C26, C9: 100nF, rcl:C-EUC0603
- added C7: 10uF, rcl:C-EUC0603
- added IO1: (no value), SparkFun:M02PTH
- added R13, R5: 1K, rcl:R-EU_R0603
- added SCREW1, SCREW2: (no value), con-weidmueller-sl35:180-3
- added USB_PWR: 5000751517_SD, 5000751517_sd:5000751517_SD
- C10: value 100uF 80V -> 100uF 80V (LOW-ESR)
- C4, C5: value 0.1uF 16V -> 0.1uF 16V MLCC
- C48: value 0.1uF -> 0.1uF MLCC
- FTDI1: value FTDI_ESP -> FTDI
- FTDI2: value FTDI_RFM -> FTDI
- GPIO_1: device con-lsta-RFM69Pi:FE05-2_RFM69PI_OUTLINERFM69PI -> con-lsta:FE05-2
- J5: value (none) -> 455-1750-1-ND
- P1: device JST-PH:B4B-PH-K -> jst-ph:B4B-PH-K
- PCF8523: device emonDC parts:PCF8523_RTC -> IotaWatt_parts:PCF8523_RTC
- R1, R14: value 1M 100V -> 100K 75V
- R10: value 301k -> 10K; device rcl:R-EU_0204/7 -> rcl:R-EU_0309/12
- R11: value 5.23k -> 3.16K; device rcl:R-EU_0204/7 -> rcl:R-EU_0309/12
- R15, R2: value 56K -> 5.6K
- R17: value 1k -> 5.6K
- R18: value 2k -> 10K
- R20: value 43k -> 57.6k; device rcl@1:R-EU_R0603 -> rcl:R-EU_R0603
- R21: value 10k -> 13.3k; device rcl@1:R-EU_R0603 -> rcl:R-EU_R0603
- R9: device rcl@1:R-EU_R0603 -> rcl:R-EU_R0603
- REG1, REG2: device burr-brown-db:REG1117 -> burr-brown:REG1117-VOUT4
- SCREW_TERM_1, SCREW_TERM_2: device EBW series SHUNT:EBW_SERIES_15.2MM -> EBW series shunt:EBW_SERIES_15.2MM
- renumbered BOOT to BOOTL, FTDI_ESP to FTDI1, FTDI_RFM to FTDI2, MICRO_SD to U$4
Connections:
- net N$1 renamed FB
- removed net +3V3: 3.3V_BAT.1, GPIO_1.2, MCP3208.CH5, P1.3, R26.2, R27.1, R28.1, SJ2.1, SJ3.2, SJ6.2, U$4.VDD
- removed net +5V: FTDI1.4, FTDI2.4, R10.2, REG2.VIN, SJ1.2, SJ5.2, U1G$1.V+
- removed net 3.3V_PRE: C18T.1, REG2.VOUT, SJ6.1, TP2.TP
- removed net 5V_PRE: C1T.1, REG1.VOUT, SJ5.1, TP1.TP
- removed net ADCSHUNT_A: MCP3208.CH0, SHUNTMON-A.VOUT
- removed net ADCSHUNT_B: MCP3208.CH2, SHUNTMON-B.VOUT
- removed net GPIO16/RST: ESP-12.GPIO16, ESP-12.REST, IO16.1, R19.1
- removed net MCP_VCC: C19.1, MCP3208.VDD, MCP3208.VREF, SJ1.1
- removed net N$17: C1.1, C23.2, D2.C, R16.2, SHUNTMON-A.RSN
- removed net N$22: C24.2, C8.1, D4.C, R23.2, SHUNTMON-B.RSN
- removed net N$23: C1.2, C25.1, D3.C, R14.2, R22.2, SHUNTMON-A.RSP, SHUNTMON-A.VCC
- removed net N$24: R9.2, SJ2.2
- removed net N$5: LED1.A, R26.1
- removed net PRE_6.5V: C3.1, C48.1, L1.2, R20.2, SJ4.1, TP3.TP
- removed net SOURCE-POS-B_T: C6.1, C8.2, D5.C, R1.2, R24.2, SHUNTMON-B.RSP, SHUNTMON-B.VCC
- removed net VBAT: 3.3V_BAT.2, CR1220.P$+, PCF8523.VBAT
- removed net VCC_ESP: C22.2, ESP-12.VCC, R12.2, R19.2, R6.2, R7.2, SJ3.1
- removed net VSENSE_A: R14.1, R15.2, U1G$1.+IN
- removed net VSENSE_A_BUFF: MCP3208.CH1, U1G$1.-IN, U1G$1.OUT
- removed net VSENSE_B: R1.1, R2.2, U1G$2.+IN
- removed net VSENSE_B_BUFF: MCP3208.CH3, U1G$2.-IN, U1G$2.OUT
- removed net V_IN1: D6.C, F1.1, PWR.2
- removed net V_IN2: C10.1, C16.1, F1.2, REG0.ON/OFF, REG0.V_IN
- new net 3.3V: C13.1, C18T.1, C22.2, ESP-12.VCC, GPIO_1.2, IO1.2, MCP3208.CH5, P1.3, R12.2, R19.2, R6.2, R7.2, R9.2, REG2.VOUT, U$4.VDD
- new net 5.0V: C14.1, C1T.1, C26.1, C9.1, FTDI1.4, FTDI2.4, MCP3208.VDD, R10.2, REG1.VOUT, REG2.VIN, SHUNTMON-A.VCC, SHUNTMON-B.VCC, USB_PWR.1
- new net ADCSHUNT-A: MCP3208.CH0, R13.2
- new net ADCSHUNT-B: MCP3208.CH2, R5.2
- new net GPIO16: ESP-12.GPIO16, IO1.1
- new net N$4: R13.1, SHUNTMON-A.VOUT
- new net N$43: CR1220.P$+, PCF8523.VBAT
- new net N$6: R5.1, SHUNTMON-B.VOUT
- new net RESTESP: C21.1, ESP-12.REST, R19.1
- new net VSENSEA: MCP3208.CH1, R14.1, R15.2
- new net VSENSEB: MCP3208.CH3, R1.1, R2.2
- new net V_IN: C10.1, C16.1, PWR.2, REG0.ON/OFF, REG0.V_IN
- net 6.5V: now also C3.1, C48.1, L1.2, R20.2; no longer SJ4.2
- net CH_PD: no longer C21.1, CH_PD.1
- net GND: now also C13.2, C14.2, C26.2, C7.2, C9.2, MCP3208.VREF, R8.1, SCREW1.2, SCREW2.2, USB_PWR.5; no longer C19.2, C7T.2, CH_PD.2, D2.A, D3.A, D4.A, D5.A, D6.A, GND.1, GND.2, IO16.2, LED1.C, R8.2, U1G$1.V-
- net GPIO12: now also R4.1, R8.2; no longer R4.2, R8.1
- net GPIO12A: now also R4.2; no longer R4.1
- net LOAD-NEG-A: now also C23.2, SCREW1.1, SHUNTMON-A.RSN; no longer MH2.MOUNT, R16.1, X3-2.1
- net LOAD-NEG-B: now also C24.2, SCREW2.1, SHUNTMON-B.RSN; no longer MH4.MOUNT, R23.1, X4-2.1
- net N$10: now also C7.1; no longer C7T.1
- net SCL: no longer R27.2
- net SDA: no longer R28.2
- net SOURCE-POS-A: now also C25.1, R14.2, SCREW1.3, SHUNTMON-A.RSP; no longer MH1.MOUNT, R22.1, X3-1.1
- net SOURCE-POS-B: now also C6.1, R1.2, SCREW2.3, SHUNTMON-B.RSP; no longer MH3.MOUNT, R24.1, X4-1.1
Other:
- note added: "Daniel Bates Dec 2017"
- note added: "FACTORY RESET"
- note added: "emonDC v1.3 : based on emonTx v3.4 by Glyn Hudson and Trystan Lea OpenEnergyMonitor.org"
- note removed: "50mV MIN output desirable"
- note removed: "OVER-VOLTAGE PROTECTION"
- note removed: "REVERSE POLARITY PROTECTION"
- note removed: "TEMP SENSOR"
- note removed: "designed by Daniel Bates July 2018"
- note removed: "emonDC v2.0 based on emonTx and Heatpumpmonitor"
- moved on the sheet: ADC-PAD, C23, C24, C25, C3, C6, J5, L1, PWR, R1, R10, R11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
