File: hardware/emonDCduo/emonDCduo-ESP v2.4.sch (EAGLE design)
At the start: 109 parts, among them IC1 ACS758LCB-050B-PFF-T, IC2 ACS758LCB-050B-PFF-T, IC3 ACS758LCB-050B-PFF-T, IC4 ACS758LCB-050B-PFF-T, P1 B4B-PH-K, X3 GMSTBV2, X4 GMSTBV2, Y1 32Khz

Commit message: starting v3.0 and ASC770 breakout
Parts:
- removed IC1, IC2, IC3, IC4: ACS758LCB-050B-PFF-T, allegro:ACS758LCB-050B-PFF-T
- LED1: device led:LEDCHIP-LED0805 -> microbuilder:LED1206
- R10: value 16.56k -> 32k
- R11, R13: value 5.23k -> 10k
- R26: value 1K -> 390R
- R5: value 517.77k -> 1M
Changed lines of the file:
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@@
 <attribute name="MPN" value="C1608X7S2A104K080AB"/>
 </part>
-<part name="R10" library="rcl" library_urn="urn:adsk.eagle:library:334" deviceset="R-EU_" device="0204/7" package3d_urn="urn:adsk.eagle:package:23498/1" value="16.56k"/>
-<part name="R11" library="rcl" library_urn="urn:adsk.eagle:library:334" deviceset="R-EU_" device="0204/7" package3d_urn="urn:adsk.eagle:package:23498/1" value="5.23k"/>
+<part name="R10" library="rcl" library_urn="urn:adsk.eagle:library:334" deviceset="R-EU_" device="0204/7" package3d_urn="urn:adsk.eagle:package:23498/1" value="32k"/>
+<part name="R11" library="rcl" library_urn="urn:adsk.eagle:library:334" deviceset="R-EU_" device="0204/7" package3d_urn="urn:adsk.eagle:package:23498/1" value="10k"/>
 <part name="SUPPLY7" library="supply1" library_urn="urn:adsk.eagle:library:371" deviceset="GND" device=""/>
 <part name="F1" library="LITTELFUSE 455:030 SERIES" deviceset="445/030_SERIES" device=""/>
 <part name="C19" library="rcl" deviceset="C-EU" device="C0603" value="0.1uF"/>
-<part name="R26" library="rcl" library_urn="urn:adsk.eagle:library:334" deviceset="R-EU_" device="R0603" package3d_urn="urn:adsk.eagle:package:23555/2" value="1K"/>
-<part name="LED1" library="led" library_urn="urn:adsk.eagle:library:259" deviceset="LED" device="CHIP-LED0805" package3d_urn="urn:adsk.eagle:package:15818/2"/>
+<part name="R26" library="rcl" library_urn="urn:adsk.eagle:library:334" deviceset="R-EU_" device="R0603" package3d_urn="urn:adsk.eagle:package:23555/2" value="390R"/>
+<part name="LED1" library="microbuilder" deviceset="LED" device="1206"/>
 <part name="SJ1" library="jumper-con_db" deviceset="SJ-CON" device="CON"/>
 <part name="SJ2" library="jumper-con_db" deviceset="SJ-CON" device="CON"/>
@@
 <part name="D7" library="diode" library_urn="urn:adsk.eagle:library:210" deviceset="DIODE-" device="DO214AA" package3d_urn="urn:adsk.eagle:package:43433/2" value="P6SMB75A"/>
 <part name="C7" library="rcl" deviceset="C-EU" device="C0603" value="0.1uF"/>
-<part name="R5" library="rcl7" deviceset="R-EU_" device="R0603" value="517.77k"/>
-<part name="R13" library="rcl7" deviceset="R-EU_" device="R0603" value="5.23k"/>
+<part name="R5" library="rcl7" deviceset="R-EU_" device="R0603" value="1M"/>
+<part name="R13" library="rcl7" deviceset="R-EU_" device="R0603" value="10k"/>
 <part name="SUPPLY4" library="supply1" library_urn="urn:adsk.eagle:library:371" deviceset="GND" device=""/>
 <part name="C9" library="rcl" deviceset="C-EU" device="C0603" value="0.1uF"/>
 <part name="SJ7" library="jumper" library_urn="urn:adsk.eagle:library:252" deviceset="SJ" device="" package3d_urn="urn:adsk.eagle:package:15471/1"/>
-<part name="IC1" library="allegro" library_urn="urn:adsk.eagle:library:93" deviceset="ACS758*" device="" package3d_urn="urn:adsk.eagle:package:3449/1" technology="LCB-050B-PFF-T"/>
-<part name="IC2" library="allegro" library_urn="urn:adsk.eagle:library:93" deviceset="ACS758*" device="" package3d_urn="urn:adsk.eagle:package:3449/1" technology="LCB-050B-PFF-T"/>
-<part name="IC3" library="allegro" library_urn="urn:adsk.eagle:library:93" deviceset="ACS758*" device="" package3d_urn="urn:adsk.eagle:package:3449/1" technology="LCB-050B-PFF-T"/>
-<part name="IC4" library="allegro" library_urn="urn:adsk.eagle:library:93" deviceset="ACS758*" device="" package3d_urn="urn:adsk.eagle:package:3449/1" technology="LCB-050B-PFF-T"/>
 </parts>
 <sheets>
@@
 <attribute name="VALUE" x="119.38" y="443.23" size="1.778" layer="96" rot="R180"/>
 </instance>
-<instance part="IC1" gate="G$1" x="-154.94" y="276.86" smashed="yes">
-<attribute name="NAME" x="-157.48" y="285.75" size="1.778" layer="95"/>
-<attribute name="VALUE" x="-157.48" y="266.7" size="1.778" layer="96"/>
-</instance>
-<instance part="IC2" gate="G$1" x="-154.94" y="248.92" smashed="yes">
-<attribute name="NAME" x="-157.48" y="257.81" size="1.778" layer="95"/>
-<attribute name="VALUE" x="-157.48" y="238.76" size="1.778" layer="96"/>
-</instance>
-<instance part="IC3" gate="G$1" x="-154.94" y="218.44" smashed="yes">
-<attribute name="NAME" x="-157.48" y="227.33" size="1.778" layer="95"/>
-<attribute name="VALUE" x="-157.48" y="208.28" size="1.778" layer="96"/>
-</instance>
-<instance part="IC4" gate="G$1" x="-154.94" y="187.96" smashed="yes">
-<attribute name="NAME" x="-157.48" y="196.85" size="1.778" layer="95"/>
-<attribute name="VALUE" x="-157.48" y="177.8" size="1.778" layer="96"/>
-</instance>
 </instances>
 <busses>
@@
 <wire x1="30.48" y1="226.06" x2="50.8" y2="226.06" width="0.1524" layer="91"/>
 <wire x1="50.8" y1="226.06" x2="71.12" y2="226.06" width="0.1524" layer="91"/>
-<wire x1="71.12" y1="226.06" x2="91.44" y2="226.06" width="0.1524" layer="91"/>
-<wire x1="91.44" y1="226.06" x2="114.3" y2="226.06" width="0.1524" layer="91"/>
+<wire x1="71.12" y1="226.06" x2="114.3" y2="226.06" width="0.1524" layer="91"/>
 <wire x1="129.54" y1="226.06" x2="114.3" y2="226.06" width="0.1524" layer="91"/>
 <junction x="129.54" y="226.06"/>
@@
 <wire x1="-101.6" y1="226.06" x2="-109.22" y2="226.06" width="0.1524" layer="91"/>
 <pinref part="GND" gate="G$1" pin="1"/>
-<wire x1="-109.22" y1="226.06" x2="-119.38" y2="226.06" width="0.1524" layer="91"/>
-<wire x1="-119.38" y1="226.06" x2="-124.46" y2="226.06" width="0.1524" layer="91"/>
+<wire x1="-109.22" y1="226.06" x2="-124.46" y2="226.06" width="0.1524" layer="91"/>
 <wire x1="-124.46" y1="226.06" x2="-127" y2="226.06" width="0.1524" layer="91"/>
 <junction x="-124.46" y="226.06"/>
 <pinref part="GND" gate="G$1" pin="2"/>
 <pinref part="LED1" gate="G$1" pin="C"/>
-<wire x1="167.64" y1="231.14" x2="167.64" y2="226.06" width="0.1524" layer="91"/>
+<wire x1="170.18" y1="236.22" x2="167.64" y2="226.06" width="0.1524" layer="91"/>
 <wire x1="167.64" y1="226.06" x2="147.32" y2="226.06" width="0.1524" layer="91"/>
 <wire x1="-12.7" y1="226.06" x2="0" y2="226.06" width="0.1524" layer="91"/>
@@
 <pinref part="LED1" gate="G$1" pin="A"/>
 <wire x1="165.1" y1="243.84" x2="167.64" y2="243.84" width="0.1524" layer="91"/>
-<wire x1="167.64" y1="243.84" x2="167.64" y2="238.76" width="0.1524" layer="91"/>
-</segment>
-</net>
+<wire x1="167.64" y1="243.84" x2="162.56" y2="236.22" width="0.1524" layer="91"/>
+</segment>
+</net>

Commit message: commit v3.0
Parts:
- C11T, C18T, C1T: device rcl:C-EUC0603 -> rcl7:CPOL-EUC0603POL
- C7T: device rcl@1:C-EUC0603 -> rcl7:CPOL-EUC0603POL
- R10, R11: device rcl:R-EU_0204/7 -> rcl7:R-EU_0207/10
- R16, R22, R23, R24: device rcl:R-EU_R0805 -> rcl7:R-EU_R1206
- renumbered U1 to LM258
Connections:
- removed net CH6: J5.2, MCP3208.CH6
- net +3V3: now also MCP3208.CH6
- net 3.3V_PRE: now also C18T.+; no longer C18T.1
- net 5V_PRE: now also C1T.+; no longer C1T.1
- net 6.5V: now also C11T.+; no longer C11T.1
- net GND: now also C11T.-, C18T.-, C1T.-, C7T.-, J5.2; no longer C11T.2, C18T.2, C1T.2, C7T.2
- net N$10: now also C7T.+; no longer C7T.1
