File: hardware/emonDCduo/emonDCduo-ESP v3.0.brd (EAGLE design)
At the start: 114.2 x 76.5 mm, 106 parts, among them P1 B4B-PH-K, Y1 32Khz

Commit message: commit v3.1
Parts:
- removed C18T: 10uF TANT, rcl7:C0603POL
- removed C20: 1nF, rcl:C0603
- removed C21, C22: 100nF, rcl:C0603
- removed C23, C24, C25: 0.1uF 100V, rcl:C0603
- removed C7T: 10uF, rcl7:C0603POL
- removed MOUNT_7.62_A, MOUNT_7.62_B: GMSTBV2, con-phoenix-762:GMSTBV2
- removed R18: 2k, rcl:R0603
- removed R26: 174R, rcl:R0603
- removed R27, R28: 10K, rcl:R0603
- removed SJ3: (no value), jumper-con_db:SJ-CON
- added C10, C16, C9: 1nF, rcl:C0603
- added C2, C3, C4, C5, C7: 0.1uF 100V, rcl:C0603
- added C32T, C33T: 10uF TANT, rcl7:C0603POL
- added R11, R20, R21: 10K, rcl:R0603
- added R22: 1K, rcl@1:R0603
- added TP10, TP11, TP8, TP9: TPPAD1-13Y, testpad:P1-13Y
- C17, C18: value 1nF -> 0.1uF
- LED1: value (none) -> PWR_ON
- R10: value 174R -> 2K; device rcl7:0207/10 -> rcl:R0603
- R13: value 10k -> 10K; device rcl7:0207/10 -> rcl:R0603
- R14: value 1M 100V -> 1k
- R15: value 56K -> 2k
- R17: value 1k -> 10K
- R3: value 10K -> 1M 100V
- R4: value 1K -> 56K
- R5: value 5.6k -> 174R; device rcl7:0207/10 -> rcl:R0603
- R6: value 10K -> 10k; device rcl:R0603 -> rcl7:0207/10
- R7: value 10K -> 5.6k; device rcl:R0603 -> rcl7:0207/10
- R8: value 2K -> 174R; device rcl:R0603 -> rcl7:0207/10
- R9: device rcl@1:R0603 -> rcl:R0603
- SJ2: device jumper-con_db:SJ-CON -> jumper:SJ
- UART: value UART_ESP -> UART
- moved R14 35.4 mm to (62.3, 14.3), turned to 0 degrees
- moved R13 34.5 mm to (62.3, 18.6)
- moved R15 34.2 mm to (62.3, 12.1), turned to 180 degrees
- moved C17 34.0 mm to (85.4, 26.3), flipped to the top, turned to 270 degrees
- moved C18 33.1 mm to (85.8, 20.6), flipped to the top, turned to 90 degrees
- moved R6 32.9 mm to (89.5, 38.6)
- moved R4 30.7 mm to (53.0, 18.0), turned to 90 degrees
- moved R9 30.5 mm to (73.4, 42.9), flipped to the top
- moved R5 27.0 mm to (103.9, 59.4), turned to 180 degrees
- moved R1 24.8 mm to (50.5, 45.9)
- moved R17 24.1 mm to (86.4, 14.2)
- moved R7 21.3 mm to (89.5, 35.3)
- moved R8 19.6 mm to (89.5, 32.0), turned to 0 degrees
- moved R2 19.1 mm to (50.5, 41.0)
- moved Y1 16.8 mm to (49.3, 5.17)
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- renumbered C11T to C30T, C1T to C31T, D7 to D1, R19 to R16, UART_ESP to UART
Connections:
- removed net N$24: R9.2, SJ2.2
- removed net VCC_ESP: C22.2, ESP-12.16, R12.2, R16.2, R6.2, R7.2, SJ3.1
- new net VDD_RTC_POSTJUMPER: R20.1, R21.1, R22.2, SJ2.2
- net +3V3: now also C15.1, C17.2, ESP-12.16, R12.2, R13.2, R16.2, R17.2, R5.2; no longer C18.1, R26.2, R27.1, R28.1, SJ3.2
- net +5V: now also R6.2; no longer R13.2
- net 3.3V_PRE: now also C32T.1; no longer C18T.1
- net ADCSHUNT_A: now also C9.1; no longer C17.1
- net ADCSHUNT_B: now also C11.1; no longer C12.1
- net BI_REF: now also C13.1, R6.1, R7.2; no longer C14.1, R13.1, R5.2
- net CH7: now also C16.1; no longer C20.1
- net CH_PD: now also C18.1, R17.1; no longer C21.1, R7.1
- net ESPRX: now also R14.2, R15.1; no longer R17.2, R18.1
- net GND: now also C1.2, C17.1, C3.2, C32T.2, C33T.2, C4.2, C7.2, C8.2, R10.2, R11.2, R15.2, R4.1, R8.1; no longer C18T.2, C22.1, C23.1, C24.1, C25.2, C7T.2, R10.1, R15.1, R18.2, R3.2, R8.2
- net GPIO0: now also R13.1; no longer R12.1
- net GPIO12: now also R10.1, R9.2; no longer R4.2, R8.1
- net GPIO12A: now also R9.1; no longer R4.1
- net GPIO15: now also R11.1; no longer R3.1
- net GPIO2: now also R12.1; no longer R6.1
- net LOAD-NEG-A: now also TP11.TP; no longer MOUNT_7.62_B.2
- net LOAD-NEG-A_T: now also C2.1; no longer C23.2
- net LOAD-NEG-B: now also TP9.TP; no longer MOUNT_7.62_A.2
- net LOAD-NEG-B_T: now also C4.1, C5.1; no longer C24.2, C8.1
- net N$36: now also R14.1; no longer R17.1
- net N$5: now also R5.1; no longer R26.1
- net REF_A_INPUT: now also C7.1
- net REF_B_INPUT: now also C8.1
- net RESET: now also C18.2; no longer C21.2
- net SCL: no longer R27.2
- net SDA: no longer R28.2
- net SOURCE-POS-A: now also TP10.TP; no longer MOUNT_7.62_B.1
- net SOURCE-POS-A_T: now also C2.2, C3.1, R1.2; no longer C1.2, C25.1, R14.2
- net SOURCE-POS-B: now also TP8.TP; no longer MOUNT_7.62_A.1
- net SOURCE-POS-B_T: now also C5.2, R3.2; no longer C8.2, R1.2
- net UNI_REF: now also C14.1, R7.1, R8.2; no longer C15.1, R10.2, R5.1
- net VDD_PCF: now also C33T.1, R22.1; no longer C7T.1, R9.1
- net VSENSE_A: now also R1.1, R2.2; no longer R14.1, R15.2
- net VSENSE_A_BUFF: now also C10.1; no longer C11.1
- net VSENSE_B: now also R3.1, R4.2; no longer R1.1, R2.2
- net VSENSE_B_BUFF: now also C12.1; no longer C13.1
Routing:
- net +3V3: track 24.9 -> 172.3 mm, vias 1 -> 8
- net +5V: track 17.6 -> 113.2 mm, vias 1 -> 8
- net GPIO14: track 0.00 -> 82.7 mm, vias 0 -> 6
- net GPIO12: track 1.84 -> 79.1 mm, vias 0 -> 6
- net GPIO13: track 0.00 -> 71.4 mm, vias 0 -> 7
- net UNI_REF: track 13.2 -> 81.1 mm, vias 0 -> 3
- net BI_REF: track 16.1 -> 79.0 mm, vias 0 -> 5
- net ESPTX: track 0.00 -> 52.8 mm, vias 0 -> 1
- net ESPRX: track 0.00 -> 46.8 mm, vias 0 -> 2
- net GPIO15: track 0.00 -> 31.6 mm
- net GPIO2: track 0.00 -> 28.6 mm, vias 0 -> 2
- net VSENSE_B: track 0.00 -> 25.2 mm, vias 0 -> 2
- net ADCSHUNT_B: track 0.00 -> 25.1 mm, vias 0 -> 3
- net 3.3V_PRE: track 12.6 -> 37.4 mm
- net D0/RX: track 0.00 -> 24.0 mm
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Other:
- board text added: "5x20"
- board text added: "Open Hardware"
- board text added: "PWR_ON"
- board text added: "TR5 FUSES"
- board text removed: "EN"
- board text removed: "Open-Hardware"
- board text removed: "RESET"
