File: hardware/emonDCduo/emonDCduo-ESP v3.1.sch (EAGLE design)
At the start: 101 parts, among them P1 B4B-PH-K, X3 GMSTBV2, X4 GMSTBV2, Y1 32Khz

Commit message: commit v3.1
Parts:
- removed C11T, C18T, C1T: 10uF TANT, rcl:C-EUC0603
- removed C23, C24, C25: 0.1uF 100V, rcl:C-EUC0603
- removed C48: 0.1uF, rcl:C-EUC0603
- removed C7T: 10uF, rcl@1:C-EUC0603
- removed D6: P6SMB75A, diode:DIODE-DO214AA
- removed FTDI_RFM: FTDI_RFM, JeeLabs:MA06-1
- removed L1: SRR1208, inductor-bourns:SRR1208
- removed R18: 2k, rcl:R-EU_R0603
- removed R19, R27, R28: 10K, rcl:R-EU_R0603
- removed R23, R24: 3R 0.5W 0.1%, rcl:R-EU_R0805
- removed R25: (no value), sensor-heraeus:3220824X
- removed R26: 1K, rcl:R-EU_R0603
- removed REG0: MAX5035, MAX5035:MAX5035
- removed SJ3: (no value), jumper-con_db:SJ-CONCON
- removed X3, X4: GMSTBV2, con-phoenix-762:GMSTBV2
- added 7.62_BARRIER: GMSTBA2, con-phoenix-762:GMSTBA2
- added C11, C12, C13, C14, C15, C9: 1nF, rcl:C-EUC0603
- added C30T, C31T, C32T, C33T: 10uF TANT, rcl7:CPOL-EUC0603POL
- added C7: 0.1uF 100V, rcl:C-EUC0603
- added F2, F3, F4, F5: (no value), fuse:TR5
- added MOUNT_10.16_A, MOUNT_10.16_B: MOLEX_39970-003, 10.16mm terminal block:MOLEX_39970-003
- added R13: 10K, rcl:R-EU_R0603
- added R5: 174R, rcl:R-EU_R0603
- added TP10, TP11, TP4, TP5, TP6, TP7, TP8, TP9: TPPAD1-13Y, testpad:TPPAD1-13Y
- C10: value 100uF 80V -> 1nF; device Panasonic-EEE-EEV-EEF-ECQ:EEV-FK1K101Q-CASE-H13 -> rcl:C-EUC0603
- C16: value 0.1uF 100V -> 1nF
- C17, C18: value 100nF -> 0.1uF
- C2: value 100nF -> 0.1uF 100V; MPN (none) -> C1608X7S2A104K080AB
- C3: value 470uF 16V -> 0.1uF 100V; device Panasonic-EEEFK_EEEFP:EEE-FK1C471P-CASE-F -> rcl:C-EUC0603; MPN (none) -> C1608X7S2A104K080AB
- C4, C5: value 0.1uF 16V -> 0.1uF 100V; MPN (none) -> C1608X7S2A104K080AB
- D1: value MBRS1100T3G -> P6SMB75A; device diodes:MBRS1100T3G -> diode:DIODE-DO214AA; MPN MBRS1100T3G -> (none)
- LED1: value (none) -> PWR_ON; device led:LEDCHIP-LED0805 -> microbuilder:LED1206
- R10: value 301k -> 2K; device rcl:R-EU_0204/7 -> rcl:R-EU_R0603; MPN (none) -> MCWR06X5901FTL
- R11: value 5.23k -> 10K; device rcl:R-EU_0204/7 -> rcl:R-EU_R0603
- R14: value 1M 100V -> 1k; MPN MCWR06X1003FTL -> (none)
- R15: value 56K -> 2k; MPN MCWR06X5901FTL -> (none)
- R16: value 3R 0.5W 0.1% -> 10K; device rcl:R-EU_R0805 -> rcl:R-EU_R0603
- R17: value 1k -> 10K
- R20: value 43k -> 10K; device rcl@1:R-EU_R0603 -> rcl:R-EU_R0603
- R21: value 10k -> 10K; device rcl@1:R-EU_R0603 -> rcl:R-EU_R0603
- R22: value 3R 0.5W 0.1% -> 1K; device rcl:R-EU_R0805 -> rcl@1:R-EU_R0603
- R3: value 10K -> 1M 100V; MPN (none) -> MCWR06X1003FTL
- R4: value 1K -> 56K
- R6: value 10K -> 10k; device rcl:R-EU_R0603 -> rcl7:R-EU_0207/10
- R7: value 10K -> 5.6k; device rcl:R-EU_R0603 -> rcl7:R-EU_0207/10
- R8: value 2K -> 174R; device rcl:R-EU_R0603 -> rcl7:R-EU_0207/10; MPN MCWR06X5901FTL -> (none)
- R9: device rcl@1:R-EU_R0603 -> rcl:R-EU_R0603; MPN (none) -> MCWR06X5901FTL
- SJ2: device jumper-con_db:SJ-CONCON -> jumper:SJ
- UART: value FTDI_ESP -> UART
- renumbered ADC-PAD to ADC, BOOT to ESPBOOT, C21 to C18, C22 to C17, FTDI_ESP to UART, SCREW_TERM_1 to EBW_B, SCREW_TERM_2 to EBW_A, U1 to LM258
Connections:
- net N$30 renamed RESET
- removed net BST: C4.1, REG0.BST
- removed net CH6: J5.2, MCP3208.CH6
- removed net GPIO16/RST: ESP-12.GPIO16, ESP-12.REST, IO16.1, R19.1
- removed net LX: C4.2, D1.C, L1.1, REG0.LX/OUT
- removed net MCP_VCC: C19.1, MCP3208.VDD, MCP3208.VREF, SJ1.1
- removed net N$10: C7T.1, PCF8523.VDD, R9.1
- removed net N$17: C1.1, C23.2, D2.C, R16.2, SHUNTMON-A.RSN
- removed net N$20: FTDI_RFM.5
- removed net N$22: C24.2, C8.1, D4.C, R23.2, SHUNTMON-B.RSN
- removed net N$23: C1.2, C25.1, D3.C, R14.2, R22.2, SHUNTMON-A.RSP, SHUNTMON-A.VCC
- removed net N$24: R9.2, SJ2.2
- removed net N$301: C2.2, FTDI_RFM.1
- removed net PRE_6.5V: C3.1, C48.1, L1.2, R20.2, SJ4.1, TP3.TP
- removed net REF_INPUT: MCP3208.CH4, R10.1, R11.2, REF_SEL_A.3, REF_SEL_B.3
- removed net VCC_ESP: C17.2, ESP-12.VCC, R12.2, R19.2, R6.2, R7.2, SJ3.1
- removed net VD: C5.1, REG0.VD
- removed net V_IN1: D6.C, F1.1, PWR.2
- removed net V_IN2: C10.1, C16.1, F1.2, REG0.ON/OFF, REG0.V_IN
- new net BI_REF: C13.1, MCP3208.CH4, R6.1, R7.2, REF_SEL_A.3, REF_SEL_B.3
- new net GPIO16: ESP-12.GPIO16, IO16.1, SJ1.2
- new net LOAD-NEG-A_T: C1.1, C2.1, D2.C, F2.2, SHUNTMON-A.RSN
- new net LOAD-NEG-B_T: C4.1, C5.1, D4.C, F4.2, SHUNTMON-B.RSN
- new net RST: ESP-12.REST, R16.1, SJ1.1
- new net SOURCE-POS-A_T: C2.2, C3.1, D3.C, F3.2, R1.2, SHUNTMON-A.RSP
- new net UNI_REF: C14.1, MCP3208.CH5, R7.1, R8.2, REF_SEL_A.1, REF_SEL_B.1
- new net VDD_PCF: C33T.+, PCF8523.VDD, R22.1
- new net VDD_RTC_POSTJUMPER: R20.1, R21.1, R22.2, SJ2.2
- new net V_IN_POSTFUSE: D1.C, F1.2, TP4.TP
- new net V_IN_PREFUSE: F1.1, PWR.2
- net +3V3: now also C15.1, C17.2, ESP-12.VCC, MCP3208.CH6, R12.2, R13.2, R16.2, R17.2, R5.2; no longer MCP3208.CH5, R26.2, R27.1, R28.1, SJ3.2
- net +5V: now also C19.1, MCP3208.VDD, MCP3208.VREF, R6.2, SHUNTMON-A.VCC, SHUNTMON-B.VCC; no longer FTDI_RFM.4, R10.2, SJ1.2
- net 3.3V_PRE: now also C32T.+, TP3.TP; no longer C18T.1, TP2.TP
- net 5V_PRE: now also 7.62_BARRIER-2.1, C31T.+, TP2.TP; no longer C1T.1, TP1.TP
- net 6.5V: now also C30T.+; no longer C11T.1
- net ADCSHUNT_A: now also C9.1
- net ADCSHUNT_B: now also C11.1
- net CH7: now also C16.1
- net CH_PD: now also R17.1; no longer R7.1
- net D0/RX: no longer FTDI_RFM.2
- net D1/TX: no longer FTDI_RFM.3
- net ESPRX: now also R14.2, R15.1; no longer R17.2, R18.1
- net GND: now also 7.62_BARRIER-1.1, C1.2, C30T.-, C31T.-, C32T.-, C33T.-, C4.2, C7.2, C8.2, J5.2, R10.2, R11.2, R15.2, R4.1, R8.1, TP6.TP, TP7.TP; no longer C10.2, C11T.2, C16.2, C18T.2, C1T.2, C23.1, C24.1, C25.2, C48.2, C5.2, C7T.2, D6.A, FTDI_RFM.6, R11.1, R15.1, R18.2, R21.1, R3.2, R8.2, REF_SEL_A.1, REF_SEL_B.1, REG0.GND, REG0.SGND
- net GPIO0: now also R13.1; no longer R12.1
- net GPIO12: now also R10.1, R9.2; no longer R4.2, R8.1
- net GPIO12A: now also R9.1; no longer R4.1
- net GPIO15: now also R11.1; no longer R3.1
- net GPIO2: now also R12.1; no longer R6.1
- net LOAD-NEG-A: now also F2.1, MOUNT_10.16_A.P$1, TP11.TP; no longer R16.1, X3-2.1
- net LOAD-NEG-B: now also F4.1, MOUNT_10.16_B.P$1, TP9.TP; no longer R23.1, X4-2.1
- net N$1: now also SJ4.1, TP1.TP, TP5.TP; no longer R20.1, R21.2, REG0.FB
- net N$36: now also R14.1; no longer R17.1
- net N$5: now also R5.1; no longer R26.1
- net REF_A_INPUT: now also C7.1
- net REF_B_INPUT: now also C8.1
- net SCL: no longer R27.2
- net SDA: no longer R28.2
- net SOURCE-POS-A: now also F3.1, MOUNT_10.16_A.P$2, TP10.TP; no longer R22.1, X3-1.1
- net SOURCE-POS-B: now also F5.1, MOUNT_10.16_B.P$2, TP8.TP; no longer R24.1, X4-1.1
- net SOURCE-POS-B_T: now also C5.2, F5.2, R3.2; no longer C8.2, R1.2, R24.2, SHUNTMON-B.VCC
- net VSENSE_A: now also R1.1, R2.2; no longer R14.1, R15.2
- net VSENSE_A_BUFF: now also C10.1
- net VSENSE_B: now also R3.1, R4.2; no longer R1.1, R2.2
- net VSENSE_B_BUFF: now also C12.1
- net _RESET: no longer C2.1
Other:
- note added: "ESP-12E/S/F"
- note added: "REF VOLTAGE"
- note added: "designed by Daniel Bates November 2018"
- note added: "emonDC v3.0 use of ESP module inspired by Heatpumpmonitor project. RTC layout taken from IoTaWatt."
- note removed: "ESP-12S"
- note removed: "designed by Daniel Bates July 2018"
- note removed: "emonDC v2.0 based on emonTx and Heatpumpmonitor"
- moved on the sheet: C1, C16, C2, C4, C5, C8, F1, GND, R1, R10, R11, R12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
