File: hardware/emonDCduo/emonDCduo-ESP v3.4.sch (EAGLE design)
At the start: 124 parts, among them IC1 DS18B20, P1 B4B-PH-K, Y1 32Khz

Commit message: commit v3.4
curvy corners!
Other:
- note added: "emonDC v3.4 use of ESP module inspired by Heatpumpmonitor project. RTC layout taken from IoTaWatt."
- note removed: "emonDC v3.0 use of ESP module inspired by Heatpumpmonitor project. RTC layout taken from IoTaWatt."
Changed lines of the file:
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@@
 <sheet>
 <plain>
-<text x="-82.55" y="184.15" size="1.778" layer="97">emonDC v3.0
+<text x="-82.55" y="184.15" size="1.778" layer="97">emonDC v3.4
 use of ESP module inspired by Heatpumpmonitor project. RTC layout taken from IoTaWatt.</text>
 <text x="-82.55" y="180.34" size="1.778" layer="97">designed by Daniel Bates     November 2018</text>

Commit message: commit v3.4
Parts:
- removed P1: B4B-PH-K, JST-PH:B4B-PH-K
- removed TP1, TP2, TP3: TPPAD1-13, testpad:TPPAD1-13
- removed TP12, TP13: TPPAD1-13Y, testpad:TPPAD1-13Y
- added SV1: (no value), con-lstb:MA04-1
- added U$7, U$8, U$9: TP0.8MM, testpad_db:TP0.8MM
- added X1: (no value), con-weidmueller-sl35_db:180-2
- U$1, U$4, U$5, U$6: value TP1.0MM -> TP0.8MM; device 1mm tesp pad:TP1.0MM -> testpad_db:TP0.8MM
Connections:
- net +3V3: now also SV1.3; no longer P1.3
- net 3.3V_PRE: now also U$8.P$1; no longer TP3.TP
- net 5V_PRE: now also U$7.P$1; no longer TP2.TP
- net GND: now also C10.2, C11.2, C12.2, C13.2, C14.2, C15.2, C16.2, C9.2, SV1.4, X1.1, X1.2; no longer P1.4, TP12.TP, TP13.TP
- net N$1: now also U$9.P$1; no longer TP1.TP
- net SCL: now also SV1.2; no longer P1.2
- net SDA: now also SV1.1; no longer P1.1
