File: hardware/emonDCduo/eagle7files/emonDCduo-ESP v1.3.brd (EAGLE design)
At the start: 99.1 x 76.5 mm, 81 parts, among them J5 455-1750-1-ND, P1 B4B-PH-K, Y1 32Khz

Commit message: readme updated
Parts:
- removed C1, C11, C12, C15, C17, C18, C19, C8: 100nF, rcl:C0603
- removed GND: (no value), con-weidmueller-sl35:180-2
- added USB_PWR: 5000751517_SD, 5000751517_sd:5000751517_SD
- moved SCREW_TERM_2 8.02 mm to (5.84, 32.8)
- moved SCREW_TERM_1 8.00 mm to (5.84, 51.3)
- moved R21 2.84 mm to (60.5, 74.9), turned to 0 degrees
- moved R20 2.30 mm to (63.8, 74.9)
- moved L1 1.02 mm to (48.8, 70.4)
- moved C24 0.51 mm to (28.5, 37.7)
- moved C6 0.51 mm to (28.5, 27.8)
- moved R5 0.51 mm to (33.6, 34.9)
- moved SCREW2 0.51 mm to (23.3, 32.8)
- moved SHUNTMON-B 0.51 mm to (29.8, 32.8)
- moved C9 0.51 mm to (30.7, 27.8)
- moved R1 0.51 mm to (35.8, 29.5)
- moved R2 0.51 mm to (35.8, 26.2)
- moved C3 0.25 mm to (62.1, 69.2)
Connections:
- net 3.3V: no longer C17.1
- net 5.0V: now also USB_PWR.VBUS; no longer MCP3208.15
- net ADCSHUNT-A: no longer C1.1
- net ADCSHUNT-B: no longer C11.1
- net CH6: no longer C18.1
- net CH7: no longer C19.1
- net GND: now also MCP3208.15, SCREW1.2, SCREW2.2, USB_PWR.GND1, USB_PWR.GND2, USB_PWR.GND3; no longer C1.2, C11.2, C12.2, C15.2, C17.2, C18.2, C19.2, C8.2, GND.1, GND.2
- net REF_INPUT: no longer C15.1
- net VSENSEA: no longer C8.1
- net VSENSEB: no longer C12.1
Routing:
- net SOURCE-POS-A: track 41.8 -> 68.3 mm, vias 38 -> 32
- net LOAD-NEG-B: track 9.89 -> 35.5 mm, vias 37 -> 31
- net SOURCE-POS-B: track 63.7 -> 81.6 mm, vias 38 -> 32
- net LOAD-NEG-A: track 10.4 -> 26.1 mm, vias 37 -> 31
- net GND: track 6.93 -> 0.00 mm, vias 61 -> 45
- net FB: track 23.5 -> 26.0 mm
- net 5.0V: track 168.9 -> 171.2 mm
- net 6.5V: track 27.5 -> 26.0 mm
- net GPIO12: track 106.3 -> 105.4 mm
- net REF_B_INPUT: track 17.7 -> 16.8 mm
- net VSENSEB: track 55.0 -> 55.7 mm
- removed copper zone on layer 1, net LOAD-NEG-A
- removed copper zone on layer 16, net LOAD-NEG-A
- removed copper zone on layer 1, net LOAD-NEG-B
- removed copper zone on layer 16, net LOAD-NEG-B
- removed copper zone on layer 1, net SOURCE-POS-A
- removed copper zone on layer 16, net SOURCE-POS-A
- removed copper zone on layer 1, net SOURCE-POS-B
- removed copper zone on layer 16, net SOURCE-POS-B
Other:
- board text added: "Designed in North Wales UK by Megni"
- board text added: "USB_PWR"
- board text added: "v1.3 Dec 2017 by DB"
- board text removed: "Designed in North Wales UK by Daniel Bates"
- board text removed: "by DB"
- board text removed: "v1.4 March 2018"
