File: hardware/emonDCduo/eagle7files/emonDCduo-ESP v1.3.sch (EAGLE design)
At the start: 81 parts, among them J5 455-1750-1-ND, P1 B4B-PH-K, Y1 32Khz

Commit message: readme updated
Parts:
- removed C1, C11, C12, C15, C17, C18, C19, C8: 100nF, rcl:C-EUC0603
- removed GND: (no value), con-weidmueller-sl35:180-2
- added USB_PWR: 5000751517_SD, 5000751517_sd:5000751517_SD
Connections:
- net 3.3V: no longer C17.1
- net 5.0V: now also USB_PWR.1; no longer MCP3208.VREF
- net ADCSHUNT-A: no longer C1.1
- net ADCSHUNT-B: no longer C11.1
- net CH6: no longer C18.1
- net CH7: no longer C19.1
- net GND: now also MCP3208.VREF, SCREW1.2, SCREW2.2, USB_PWR.5; no longer C1.2, C11.2, C12.2, C15.2, C17.2, C18.2, C19.2, C8.2, GND.1, GND.2
- net REF_INPUT: no longer C15.1
- net VSENSEA: no longer C8.1
- net VSENSEB: no longer C12.1
Other:
- note added: "Daniel Bates Dec 2017"
- note added: "emonDC v1.3 : based on emonTx v3.4 by Glyn Hudson and Trystan Lea OpenEnergyMonitor.org"
- note removed: "designed by Daniel Bates March 2018"
- note removed: "emonDC v1.4 : based on emonTx v3.4 OpenEnergyMonitor.org"
